Commit message: fix the planning group

File: pepper_robot_moveit_config/srdf/pepper_arms.xacro (robot description, xacro)
@@ -1,182 +1,62 @@
-<?xml version="1.0" ?>
-<!--******************************************************************
- ****** File automatically generated by generate_urdf.py script ******
- *********************************************************************-->
-<robot xmlns:xacro="http://www.ros.org/wiki/xacro">
-	<joint name="LShoulderPitch" type="revolute">
-		<parent link="torso"/>
-		<child link="LShoulder"/>
-		<origin rpy="0 0 0" xyz="-0.057 0.14974 0.08682"/>
-		<axis xyz="0 1.0 0"/>
-		<limit effort="5.428" lower="-2.08567" upper="2.08567" velocity="7.33998"/>
-	</joint>
-	<link name="LShoulder">
-		<inertial>
-			<mass value="0.3125"/>
-			<inertia ixx="0.000361198" ixy="-1.98347e-06" ixz="6.35907e-07" iyy="0.000137229" iyz="-5.68878e-06" izz="0.000399194"/>
-			<origin rpy="0 0 0" xyz="0.00018 -0.01856 0.00099"/>
-		</inertial>
-		<xacro:insert_visu_LShoulder/>
-	</link>
-	<joint name="LShoulderRoll" type="revolute">
-		<parent link="LShoulder"/>
-		<child link="LBicep"/>
-		<origin rpy="0 0 0" xyz="0 0 0"/>
-		<axis xyz="0 0 1.0"/>
-		<limit effort="2.666" lower="0.00872665" upper="1.56207" velocity="9.22756"/>
-	</joint>
-	<link name="LBicep">
-		<inertial>
-			<mass value="0.50527"/>
-			<inertia ixx="0.000500872" ixy="-3.55918e-05" ixz="8.51263e-05" iyy="0.00126284" iyz="9.06813e-06" izz="0.00115718"/>
-			<origin rpy="0 0 0" xyz="0.08151 0.01284 -0.01017"/>
-		</inertial>
-		<xacro:insert_visu_LBicep/>
-	</link>
-	<joint name="LElbowYaw" type="revolute">
-		<parent link="LBicep"/>
-		<child link="LElbow"/>
-		<origin rpy="0 -0.157079 0" xyz="0.1812 0.015 0.00013"/>
-		<axis xyz="1.0 0 0"/>
-		<limit effort="5.428" lower="-2.08567" upper="2.08567" velocity="7.33998"/>
-	</joint>
-	<link name="LElbow">
-		<inertial>
-			<mass value="0.27495"/>
-			<inertia ixx="0.000122971" ixy="9.86024e-07" ixz="-2.55838e-05" iyy="0.000331766" iyz="-1.98925e-06" izz="0.000303047"/>
-			<origin rpy="0 0 0" xyz="-0.02297 -0.00019 0.00119"/>
-		</inertial>
-		<xacro:insert_visu_LElbow/>
-	</link>
-	<joint name="LElbowRoll" type="revolute">
-		<parent link="LElbow"/>
-		<child link="LForeArm"/>
-		<origin rpy="0 0 0" xyz="0 0 0"/>
-		<axis xyz="0 0 1.0"/>
-		<limit effort="2.666" lower="-1.56207" upper="-0.00872665" velocity="9.22756"/>
-	</joint>
-	<link name="LForeArm">
-		<inertial>
-			<mass value="0.16579"/>
-			<inertia ixx="0.00156513" ixy="1.47517e-05" ixz="-6.05746e-05" iyy="0.00173219" iyz="-1.7619e-07" izz="0.000273081"/>
-			<origin rpy="0 0 0" xyz="0.0593 0.00271 -0.01014"/>
-		</inertial>
-		<xacro:insert_visu_LForeArm/>
-	</link>
-	<joint name="LWristYaw" type="revolute">
-		<parent link="LForeArm"/>
-		<child link="l_wrist"/>
-		<origin rpy="0 0 0" xyz="0.15 0 0"/>
-		<axis xyz="1.0 0 0"/>
-		<limit effort="0.2014" lower="-1.82387" upper="1.82387" velocity="17.3835"/>
-	</joint>
-	<link name="l_wrist">
-		<inertial>
-			<mass value="0.27555"/>
-			<inertia ixx="0.000151643" ixy="1.06629e-05" ixz="2.89509e-06" iyy="0.000431099" iyz="-3.13715e-06" izz="0.000456172"/>
-			<origin rpy="0 0 0" xyz="0.03536 -0.00072 -0.00207"/>
-		</inertial>
-		<xacro:insert_visu_l_wrist/>
-	</link>
-	<joint name="LHand" type="revolute">
-		<parent link="l_wrist"/>
-		<child link="l_gripper"/>
-		<origin rpy="0 0 0" xyz="0.025 0 0"/>
-		<axis xyz="1.0 0 0"/>
-		<limit effort="0.144" lower="0.02" upper="0.98" velocity="12.56"/>
-	</joint>
-	<link name="l_gripper">
-		<inertial>
-			<mass value="2e-06"/>
-			<inertia ixx="1.1e-09" ixy="0" ixz="0" iyy="1.1e-09" iyz="0" izz="1.1e-09"/>
-		</inertial>
-	</link>
-	<joint name="RShoulderPitch" type="revolute">
-		<parent link="torso"/>
-		<child link="RShoulder"/>
-		<origin rpy="0 0 0" xyz="-0.057 -0.14974 0.08682"/>
-		<axis xyz="0 1.0 0"/>
-		<limit effort="5.428" lower="-2.08567" upper="2.08567" velocity="7.33998"/>
-	</joint>
-	<link name="RShoulder">
-		<inertial>
-			<mass value="0.3125"/>
-			<inertia ixx="0.000361198" ixy="1.98347e-06" ixz="6.35907e-07" iyy="0.000137229" iyz="5.68878e-06" izz="0.000399194"/>
-			<origin rpy="0 0 0" xyz="0.00018 0.01856 0.00099"/>
-		</inertial>
-		<xacro:insert_visu_RShoulder/>
-	</link>
-	<joint name="RShoulderRoll" type="revolute">
-		<parent link="RShoulder"/>
-		<child link="RBicep"/>
-		<origin rpy="0 0 0" xyz="0 0 0"/>
-		<axis xyz="0 0 1.0"/>
-		<limit effort="2.666" lower="-1.56207" upper="-0.00872665" velocity="9.22756"/>
-	</joint>
-	<link name="RBicep">
-		<inertial>
-			<mass value="0.50527"/>
-			<inertia ixx="0.000500872" ixy="3.55918e-05" ixz="8.51263e-05" iyy="0.00126284" iyz="-9.06813e-06" izz="0.00115718"/>
-			<origin rpy="0 0 0" xyz="0.08151 -0.01284 -0.01017"/>
-		</inertial>
-		<xacro:insert_visu_RBicep/>
-	</link>
-	<joint name="RElbowYaw" type="revolute">
-		<parent link="RBicep"/>
-		<child link="RElbow"/>
-		<origin rpy="0 -0.157079 0" xyz="0.1812 -0.015 0.00013"/>
-		<axis xyz="1.0 0 0"/>
-		<limit effort="5.428" lower="-2.08567" upper="2.08567" velocity="7.33998"/>
-	</joint>
-	<link name="RElbow">
-		<inertial>
-			<mass value="0.27495"/>
-			<inertia ixx="0.000122971" ixy="-9.86024e-07" ixz="-2.55838e-05" iyy="0.000331766" iyz="1.98925e-06" izz="0.000303047"/>
-			<origin rpy="0 0 0" xyz="-0.02297 0.00019 0.00119"/>
-		</inertial>
-		<xacro:insert_visu_RElbow/>
-	</link>
-	<joint name="RElbowRoll" type="revolute">
-		<parent link="RElbow"/>
-		<child link="RForeArm"/>
-		<origin rpy="0 0 0" xyz="0 0 0"/>
-		<axis xyz="0 0 1.0"/>
-		<limit effort="2.666" lower="0.00872665" upper="1.56207" velocity="9.22756"/>
-	</joint>
-	<link name="RForeArm">
-		<inertial>
-			<mass value="0.16579"/>
-			<inertia ixx="0.00156513" ixy="-1.47517e-05" ixz="-6.05746e-05" iyy="0.00173219" iyz="1.7619e-07" izz="0.000273081"/>
-			<origin rpy="0 0 0" xyz="0.0593 -0.00271 -0.01014"/>
-		</inertial>
-		<xacro:insert_visu_RForeArm/>
-	</link>
-	<joint name="RWristYaw" type="revolute">
-		<parent link="RForeArm"/>
-		<child link="r_wrist"/>
-		<origin rpy="0 0 0" xyz="0.15 0 0"/>
-		<axis xyz="1.0 0 0"/>
-		<limit effort="0.2014" lower="-1.82387" upper="1.82387" velocity="17.3835"/>
-	</joint>
-	<link name="r_wrist">
-		<inertial>
-			<mass value="0.27555"/>
-			<inertia ixx="0.000151643" ixy="-1.06629e-05" ixz="2.89509e-06" iyy="0.000431099" iyz="3.13715e-06" izz="0.000456172"/>
-			<origin rpy="0 0 0" xyz="0.03536 0.00072 -0.00207"/>
-		</inertial>
-		<xacro:insert_visu_r_wrist/>
-	</link>
-	<joint name="RHand" type="revolute">
-		<parent link="r_wrist"/>
-		<child link="r_gripper"/>
-		<origin rpy="0 0 0" xyz="0.025 0 0"/>
-		<axis xyz="1.0 0 0"/>
-		<limit effort="0.144" lower="0.02" upper="0.98" velocity="12.56"/>
-	</joint>
-	<link name="r_gripper">
-		<inertial>
-			<mass value="2e-06"/>
-			<inertia ixx="1.1e-09" ixy="0" ixz="0" iyy="1.1e-09" iyz="0" izz="1.1e-09"/>
-		</inertial>
-	</link>
+<?xml version="1.0"?>
+<robot xmlns:xacro="http://wiki.ros.org/xacro">
+   <xacro:macro name="pepper_robot" params="
+   prefix:=pepper_robot_
+  ">
+    <group name="arm">
+      <chain base_link="${prefix}link_base" tip_link="${prefix}end_effector"/>
+    </group>
+    <group name="gripper">
+      <joint name="${prefix}LHand"/>
+      <passive_joint name="${prefix}LFinger11"/>
+      <passive_joint name="${prefix}LFinger12"/>
+      <passive_joint name="${prefix}LFinger13"/>
+      <passive_joint name="${prefix}LFinger21"/>
+      <passive_joint name="${prefix}LFinger22"/>
+      <passive_joint name="${prefix}LFinger23"/>
+      <passive_joint name="${prefix}LFinger31"/>
+      <passive_joint name="${prefix}LFinger32"/>
+      <passive_joint name="${prefix}LFinger33"/>
+      <passive_joint name="${prefix}LFinger41"/>
+      <passive_joint name="${prefix}LFinger42"/>
+      <passive_joint name="${prefix}LFinger43"/>
+      <passive_joint name="${prefix}LThumb1"/>
+      <passive_joint name="${prefix}LThumb2"/>
+    </group>
+    <group_state name="vertical" group="arm">
+      <joint name="${prefix}LElbowRoll" value="${-1*pi/180}"/>
+      <joint name="${prefix}LElbowYaw" value="${120*pi/180}"/>
+      <joint name="${prefix}LShoulderPitch" value="${120*pi/180}"/>
+      <joint name="${prefix}LShoulderRoll" value="${90*pi/180}"/>
+      <joint name="${prefix}LWristYaw" value="${105*pi/180}"/>
+    </group_state>
+    <group_state name="home" group="arm">
+      <joint name="${prefix}LElbowRoll" value="${-90*pi/180}"/>
+      <joint name="${prefix}LElbowYaw" value="${-120*pi/180}"/>
+      <joint name="${prefix}LShoulderPitch" value="${-120*pi/180}"/>
+      <joint name="${prefix}LShoulderRoll" value="${1*pi/180}"/>
+      <joint name="${prefix}LWristYaw" value="${-105*pi/180}"/>
+    </group_state>
+    <group_state name="open" group="gripper">
+      <joint name="${prefix}LHand" value="${56*pi/180}"/>
+    </group_state>
+    <group_state name="close" group="gripper">
+      <joint name="${prefix}LHand" value="${1*pi/180}"/>
+    </group_state>
+    <end_effector name="gripper" parent_link="${prefix}end_effector" group="gripper" parent_group="arm"/>
+    <passive_joint name="${prefix}LFinger11"/>
+    <passive_joint name="${prefix}LFinger12"/>
+    <passive_joint name="${prefix}LFinger13"/>
+    <passive_joint name="${prefix}LFinger21"/>
+    <passive_joint name="${prefix}LFinger22"/>
+    <passive_joint name="${prefix}LFinger23"/>
+    <passive_joint name="${prefix}LFinger31"/>
+    <passive_joint name="${prefix}LFinger32"/>
+    <passive_joint name="${prefix}LFinger33"/>
+    <passive_joint name="${prefix}LFinger41"/>
+    <passive_joint name="${prefix}LFinger42"/>
+    <passive_joint name="${prefix}LFinger43"/>
+    <passive_joint name="${prefix}LThumb1"/>
+    <passive_joint name="${prefix}LThumb2"/>
+  </xacro:macro>
 </robot>
