Commit message: test

File: pepper_robot_moveit_config/srdf/pepper_robot.xacro (robot description, xacro)
@@ -1,1042 +1,23 @@
 <?xml version="1.0" ?>
-<!--This does not replace URDF, and is not an extension of URDF.
-    This is a format for representing semantic information about the robot structure.
-    A URDF file must exist for this robot as well, where the joints and the links that are referenced are defined
--->
-<robot name="JulietteY20MP">
-    <!--GROUPS: Representation of a set of joints and links. This can be useful for specifying DOF to plan for, defining arms, end effectors, etc-->
-    <!--LINKS: When a link is specified, the parent joint of that link (if it exists) is automatically included-->
-    <!--JOINTS: When a joint is specified, the child link of that joint (which will always exist) is automatically included-->
-    <!--CHAINS: When a chain is specified, all the links along the chain (including endpoints) are included in the group. Additionally, all the joints that are parents to included links are also included. This means that joints along the chain and the parent joint of the base link are included in the group-->
-    <!--SUBGROUPS: Groups can also be formed by referencing to already defined group names-->
-    <group name="right_arm">
-        <chain base_link="torso" tip_link="r_wrist" />
-    </group>
-    <group name="left_arm">
-        <chain base_link="torso" tip_link="l_wrist" />
-    </group>
-    <group name="both_arms">
-        <group name="left_arm" />
-        <group name="right_arm" />
-    </group>
-    <group name="right_hand">
-        <link name="RFinger11_link" />
-        <link name="RFinger12_link" />
-        <link name="RFinger13_link" />
-        <link name="RFinger21_link" />
-        <link name="RFinger22_link" />
-        <link name="RFinger23_link" />
-        <link name="RFinger31_link" />
-        <link name="RFinger32_link" />
-        <link name="RFinger33_link" />
-        <link name="RFinger41_link" />
-        <link name="RFinger42_link" />
-        <link name="RFinger43_link" />
-        <link name="r_gripper" />
-        <link name="RThumb1_link" />
-        <link name="RThumb2_link" />
-        <joint name="RHand" />
-    </group>
-    <group name="left_hand">
-        <link name="LFinger11_link" />
-        <link name="LFinger12_link" />
-        <link name="LFinger13_link" />
-        <link name="LFinger21_link" />
-        <link name="LFinger22_link" />
-        <link name="LFinger23_link" />
-        <link name="LFinger31_link" />
-        <link name="LFinger32_link" />
-        <link name="LFinger33_link" />
-        <link name="LFinger41_link" />
-        <link name="LFinger42_link" />
-        <link name="LFinger43_link" />
-        <link name="l_gripper" />
-        <link name="LThumb1_link" />
-        <link name="LThumb2_link" />
-        <joint name="LHand" />
-    </group>
-    <group name="base">
-        <joint name="virtual_odom" />
-    </group>
-    <group name="head">
-        <chain base_link="torso" tip_link="Head" />
-    </group>
-    <!--END EFFECTOR: Purpose: Represent information about an end effector.-->
-    <end_effector name="left_eef" parent_link="l_wrist" group="left_hand" />
-    <end_effector name="right_eef" parent_link="r_wrist" group="right_hand" />
-    <!--VIRTUAL JOINT: Purpose: this element defines a virtual joint between a robot link and an external frame of reference (considered fixed with respect to the robot)-->
-    <virtual_joint name="virtual_odom" type="floating" parent_frame="odom" child_link="base_link" />
-    <!--PASSIVE JOINT: Purpose: this element is used to mark joints that are not actuated-->
-    <passive_joint name="virtual_odom" />
-    <passive_joint name="LFinger11" />
-    <passive_joint name="LFinger12" />
-    <passive_joint name="LFinger13" />
-    <passive_joint name="LFinger21" />
-    <passive_joint name="LFinger22" />
-    <passive_joint name="LFinger23" />
-    <passive_joint name="LFinger31" />
-    <passive_joint name="LFinger32" />
-    <passive_joint name="LFinger33" />
-    <passive_joint name="LFinger41" />
-    <passive_joint name="LFinger42" />
-    <passive_joint name="LFinger43" />
-    <passive_joint name="LThumb1" />
-    <passive_joint name="LThumb2" />
-    <passive_joint name="RFinger11" />
-    <passive_joint name="RFinger12" />
-    <passive_joint name="RFinger13" />
-    <passive_joint name="RFinger21" />
-    <passive_joint name="RFinger22" />
-    <passive_joint name="RFinger23" />
-    <passive_joint name="RFinger31" />
-    <passive_joint name="RFinger32" />
-    <passive_joint name="RFinger33" />
-    <passive_joint name="RFinger41" />
-    <passive_joint name="RFinger42" />
-    <passive_joint name="RFinger43" />
-    <passive_joint name="RThumb1" />
-    <passive_joint name="RThumb2" />
-    <passive_joint name="WheelFL" />
-    <passive_joint name="WheelFR" />
-    <passive_joint name="WheelB" />
-    <!--DISABLE COLLISIONS: By default it is assumed that any link of the robot could potentially come into collision with any other link in the robot. This tag disables collision checking between a specified pair of links. -->
-    <disable_collisions link1="Head" link2="Hip" reason="Never" />
-    <disable_collisions link1="Head" link2="LShoulder" reason="Never" />
-    <disable_collisions link1="Head" link2="Neck" reason="Adjacent" />
-    <disable_collisions link1="Head" link2="Pelvis" reason="Never" />
-    <disable_collisions link1="Head" link2="RShoulder" reason="Never" />
-    <disable_collisions link1="Head" link2="Tibia" reason="Never" />
-    <disable_collisions link1="Head" link2="WheelB_link" reason="Never" />
-    <disable_collisions link1="Head" link2="WheelFL_link" reason="Never" />
-    <disable_collisions link1="Head" link2="WheelFR_link" reason="Never" />
-    <disable_collisions link1="Hip" link2="LBicep" reason="Never" />
-    <disable_collisions link1="Hip" link2="LElbow" reason="Never" />
-    <disable_collisions link1="Hip" link2="LForeArm" reason="Never" />
-    <disable_collisions link1="Hip" link2="LShoulder" reason="Never" />
-    <disable_collisions link1="Hip" link2="Neck" reason="Never" />
-    <disable_collisions link1="Hip" link2="Pelvis" reason="Adjacent" />
-    <disable_collisions link1="Hip" link2="RBicep" reason="Never" />
-    <disable_collisions link1="Hip" link2="RElbow" reason="Never" />
-    <disable_collisions link1="Hip" link2="RForeArm" reason="Never" />
-    <disable_collisions link1="Hip" link2="RShoulder" reason="Never" />
-    <disable_collisions link1="Hip" link2="Tibia" reason="Never" />
-    <disable_collisions link1="Hip" link2="WheelB_link" reason="Never" />
-    <disable_collisions link1="Hip" link2="WheelFL_link" reason="Never" />
-    <disable_collisions link1="Hip" link2="WheelFR_link" reason="Never" />
-    <disable_collisions link1="Hip" link2="torso" reason="Adjacent" />
-    <disable_collisions link1="LBicep" link2="LElbow" reason="Adjacent" />
-    <disable_collisions link1="LBicep" link2="LFinger11_link" reason="Never" />
-    <disable_collisions link1="LBicep" link2="LFinger12_link" reason="Never" />
-    <disable_collisions link1="LBicep" link2="LFinger13_link" reason="Never" />
-    <disable_collisions link1="LBicep" link2="LFinger21_link" reason="Never" />
-    <disable_collisions link1="LBicep" link2="LFinger22_link" reason="Never" />
-    <disable_collisions link1="LBicep" link2="LFinger23_link" reason="Never" />
-    <disable_collisions link1="LBicep" link2="LFinger31_link" reason="Never" />
-    <disable_collisions link1="LBicep" link2="LFinger32_link" reason="Never" />
-    <disable_collisions link1="LBicep" link2="LFinger33_link" reason="Never" />
-    <disable_collisions link1="LBicep" link2="LFinger41_link" reason="Never" />
-    <disable_collisions link1="LBicep" link2="LFinger42_link" reason="Never" />
-    <disable_collisions link1="LBicep" link2="LFinger43_link" reason="Never" />
-    <disable_collisions link1="LBicep" link2="LShoulder" reason="Adjacent" />
-    <disable_collisions link1="LBicep" link2="LThumb1_link" reason="Never" />
-    <disable_collisions link1="LBicep" link2="LThumb2_link" reason="Never" />
-    <disable_collisions link1="LBicep" link2="Neck" reason="Never" />
-    <disable_collisions link1="LBicep" link2="Pelvis" reason="Never" />
-    <disable_collisions link1="LBicep" link2="RBicep" reason="Never" />
-    <disable_collisions link1="LBicep" link2="RElbow" reason="Never" />
-    <disable_collisions link1="LBicep" link2="RFinger11_link" reason="Never" />
-    <disable_collisions link1="LBicep" link2="RFinger12_link" reason="Never" />
-    <disable_collisions link1="LBicep" link2="RFinger13_link" reason="Never" />
-    <disable_collisions link1="LBicep" link2="RFinger21_link" reason="Never" />
-    <disable_collisions link1="LBicep" link2="RFinger22_link" reason="Never" />
-    <disable_collisions link1="LBicep" link2="RFinger23_link" reason="Never" />
-    <disable_collisions link1="LBicep" link2="RFinger31_link" reason="Never" />
-    <disable_collisions link1="LBicep" link2="RFinger32_link" reason="Never" />
-    <disable_collisions link1="LBicep" link2="RFinger33_link" reason="Never" />
-    <disable_collisions link1="LBicep" link2="RFinger41_link" reason="Never" />
-    <disable_collisions link1="LBicep" link2="RFinger42_link" reason="Never" />
-    <disable_collisions link1="LBicep" link2="RFinger43_link" reason="Never" />
-    <disable_collisions link1="LBicep" link2="RForeArm" reason="Never" />
-    <disable_collisions link1="LBicep" link2="RShoulder" reason="Never" />
-    <disable_collisions link1="LBicep" link2="RThumb1_link" reason="Never" />
-    <disable_collisions link1="LBicep" link2="RThumb2_link" reason="Never" />
-    <disable_collisions link1="LBicep" link2="Tibia" reason="Never" />
-    <disable_collisions link1="LBicep" link2="WheelB_link" reason="Never" />
-    <disable_collisions link1="LBicep" link2="WheelFL_link" reason="Never" />
-    <disable_collisions link1="LBicep" link2="WheelFR_link" reason="Never" />
-    <disable_collisions link1="LBicep" link2="l_wrist" reason="Never" />
-    <disable_collisions link1="LBicep" link2="r_wrist" reason="Never" />
-    <disable_collisions link1="LBicep" link2="torso" reason="Default" />
-    <disable_collisions link1="LElbow" link2="LFinger11_link" reason="Never" />
-    <disable_collisions link1="LElbow" link2="LFinger12_link" reason="Never" />
-    <disable_collisions link1="LElbow" link2="LFinger13_link" reason="Never" />
-    <disable_collisions link1="LElbow" link2="LFinger21_link" reason="Never" />
-    <disable_collisions link1="LElbow" link2="LFinger22_link" reason="Never" />
-    <disable_collisions link1="LElbow" link2="LFinger23_link" reason="Never" />
-    <disable_collisions link1="LElbow" link2="LFinger31_link" reason="Never" />
-    <disable_collisions link1="LElbow" link2="LFinger32_link" reason="Never" />
-    <disable_collisions link1="LElbow" link2="LFinger33_link" reason="Never" />
-    <disable_collisions link1="LElbow" link2="LFinger41_link" reason="Never" />
-    <disable_collisions link1="LElbow" link2="LFinger42_link" reason="Never" />
-    <disable_collisions link1="LElbow" link2="LFinger43_link" reason="Never" />
-    <disable_collisions link1="LElbow" link2="LForeArm" reason="Adjacent" />
-    <disable_collisions link1="LElbow" link2="LShoulder" reason="Never" />
-    <disable_collisions link1="LElbow" link2="LThumb1_link" reason="Never" />
-    <disable_collisions link1="LElbow" link2="LThumb2_link" reason="Never" />
-    <disable_collisions link1="LElbow" link2="Neck" reason="Never" />
-    <disable_collisions link1="LElbow" link2="Pelvis" reason="Never" />
-    <disable_collisions link1="LElbow" link2="RBicep" reason="Never" />
-    <disable_collisions link1="LElbow" link2="RElbow" reason="Never" />
-    <disable_collisions link1="LElbow" link2="RFinger11_link" reason="Never" />
-    <disable_collisions link1="LElbow" link2="RFinger12_link" reason="Never" />
-    <disable_collisions link1="LElbow" link2="RFinger13_link" reason="Never" />
-    <disable_collisions link1="LElbow" link2="RFinger21_link" reason="Never" />
-    <disable_collisions link1="LElbow" link2="RFinger22_link" reason="Never" />
-    <disable_collisions link1="LElbow" link2="RFinger23_link" reason="Never" />
-    <disable_collisions link1="LElbow" link2="RFinger31_link" reason="Never" />
-    <disable_collisions link1="LElbow" link2="RFinger32_link" reason="Never" />
-    <disable_collisions link1="LElbow" link2="RFinger33_link" reason="Never" />
-    <disable_collisions link1="LElbow" link2="RFinger41_link" reason="Never" />
-    <disable_collisions link1="LElbow" link2="RFinger42_link" reason="Never" />
-    <disable_collisions link1="LElbow" link2="RFinger43_link" reason="Never" />
-    <disable_collisions link1="LElbow" link2="RForeArm" reason="Never" />
-    <disable_collisions link1="LElbow" link2="RShoulder" reason="Never" />
-    <disable_collisions link1="LElbow" link2="RThumb1_link" reason="Never" />
-    <disable_collisions link1="LElbow" link2="RThumb2_link" reason="Never" />
-    <disable_collisions link1="LElbow" link2="Tibia" reason="Never" />
-    <disable_collisions link1="LElbow" link2="WheelB_link" reason="Never" />
-    <disable_collisions link1="LElbow" link2="WheelFL_link" reason="Never" />
-    <disable_collisions link1="LElbow" link2="WheelFR_link" reason="Never" />
-    <disable_collisions link1="LElbow" link2="l_wrist" reason="Never" />
-    <disable_collisions link1="LElbow" link2="r_wrist" reason="Never" />
-    <disable_collisions link1="LElbow" link2="torso" reason="Never" />
-    <disable_collisions link1="LFinger11_link" link2="LFinger12_link" reason="Adjacent" />
-    <disable_collisions link1="LFinger11_link" link2="LFinger13_link" reason="Never" />
-    <disable_collisions link1="LFinger11_link" link2="LFinger21_link" reason="Never" />
-    <disable_collisions link1="LFinger11_link" link2="LFinger22_link" reason="Never" />
-    <disable_collisions link1="LFinger11_link" link2="LFinger23_link" reason="Never" />
-    <disable_collisions link1="LFinger11_link" link2="LFinger31_link" reason="Never" />
-    <disable_collisions link1="LFinger11_link" link2="LFinger32_link" reason="Never" />
-    <disable_collisions link1="LFinger11_link" link2="LFinger33_link" reason="Never" />
-    <disable_collisions link1="LFinger11_link" link2="LFinger41_link" reason="Never" />
-    <disable_collisions link1="LFinger11_link" link2="LFinger42_link" reason="Never" />
-    <disable_collisions link1="LFinger11_link" link2="LFinger43_link" reason="Never" />
-    <disable_collisions link1="LFinger11_link" link2="LForeArm" reason="Never" />
-    <disable_collisions link1="LFinger11_link" link2="LShoulder" reason="Never" />
-    <disable_collisions link1="LFinger11_link" link2="LThumb1_link" reason="Never" />
-    <disable_collisions link1="LFinger11_link" link2="LThumb2_link" reason="Never" />
-    <disable_collisions link1="LFinger11_link" link2="Neck" reason="Never" />
-    <disable_collisions link1="LFinger11_link" link2="RBicep" reason="Never" />
-    <disable_collisions link1="LFinger11_link" link2="RElbow" reason="Never" />
-    <disable_collisions link1="LFinger11_link" link2="RFinger11_link" reason="Never" />
-    <disable_collisions link1="LFinger11_link" link2="RFinger12_link" reason="Never" />
-    <disable_collisions link1="LFinger11_link" link2="RFinger13_link" reason="Never" />
-    <disable_collisions link1="LFinger11_link" link2="RFinger21_link" reason="Never" />
-    <disable_collisions link1="LFinger11_link" link2="RFinger22_link" reason="Never" />
-    <disable_collisions link1="LFinger11_link" link2="RFinger23_link" reason="Never" />
-    <disable_collisions link1="LFinger11_link" link2="RFinger31_link" reason="Never" />
-    <disable_collisions link1="LFinger11_link" link2="RFinger32_link" reason="Never" />
-    <disable_collisions link1="LFinger11_link" link2="RFinger33_link" reason="Never" />
-    <disable_collisions link1="LFinger11_link" link2="RFinger41_link" reason="Never" />
-    <disable_collisions link1="LFinger11_link" link2="RFinger42_link" reason="Never" />
-    <disable_collisions link1="LFinger11_link" link2="RFinger43_link" reason="Never" />
-    <disable_collisions link1="LFinger11_link" link2="RForeArm" reason="Never" />
-    <disable_collisions link1="LFinger11_link" link2="RShoulder" reason="Never" />
-    <disable_collisions link1="LFinger11_link" link2="RThumb1_link" reason="Never" />
-    <disable_collisions link1="LFinger11_link" link2="RThumb2_link" reason="Never" />
-    <disable_collisions link1="LFinger11_link" link2="Tibia" reason="Never" />
-    <disable_collisions link1="LFinger11_link" link2="WheelB_link" reason="Never" />
-    <disable_collisions link1="LFinger11_link" link2="WheelFL_link" reason="Never" />
-    <disable_collisions link1="LFinger11_link" link2="WheelFR_link" reason="Never" />
-    <disable_collisions link1="LFinger11_link" link2="l_wrist" reason="Adjacent" />
-    <disable_collisions link1="LFinger11_link" link2="r_wrist" reason="Never" />
-    <disable_collisions link1="LFinger12_link" link2="LFinger13_link" reason="Adjacent" />
-    <disable_collisions link1="LFinger12_link" link2="LFinger21_link" reason="Never" />
-    <disable_collisions link1="LFinger12_link" link2="LFinger22_link" reason="Never" />
-    <disable_collisions link1="LFinger12_link" link2="LFinger23_link" reason="Never" />
-    <disable_collisions link1="LFinger12_link" link2="LFinger31_link" reason="Never" />
-    <disable_collisions link1="LFinger12_link" link2="LFinger32_link" reason="Never" />
-    <disable_collisions link1="LFinger12_link" link2="LFinger33_link" reason="Never" />
-    <disable_collisions link1="LFinger12_link" link2="LFinger41_link" reason="Never" />
-    <disable_collisions link1="LFinger12_link" link2="LFinger42_link" reason="Never" />
-    <disable_collisions link1="LFinger12_link" link2="LFinger43_link" reason="Never" />
-    <disable_collisions link1="LFinger12_link" link2="LForeArm" reason="Never" />
-    <disable_collisions link1="LFinger12_link" link2="LShoulder" reason="Never" />
-    <disable_collisions link1="LFinger12_link" link2="LThumb1_link" reason="Never" />
-    <disable_collisions link1="LFinger12_link" link2="LThumb2_link" reason="Never" />
-    <disable_collisions link1="LFinger12_link" link2="Neck" reason="Never" />
-    <disable_collisions link1="LFinger12_link" link2="RBicep" reason="Never" />
-    <disable_collisions link1="LFinger12_link" link2="RElbow" reason="Never" />
-    <disable_collisions link1="LFinger12_link" link2="RFinger11_link" reason="Never" />
-    <disable_collisions link1="LFinger12_link" link2="RFinger12_link" reason="Never" />
-    <disable_collisions link1="LFinger12_link" link2="RFinger13_link" reason="Never" />
-    <disable_collisions link1="LFinger12_link" link2="RFinger21_link" reason="Never" />
-    <disable_collisions link1="LFinger12_link" link2="RFinger22_link" reason="Never" />
-    <disable_collisions link1="LFinger12_link" link2="RFinger23_link" reason="Never" />
-    <disable_collisions link1="LFinger12_link" link2="RFinger31_link" reason="Never" />
-    <disable_collisions link1="LFinger12_link" link2="RFinger32_link" reason="Never" />
-    <disable_collisions link1="LFinger12_link" link2="RFinger33_link" reason="Never" />
-    <disable_collisions link1="LFinger12_link" link2="RFinger41_link" reason="Never" />
-    <disable_collisions link1="LFinger12_link" link2="RFinger42_link" reason="Never" />
-    <disable_collisions link1="LFinger12_link" link2="RFinger43_link" reason="Never" />
-    <disable_collisions link1="LFinger12_link" link2="RForeArm" reason="Never" />
-    <disable_collisions link1="LFinger12_link" link2="RShoulder" reason="Never" />
-    <disable_collisions link1="LFinger12_link" link2="RThumb1_link" reason="Never" />
-    <disable_collisions link1="LFinger12_link" link2="RThumb2_link" reason="Never" />
-    <disable_collisions link1="LFinger12_link" link2="WheelB_link" reason="Never" />
-    <disable_collisions link1="LFinger12_link" link2="WheelFL_link" reason="Never" />
-    <disable_collisions link1="LFinger12_link" link2="WheelFR_link" reason="Never" />
-    <disable_collisions link1="LFinger12_link" link2="l_wrist" reason="Never" />
-    <disable_collisions link1="LFinger12_link" link2="r_wrist" reason="Never" />
-    <disable_collisions link1="LFinger13_link" link2="LFinger21_link" reason="Never" />
-    <disable_collisions link1="LFinger13_link" link2="LFinger22_link" reason="Never" />
-    <disable_collisions link1="LFinger13_link" link2="LFinger23_link" reason="Never" />
-    <disable_collisions link1="LFinger13_link" link2="LFinger31_link" reason="Never" />
-    <disable_collisions link1="LFinger13_link" link2="LFinger32_link" reason="Never" />
-    <disable_collisions link1="LFinger13_link" link2="LFinger33_link" reason="Never" />
-    <disable_collisions link1="LFinger13_link" link2="LFinger41_link" reason="Never" />
-    <disable_collisions link1="LFinger13_link" link2="LFinger42_link" reason="Never" />
-    <disable_collisions link1="LFinger13_link" link2="LFinger43_link" reason="Never" />
-    <disable_collisions link1="LFinger13_link" link2="LForeArm" reason="Never" />
-    <disable_collisions link1="LFinger13_link" link2="LShoulder" reason="Never" />
-    <disable_collisions link1="LFinger13_link" link2="LThumb1_link" reason="Never" />
-    <disable_collisions link1="LFinger13_link" link2="LThumb2_link" reason="Never" />
-    <disable_collisions link1="LFinger13_link" link2="Neck" reason="Never" />
-    <disable_collisions link1="LFinger13_link" link2="RBicep" reason="Never" />
-    <disable_collisions link1="LFinger13_link" link2="RElbow" reason="Never" />
-    <disable_collisions link1="LFinger13_link" link2="RFinger11_link" reason="Never" />
-    <disable_collisions link1="LFinger13_link" link2="RFinger12_link" reason="Never" />
-    <disable_collisions link1="LFinger13_link" link2="RFinger13_link" reason="Never" />
-    <disable_collisions link1="LFinger13_link" link2="RFinger21_link" reason="Never" />
-    <disable_collisions link1="LFinger13_link" link2="RFinger22_link" reason="Never" />
-    <disable_collisions link1="LFinger13_link" link2="RFinger23_link" reason="Never" />
-    <disable_collisions link1="LFinger13_link" link2="RFinger31_link" reason="Never" />
-    <disable_collisions link1="LFinger13_link" link2="RFinger32_link" reason="Never" />
-    <disable_collisions link1="LFinger13_link" link2="RFinger33_link" reason="Never" />
-    <disable_collisions link1="LFinger13_link" link2="RFinger41_link" reason="Never" />
-    <disable_collisions link1="LFinger13_link" link2="RFinger42_link" reason="Never" />
-    <disable_collisions link1="LFinger13_link" link2="RFinger43_link" reason="Never" />
-    <disable_collisions link1="LFinger13_link" link2="RForeArm" reason="Never" />
-    <disable_collisions link1="LFinger13_link" link2="RShoulder" reason="Never" />
-    <disable_collisions link1="LFinger13_link" link2="RThumb1_link" reason="Never" />
-    <disable_collisions link1="LFinger13_link" link2="RThumb2_link" reason="Never" />
-    <disable_collisions link1="LFinger13_link" link2="Tibia" reason="Never" />
-    <disable_collisions link1="LFinger13_link" link2="WheelB_link" reason="Never" />
-    <disable_collisions link1="LFinger13_link" link2="WheelFL_link" reason="Never" />
-    <disable_collisions link1="LFinger13_link" link2="WheelFR_link" reason="Never" />
-    <disable_collisions link1="LFinger13_link" link2="l_wrist" reason="Never" />
-    <disable_collisions link1="LFinger13_link" link2="r_wrist" reason="Never" />
-    <disable_collisions link1="LFinger21_link" link2="LFinger22_link" reason="Adjacent" />
-    <disable_collisions link1="LFinger21_link" link2="LFinger23_link" reason="Never" />
-    <disable_collisions link1="LFinger21_link" link2="LFinger31_link" reason="Never" />
-    <disable_collisions link1="LFinger21_link" link2="LFinger32_link" reason="Never" />
-    <disable_collisions link1="LFinger21_link" link2="LFinger33_link" reason="Never" />
-    <disable_collisions link1="LFinger21_link" link2="LFinger41_link" reason="Never" />
-    <disable_collisions link1="LFinger21_link" link2="LFinger42_link" reason="Never" />
-    <disable_collisions link1="LFinger21_link" link2="LFinger43_link" reason="Never" />
-    <disable_collisions link1="LFinger21_link" link2="LForeArm" reason="Never" />
-    <disable_collisions link1="LFinger21_link" link2="LShoulder" reason="Never" />
-    <disable_collisions link1="LFinger21_link" link2="LThumb1_link" reason="Never" />
-    <disable_collisions link1="LFinger21_link" link2="LThumb2_link" reason="Never" />
-    <disable_collisions link1="LFinger21_link" link2="Neck" reason="Never" />
-    <disable_collisions link1="LFinger21_link" link2="RBicep" reason="Never" />
-    <disable_collisions link1="LFinger21_link" link2="RElbow" reason="Never" />
-    <disable_collisions link1="LFinger21_link" link2="RFinger11_link" reason="Never" />
-    <disable_collisions link1="LFinger21_link" link2="RFinger12_link" reason="Never" />
-    <disable_collisions link1="LFinger21_link" link2="RFinger13_link" reason="Never" />
-    <disable_collisions link1="LFinger21_link" link2="RFinger21_link" reason="Never" />
-    <disable_collisions link1="LFinger21_link" link2="RFinger22_link" reason="Never" />
-    <disable_collisions link1="LFinger21_link" link2="RFinger23_link" reason="Never" />
-    <disable_collisions link1="LFinger21_link" link2="RFinger31_link" reason="Never" />
-    <disable_collisions link1="LFinger21_link" link2="RFinger32_link" reason="Never" />
-    <disable_collisions link1="LFinger21_link" link2="RFinger33_link" reason="Never" />
-    <disable_collisions link1="LFinger21_link" link2="RFinger41_link" reason="Never" />
-    <disable_collisions link1="LFinger21_link" link2="RFinger42_link" reason="Never" />
-    <disable_collisions link1="LFinger21_link" link2="RFinger43_link" reason="Never" />
-    <disable_collisions link1="LFinger21_link" link2="RForeArm" reason="Never" />
-    <disable_collisions link1="LFinger21_link" link2="RShoulder" reason="Never" />
-    <disable_collisions link1="LFinger21_link" link2="RThumb1_link" reason="Never" />
-    <disable_collisions link1="LFinger21_link" link2="RThumb2_link" reason="Never" />
-    <disable_collisions link1="LFinger21_link" link2="WheelB_link" reason="Never" />
-    <disable_collisions link1="LFinger21_link" link2="WheelFL_link" reason="Never" />
-    <disable_collisions link1="LFinger21_link" link2="WheelFR_link" reason="Never" />
-    <disable_collisions link1="LFinger21_link" link2="l_wrist" reason="Adjacent" />
-    <disable_collisions link1="LFinger21_link" link2="r_wrist" reason="Never" />
-    <disable_collisions link1="LFinger22_link" link2="LFinger23_link" reason="Adjacent" />
-    <disable_collisions link1="LFinger22_link" link2="LFinger31_link" reason="Never" />
-    <disable_collisions link1="LFinger22_link" link2="LFinger32_link" reason="Never" />
-    <disable_collisions link1="LFinger22_link" link2="LFinger33_link" reason="Never" />
-    <disable_collisions link1="LFinger22_link" link2="LFinger41_link" reason="Never" />
-    <disable_collisions link1="LFinger22_link" link2="LFinger42_link" reason="Never" />
-    <disable_collisions link1="LFinger22_link" link2="LFinger43_link" reason="Never" />
-    <disable_collisions link1="LFinger22_link" link2="LForeArm" reason="Never" />
-    <disable_collisions link1="LFinger22_link" link2="LShoulder" reason="Never" />
-    <disable_collisions link1="LFinger22_link" link2="LThumb1_link" reason="Never" />
-    <disable_collisions link1="LFinger22_link" link2="LThumb2_link" reason="Never" />
-    <disable_collisions link1="LFinger22_link" link2="Neck" reason="Never" />
-    <disable_collisions link1="LFinger22_link" link2="RBicep" reason="Never" />
-    <disable_collisions link1="LFinger22_link" link2="RElbow" reason="Never" />
-    <disable_collisions link1="LFinger22_link" link2="RFinger11_link" reason="Never" />
-    <disable_collisions link1="LFinger22_link" link2="RFinger12_link" reason="Never" />
-    <disable_collisions link1="LFinger22_link" link2="RFinger13_link" reason="Never" />
-    <disable_collisions link1="LFinger22_link" link2="RFinger21_link" reason="Never" />
-    <disable_collisions link1="LFinger22_link" link2="RFinger22_link" reason="Never" />
-    <disable_collisions link1="LFinger22_link" link2="RFinger23_link" reason="Never" />
-    <disable_collisions link1="LFinger22_link" link2="RFinger31_link" reason="Never" />
-    <disable_collisions link1="LFinger22_link" link2="RFinger32_link" reason="Never" />
-    <disable_collisions link1="LFinger22_link" link2="RFinger33_link" reason="Never" />
-    <disable_collisions link1="LFinger22_link" link2="RFinger41_link" reason="Never" />
-    <disable_collisions link1="LFinger22_link" link2="RFinger42_link" reason="Never" />
-    <disable_collisions link1="LFinger22_link" link2="RFinger43_link" reason="Never" />
-    <disable_collisions link1="LFinger22_link" link2="RForeArm" reason="Never" />
-    <disable_collisions link1="LFinger22_link" link2="RShoulder" reason="Never" />
-    <disable_collisions link1="LFinger22_link" link2="RThumb1_link" reason="Never" />
-    <disable_collisions link1="LFinger22_link" link2="RThumb2_link" reason="Never" />
-    <disable_collisions link1="LFinger22_link" link2="WheelB_link" reason="Never" />
-    <disable_collisions link1="LFinger22_link" link2="WheelFL_link" reason="Never" />
-    <disable_collisions link1="LFinger22_link" link2="WheelFR_link" reason="Never" />
-    <disable_collisions link1="LFinger22_link" link2="l_wrist" reason="Never" />
-    <disable_collisions link1="LFinger22_link" link2="r_wrist" reason="Never" />
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