Commit message: fix joint limits

File: pepper_robot_description/urdf/pepper_head.xacro (robot description, xacro)
@@ -24,5 +24,5 @@
 		<origin rpy="0 0 0" xyz="0 0 0"/>
 		<axis xyz="0 1.0 0"/>
-		<limit effort="2.666" lower="-0.706858" upper="0.637045" velocity="9.22756"/>
+		<limit effort="2.666" lower="-0.706858" upper="0.4451" velocity="9.22756"/>
 	</joint>
 	<link name="Head">

File: pepper_robot_description/urdf/pepper_robot.urdf (robot description, URDF)
Before this commit: robot JulietteY20MP, 83 links, 82 joints
Joints:
- joint HeadPitch: limit lower=-0.706858 upper=0.637045 effort=2.666 velocity=9.22756 -> lower=-0.706858 upper=0.4451 effort=2.666 velocity=9.22756
