Commit message: fix joint limits

File: pepper_robot_description/urdf/pepper_arms.xacro (robot description, xacro)
@@ -84,5 +84,5 @@
 		<origin rpy="0 0 0" xyz="0.025 0 0"/>
 		<axis xyz="1.0 0 0"/>
-		<limit effort="0.144" lower="0.02" upper="0.98" velocity="12.56"/>
+		<limit effort="0.144" lower="0.0" upper="0.0174533" velocity="12.56"/>
 	</joint>
 	<link name="l_gripper">
@@ -172,5 +172,5 @@
 		<origin rpy="0 0 0" xyz="0.025 0 0"/>
 		<axis xyz="1.0 0 0"/>
-		<limit effort="0.144" lower="0.02" upper="0.98" velocity="12.56"/>
+		<limit effort="0.144" lower="0.0" upper="0.0174533" velocity="12.56"/>
 	</joint>
 	<link name="r_gripper">

File: pepper_robot_description/urdf/pepper_robot.urdf (robot description, URDF)
Before this commit: robot JulietteY20MP, 83 links, 82 joints
Joints:
- joint LHand: limit lower=0.02 upper=0.98 effort=0.144 velocity=12.56 -> lower=0.0 upper=0.0174533 effort=0.144 velocity=12.56
- joint RHand: limit lower=0.02 upper=0.98 effort=0.144 velocity=12.56 -> lower=0.0 upper=0.0174533 effort=0.144 velocity=12.56

Commit message: fix joint limits

File: pepper_robot_description/urdf/pepper_arms.xacro (robot description, xacro)
@@ -84,5 +84,5 @@
 		<origin rpy="0 0 0" xyz="0.025 0 0"/>
 		<axis xyz="1.0 0 0"/>
-		<limit effort="0.144" lower="0.0" upper="0.0174533" velocity="12.56"/>
+		<limit effort="0.144" lower="0.0174533" upper="0.0349066" velocity="12.56"/>
 	</joint>
 	<link name="l_gripper">
@@ -172,5 +172,5 @@
 		<origin rpy="0 0 0" xyz="0.025 0 0"/>
 		<axis xyz="1.0 0 0"/>
-		<limit effort="0.144" lower="0.0" upper="0.0174533" velocity="12.56"/>
+		<limit effort="0.144" lower="0.0174533" upper="0.0349066" velocity="12.56"/>
 	</joint>
 	<link name="r_gripper">

File: pepper_robot_description/urdf/pepper_robot.urdf (robot description, URDF)
Before this commit: robot JulietteY20MP, 83 links, 82 joints
Joints:
- joint LHand: limit lower=0.0 upper=0.0174533 effort=0.144 velocity=12.56 -> lower=0.0174533 upper=0.0349066 effort=0.144 velocity=12.56
- joint RHand: limit lower=0.0 upper=0.0174533 effort=0.144 velocity=12.56 -> lower=0.0174533 upper=0.0349066 effort=0.144 velocity=12.56

Commit message: fix joint limits

File: pepper_robot_description/urdf/pepper_arms.xacro (robot description, xacro)
@@ -84,5 +84,5 @@
 		<origin rpy="0 0 0" xyz="0.025 0 0"/>
 		<axis xyz="1.0 0 0"/>
-		<limit effort="0.144" lower="0.0174533" upper="0.0349066" velocity="12.56"/>
+		<limit effort="0.144" lower="0.0" upper="0.0349066" velocity="12.56"/>
 	</joint>
 	<link name="l_gripper">
@@ -172,5 +172,5 @@
 		<origin rpy="0 0 0" xyz="0.025 0 0"/>
 		<axis xyz="1.0 0 0"/>
-		<limit effort="0.144" lower="0.0174533" upper="0.0349066" velocity="12.56"/>
+		<limit effort="0.144" lower="0.0" upper="0.0349066" velocity="12.56"/>
 	</joint>
 	<link name="r_gripper">

File: pepper_robot_description/urdf/pepper_robot.urdf (robot description, URDF)
Before this commit: robot JulietteY20MP, 83 links, 82 joints
Joints:
- joint LHand: limit lower=0.0174533 upper=0.0349066 effort=0.144 velocity=12.56 -> lower=0.0 upper=0.0349066 effort=0.144 velocity=12.56
- joint RHand: limit lower=0.0174533 upper=0.0349066 effort=0.144 velocity=12.56 -> lower=0.0 upper=0.0349066 effort=0.144 velocity=12.56

Commit message: fix joint limits

File: pepper_robot_description/urdf/pepper_arms.xacro (robot description, xacro)
@@ -84,5 +84,5 @@
 		<origin rpy="0 0 0" xyz="0.025 0 0"/>
 		<axis xyz="1.0 0 0"/>
-		<limit effort="0.144" lower="0.0" upper="0.0349066" velocity="12.56"/>
+		<limit effort="0.144" lower="0.02" upper="0.98" velocity="12.56"/>
 	</joint>
 	<link name="l_gripper">
@@ -172,5 +172,5 @@
 		<origin rpy="0 0 0" xyz="0.025 0 0"/>
 		<axis xyz="1.0 0 0"/>
-		<limit effort="0.144" lower="0.0" upper="0.0349066" velocity="12.56"/>
+		<limit effort="0.144" lower="0.02" upper="0.98" velocity="12.56"/>
 	</joint>
 	<link name="r_gripper">

File: pepper_robot_description/urdf/pepper_robot.urdf (robot description, URDF)
Before this commit: robot JulietteY20MP, 83 links, 82 joints
Joints:
- joint LHand: limit lower=0.0 upper=0.0349066 effort=0.144 velocity=12.56 -> lower=0.02 upper=0.98 effort=0.144 velocity=12.56
- joint RHand: limit lower=0.0 upper=0.0349066 effort=0.144 velocity=12.56 -> lower=0.02 upper=0.98 effort=0.144 velocity=12.56
