Commit message: path to meshes

File: pepper_robot_description/urdf/pepper.urdf (robot description, URDF)
Before this commit: robot pepper, 65 links, 64 joints
Links:
- link Head: geometry collision mesh filename=/root/ws/src/pepper_ign_moveit2/pepper_robot_description/pe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 scale=0.1 0.1 0.1; visual mesh filename=/root/ws/src/pepper_ign_moveit2/pepper_robot_description/pe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 scale=0.1 0.1 0.1
- link Hip: geometry collision mesh filename=/root/ws/src/pepper_ign_moveit2/pepper_robot_description/pe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 scale=0.1 0.1 0.1; visual mesh filename=/root/ws/src/pepper_ign_moveit2/pepper_robot_description/pe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 scale=0.1 0.1 0.1
- link LBicep: geometry collision mesh filename=/root/ws/src/pepper_ign_moveit2/pepper_robot_description/pe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 scale=0.1 0.1 0.1; visual mesh filename=/root/ws/src/pepper_ign_moveit2/pepper_robot_description/pe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 scale=0.1 0.1 0.1
- link LElbow: geometry collision mesh filename=/root/ws/src/pepper_ign_moveit2/pepper_robot_description/pe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 scale=0.1 0.1 0.1; visual mesh filename=/root/ws/src/pepper_ign_moveit2/pepper_robot_description/pe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 scale=0.1 0.1 0.1
- link LFinger11_link: geometry collision mesh filename=/root/ws/src/pepper_ign_moveit2/pepper_robot_description/pe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 scale=0.1 0.1 0.1; visual mesh filename=/root/ws/src/pepper_ign_moveit2/pepper_robot_description/pe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 scale=0.1 0.1 0.1
- link LFinger12_link: geometry collision mesh filename=/root/ws/src/pepper_ign_moveit2/pepper_robot_description/pe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 scale=0.1 0.1 0.1; visual mesh filename=/root/ws/src/pepper_ign_moveit2/pepper_robot_description/pe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 scale=0.1 0.1 0.1
- link LFinger13_link: geometry collision mesh filename=/root/ws/src/pepper_ign_moveit2/pepper_robot_description/pe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 scale=0.1 0.1 0.1; visual mesh filename=/root/ws/src/pepper_ign_moveit2/pepper_robot_description/pe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 scale=0.1 0.1 0.1
- link LFinger21_link: geometry collision mesh filename=/root/ws/src/pepper_ign_moveit2/pepper_robot_description/pe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 scale=0.1 0.1 0.1; visual mesh filename=/root/ws/src/pepper_ign_moveit2/pepper_robot_description/pe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 scale=0.1 0.1 0.1
- link LFinger22_link: geometry collision mesh filename=/root/ws/src/pepper_ign_moveit2/pepper_robot_description/pe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 scale=0.1 0.1 0.1; visual mesh filename=/root/ws/src/pepper_ign_moveit2/pepper_robot_description/pe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 scale=0.1 0.1 0.1
- link LFinger23_link: geometry collision mesh filename=/root/ws/src/pepper_ign_moveit2/pepper_robot_description/pe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 scale=0.1 0.1 0.1; visual mesh filename=/root/ws/src/pepper_ign_moveit2/pepper_robot_description/pe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 scale=0.1 0.1 0.1
- link LFinger31_link: geometry collision mesh filename=/root/ws/src/pepper_ign_moveit2/pepper_robot_description/pe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 scale=0.1 0.1 0.1; visual mesh filename=/root/ws/src/pepper_ign_moveit2/pepper_robot_description/pe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 scale=0.1 0.1 0.1
- link LFinger32_link: geometry collision mesh filename=/root/ws/src/pepper_ign_moveit2/pepper_robot_description/pe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 scale=0.1 0.1 0.1; visual mesh filename=/root/ws/src/pepper_ign_moveit2/pepper_robot_description/pe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 scale=0.1 0.1 0.1
- link LFinger33_link: geometry collision mesh filename=/root/ws/src/pepper_ign_moveit2/pepper_robot_description/pe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 scale=0.1 0.1 0.1; visual mesh filename=/root/ws/src/pepper_ign_moveit2/pepper_robot_description/pe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 scale=0.1 0.1 0.1
- link LFinger41_link: geometry collision mesh filename=/root/ws/src/pepper_ign_moveit2/pepper_robot_description/pe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 scale=0.1 0.1 0.1; visual mesh filename=/root/ws/src/pepper_ign_moveit2/pepper_robot_description/pe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 scale=0.1 0.1 0.1
- link LFinger42_link: geometry collision mesh filename=/root/ws/src/pepper_ign_moveit2/pepper_robot_description/pe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 scale=0.1 0.1 0.1; visual mesh filename=/root/ws/src/pepper_ign_moveit2/pepper_robot_description/pe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 scale=0.1 0.1 0.1
- link LFinger43_link: geometry collision mesh filename=/root/ws/src/pepper_ign_moveit2/pepper_robot_description/pe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 scale=0.1 0.1 0.1; visual mesh filename=/root/ws/src/pepper_ign_moveit2/pepper_robot_description/pe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 scale=0.1 0.1 0.1
- link LForeArm: geometry collision mesh filename=/root/ws/src/pepper_ign_moveit2/pepper_robot_description/pe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 scale=0.1 0.1 0.1; visual mesh filename=/root/ws/src/pepper_ign_moveit2/pepper_robot_description/pe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 scale=0.1 0.1 0.1
- link LShoulder: geometry collision mesh filename=/root/ws/src/pepper_ign_moveit2/pepper_robot_description/pe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 scale=0.1 0.1 0.1; visual mesh filename=/root/ws/src/pepper_ign_moveit2/pepper_robot_description/pe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 scale=0.1 0.1 0.1
- link LThumb1_link: geometry collision mesh filename=/root/ws/src/pepper_ign_moveit2/pepper_robot_description/pe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 scale=0.1 0.1 0.1; visual mesh filename=/root/ws/src/pepper_ign_moveit2/pepper_robot_description/pe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 scale=0.1 0.1 0.1
- link LThumb2_link: geometry collision mesh filename=/root/ws/src/pepper_ign_moveit2/pepper_robot_description/pe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 scale=0.1 0.1 0.1; visual mesh filename=/root/ws/src/pepper_ign_moveit2/pepper_robot_description/pe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 scale=0.1 0.1 0.1
- link Neck: geometry collision mesh filename=/root/ws/src/pepper_ign_moveit2/pepper_robot_description/pe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 scale=0.1 0.1 0.1; visual mesh filename=/root/ws/src/pepper_ign_moveit2/pepper_robot_description/pe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 scale=0.1 0.1 0.1
- link Pelvis: geometry collision mesh filename=/root/ws/src/pepper_ign_moveit2/pepper_robot_description/pe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 scale=0.1 0.1 0.1; visual mesh filename=/root/ws/src/pepper_ign_moveit2/pepper_robot_description/pe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 scale=0.1 0.1 0.1
- link RBicep: geometry collision mesh filename=/root/ws/src/pepper_ign_moveit2/pepper_robot_description/pe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 scale=0.1 0.1 0.1; visual mesh filename=/root/ws/src/pepper_ign_moveit2/pepper_robot_description/pe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 scale=0.1 0.1 0.1
- link RElbow: geometry collision mesh filename=/root/ws/src/pepper_ign_moveit2/pepper_robot_description/pe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 scale=0.1 0.1 0.1; visual mesh filename=/root/ws/src/pepper_ign_moveit2/pepper_robot_description/pe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 scale=0.1 0.1 0.1
- link RFinger11_link: geometry collision mesh filename=/root/ws/src/pepper_ign_moveit2/pepper_robot_description/pe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 scale=0.1 0.1 0.1; visual mesh filename=/root/ws/src/pepper_ign_moveit2/pepper_robot_description/pe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 scale=0.1 0.1 0.1
- link RFinger12_link: geometry collision mesh filename=/root/ws/src/pepper_ign_moveit2/pepper_robot_description/pe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 scale=0.1 0.1 0.1; visual mesh filename=/root/ws/src/pepper_ign_moveit2/pepper_robot_description/pe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 scale=0.1 0.1 0.1
- link RFinger13_link: geometry collision mesh filename=/root/ws/src/pepper_ign_moveit2/pepper_robot_description/pe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 scale=0.1 0.1 0.1; visual mesh filename=/root/ws/src/pepper_ign_moveit2/pepper_robot_description/pe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 scale=0.1 0.1 0.1
- link RFinger21_link: geometry collision mesh filename=/root/ws/src/pepper_ign_moveit2/pepper_robot_description/pe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 scale=0.1 0.1 0.1; visual mesh filename=/root/ws/src/pepper_ign_moveit2/pepper_robot_description/pe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 scale=0.1 0.1 0.1
- link RFinger22_link: geometry collision mesh filename=/root/ws/src/pepper_ign_moveit2/pepper_robot_description/pe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 scale=0.1 0.1 0.1; visual mesh filename=/root/ws/src/pepper_ign_moveit2/pepper_robot_description/pe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 scale=0.1 0.1 0.1
- link RFinger23_link: geometry collision mesh filename=/root/ws/src/pepper_ign_moveit2/pepper_robot_description/pe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 scale=0.1 0.1 0.1; visual mesh filename=/root/ws/src/pepper_ign_moveit2/pepper_robot_description/pe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 scale=0.1 0.1 0.1
- link RFinger31_link: geometry collision mesh filename=/root/ws/src/pepper_ign_moveit2/pepper_robot_description/pe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 scale=0.1 0.1 0.1; visual mesh filename=/root/ws/src/pepper_ign_moveit2/pepper_robot_description/pe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 scale=0.1 0.1 0.1
- link RFinger32_link: geometry collision mesh filename=/root/ws/src/pepper_ign_moveit2/pepper_robot_description/pe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 scale=0.1 0.1 0.1; visual mesh filename=/root/ws/src/pepper_ign_moveit2/pepper_robot_description/pe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 scale=0.1 0.1 0.1
- link RFinger33_link: geometry collision mesh filename=/root/ws/src/pepper_ign_moveit2/pepper_robot_description/pe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 scale=0.1 0.1 0.1; visual mesh filename=/root/ws/src/pepper_ign_moveit2/pepper_robot_description/pe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 scale=0.1 0.1 0.1
- link RFinger41_link: geometry collision mesh filename=/root/ws/src/pepper_ign_moveit2/pepper_robot_description/pe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 scale=0.1 0.1 0.1; visual mesh filename=/root/ws/src/pepper_ign_moveit2/pepper_robot_description/pe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 scale=0.1 0.1 0.1
- link RFinger42_link: geometry collision mesh filename=/root/ws/src/pepper_ign_moveit2/pepper_robot_description/pe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 scale=0.1 0.1 0.1; visual mesh filename=/root/ws/src/pepper_ign_moveit2/pepper_robot_description/pe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 scale=0.1 0.1 0.1
- link RFinger43_link: geometry collision mesh filename=/root/ws/src/pepper_ign_moveit2/pepper_robot_description/pe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 scale=0.1 0.1 0.1; visual mesh filename=/root/ws/src/pepper_ign_moveit2/pepper_robot_description/pe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 scale=0.1 0.1 0.1
- link RForeArm: geometry collision mesh filename=/root/ws/src/pepper_ign_moveit2/pepper_robot_description/pe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 scale=0.1 0.1 0.1; visual mesh filename=/root/ws/src/pepper_ign_moveit2/pepper_robot_description/pe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 scale=0.1 0.1 0.1
- link RShoulder: geometry collision mesh filename=/root/ws/src/pepper_ign_moveit2/pepper_robot_description/pe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 scale=0.1 0.1 0.1; visual mesh filename=/root/ws/src/pepper_ign_moveit2/pepper_robot_description/pe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 scale=0.1 0.1 0.1
- link RThumb1_link: geometry collision mesh filename=/root/ws/src/pepper_ign_moveit2/pepper_robot_description/pe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 scale=0.1 0.1 0.1; visual mesh filename=/root/ws/src/pepper_ign_moveit2/pepper_robot_description/pe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 scale=0.1 0.1 0.1
- link RThumb2_link: geometry collision mesh filename=/root/ws/src/pepper_ign_moveit2/pepper_robot_description/pe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 scale=0.1 0.1 0.1; visual mesh filename=/root/ws/src/pepper_ign_moveit2/pepper_robot_description/pe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 scale=0.1 0.1 0.1
- link RealSense_screw_frame: geometry visual mesh filename=/root/ws/src/pepper_ign_moveit2/pepper_robot_description/pe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
- link Tibia: geometry collision mesh filename=/root/ws/src/pepper_ign_moveit2/pepper_robot_description/pe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 scale=0.1 0.1 0.1; visual mesh filename=/root/ws/src/pepper_ign_moveit2/pepper_robot_description/pe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 scale=0.1 0.1 0.1
- link WheelB_link: geometry collision mesh filename=/root/ws/src/pepper_ign_moveit2/pepper_robot_description/pe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 scale=0.1 0.1 0.1; visual mesh filename=/root/ws/src/pepper_ign_moveit2/pepper_robot_description/pe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 scale=0.1 0.1 0.1
- link WheelFL_link: geometry collision mesh filename=/root/ws/src/pepper_ign_moveit2/pepper_robot_description/pe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 scale=0.1 0.1 0.1; visual mesh filename=/root/ws/src/pepper_ign_moveit2/pepper_robot_description/pe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 scale=0.1 0.1 0.1
- link WheelFR_link: geometry collision mesh filename=/root/ws/src/pepper_ign_moveit2/pepper_robot_description/pe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 scale=0.1 0.1 0.1; visual mesh filename=/root/ws/src/pepper_ign_moveit2/pepper_robot_description/pe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 scale=0.1 0.1 0.1
- link camera_base: geometry visual mesh filename=/root/ws/src/pepper_ign_moveit2/pepper_robot_description/pe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
- link camera_body: geometry visual mesh filename=/root/ws/src/pepper_ign_moveit2/pepper_robot_description/pe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
- link camera_visor: geometry visual mesh filename=/root/ws/src/pepper_ign_moveit2/pepper_robot_description/pe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
- link l_wrist: geometry collision mesh filename=/root/ws/src/pepper_ign_moveit2/pepper_robot_description/pe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 scale=0.1 0.1 0.1; visual mesh filename=/root/ws/src/pepper_ign_moveit2/pepper_robot_description/pe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 scale=0.1 0.1 0.1
- link r_wrist: geometry collision mesh filename=/root/ws/src/pepper_ign_moveit2/pepper_robot_description/pe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 scale=0.1 0.1 0.1; visual mesh filename=/root/ws/src/pepper_ign_moveit2/pepper_robot_description/pe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 scale=0.1 0.1 0.1
- link t265: geometry visual mesh filename=/root/ws/src/pepper_ign_moveit2/pepper_robot_description/pe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
- link torso: geometry collision mesh filename=/root/ws/src/pepper_ign_moveit2/pepper_robot_description/pe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 scale=0.1 0.1 0.1; visual mesh filename=/root/ws/src/pepper_ign_moveit2/pepper_robot_description/pe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 scale=0.1 0.1 0.1
