Commit message: fix robot name

File: pepper_robot_description/urdf/pepper_fingers.xacro (robot description, xacro)
@@ -3,5 +3,5 @@
  ****** File automatically generated by generate_urdf.py script ******
  *********************************************************************-->
-<robot name="pepper" xmlns:xacro="http://www.ros.org/wiki/xacro">
+<robot name="pepper_robot" xmlns:xacro="http://www.ros.org/wiki/xacro">
 	<link name="RFinger41_link">
 		<inertial>

File: pepper_robot_description/urdf/pepper_robot.urdf (robot description, URDF)
Before this commit: robot JulietteY20MP, 83 links, 82 joints
Links:
- link Head: geometry collision mesh filename=package://pepper_robot_meshes/meshes/1.0/HeadPitch_0.10.stl scale=0.1 0.1 0.1; visual mesh filename=package://pepper_robot_meshes/meshes/1.0/HeadPitch.dae scale=0.1 0.1 0.1
- link Hip: geometry collision mesh filename=package://pepper_robot_meshes/meshes/1.0/HipRoll_0.10.stl scale=0.1 0.1 0.1; visual mesh filename=package://pepper_robot_meshes/meshes/1.0/HipRoll.dae scale=0.1 0.1 0.1
- link LBicep: geometry collision mesh filename=package://pepper_robot_meshes/meshes/1.0/LShoulderRoll_0.10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 scale=0.1 0.1 0.1; visual mesh filename=package://pepper_robot_meshes/meshes/1.0/LShoulderRoll.dae scale=0.1 0.1 0.1
- link LElbow: geometry collision mesh filename=package://pepper_robot_meshes/meshes/1.0/LElbowYaw_0.10.stl scale=0.1 0.1 0.1; visual mesh filename=package://pepper_robot_meshes/meshes/1.0/LElbowYaw.dae scale=0.1 0.1 0.1
- link LFinger11_link: geometry collision mesh filename=package://pepper_robot_meshes/meshes/1.0/LFinger11_0.10.stl scale=0.1 0.1 0.1; visual mesh filename=package://pepper_robot_meshes/meshes/1.0/LFinger11.dae scale=0.1 0.1 0.1
- link LFinger12_link: geometry collision mesh filename=package://pepper_robot_meshes/meshes/1.0/LFinger12_0.10.stl scale=0.1 0.1 0.1; visual mesh filename=package://pepper_robot_meshes/meshes/1.0/LFinger12.dae scale=0.1 0.1 0.1
- link LFinger13_link: geometry collision mesh filename=package://pepper_robot_meshes/meshes/1.0/LFinger13_0.10.stl scale=0.1 0.1 0.1; visual mesh filename=package://pepper_robot_meshes/meshes/1.0/LFinger13.dae scale=0.1 0.1 0.1
- link LFinger21_link: geometry collision mesh filename=package://pepper_robot_meshes/meshes/1.0/LFinger21_0.10.stl scale=0.1 0.1 0.1; visual mesh filename=package://pepper_robot_meshes/meshes/1.0/LFinger21.dae scale=0.1 0.1 0.1
- link LFinger22_link: geometry collision mesh filename=package://pepper_robot_meshes/meshes/1.0/LFinger22_0.10.stl scale=0.1 0.1 0.1; visual mesh filename=package://pepper_robot_meshes/meshes/1.0/LFinger22.dae scale=0.1 0.1 0.1
- link LFinger23_link: geometry collision mesh filename=package://pepper_robot_meshes/meshes/1.0/LFinger23_0.10.stl scale=0.1 0.1 0.1; visual mesh filename=package://pepper_robot_meshes/meshes/1.0/LFinger23.dae scale=0.1 0.1 0.1
- link LFinger31_link: geometry collision mesh filename=package://pepper_robot_meshes/meshes/1.0/LFinger31_0.10.stl scale=0.1 0.1 0.1; visual mesh filename=package://pepper_robot_meshes/meshes/1.0/LFinger31.dae scale=0.1 0.1 0.1
- link LFinger32_link: geometry collision mesh filename=package://pepper_robot_meshes/meshes/1.0/LFinger32_0.10.stl scale=0.1 0.1 0.1; visual mesh filename=package://pepper_robot_meshes/meshes/1.0/LFinger32.dae scale=0.1 0.1 0.1
- link LFinger33_link: geometry collision mesh filename=package://pepper_robot_meshes/meshes/1.0/LFinger33_0.10.stl scale=0.1 0.1 0.1; visual mesh filename=package://pepper_robot_meshes/meshes/1.0/LFinger33.dae scale=0.1 0.1 0.1
- link LFinger41_link: geometry collision mesh filename=package://pepper_robot_meshes/meshes/1.0/LFinger41_0.10.stl scale=0.1 0.1 0.1; visual mesh filename=package://pepper_robot_meshes/meshes/1.0/LFinger41.dae scale=0.1 0.1 0.1
- link LFinger42_link: geometry collision mesh filename=package://pepper_robot_meshes/meshes/1.0/LFinger42_0.10.stl scale=0.1 0.1 0.1; visual mesh filename=package://pepper_robot_meshes/meshes/1.0/LFinger42.dae scale=0.1 0.1 0.1
- link LFinger43_link: geometry collision mesh filename=package://pepper_robot_meshes/meshes/1.0/LFinger43_0.10.stl scale=0.1 0.1 0.1; visual mesh filename=package://pepper_robot_meshes/meshes/1.0/LFinger43.dae scale=0.1 0.1 0.1
- link LForeArm: geometry collision mesh filename=package://pepper_robot_meshes/meshes/1.0/LElbowRoll_0.10.stl scale=0.1 0.1 0.1; visual mesh filename=package://pepper_robot_meshes/meshes/1.0/LElbowRoll.dae scale=0.1 0.1 0.1
- link LShoulder: geometry collision mesh filename=package://pepper_robot_meshes/meshes/1.0/LShoulderPitch_0.1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 scale=0.1 0.1 0.1; visual mesh filename=package://pepper_robot_meshes/meshes/1.0/LShoulderPitch.dae scale=0.1 0.1 0.1
- link LThumb1_link: geometry collision mesh filename=package://pepper_robot_meshes/meshes/1.0/LThumb1_0.10.stl scale=0.1 0.1 0.1; visual mesh filename=package://pepper_robot_meshes/meshes/1.0/LThumb1.dae scale=0.1 0.1 0.1
- link LThumb2_link: geometry collision mesh filename=package://pepper_robot_meshes/meshes/1.0/LThumb2_0.10.stl scale=0.1 0.1 0.1; visual mesh filename=package://pepper_robot_meshes/meshes/1.0/LThumb2.dae scale=0.1 0.1 0.1
- link Neck: geometry collision mesh filename=package://pepper_robot_meshes/meshes/1.0/HeadYaw_0.10.stl scale=0.1 0.1 0.1; visual mesh filename=package://pepper_robot_meshes/meshes/1.0/HeadYaw.dae scale=0.1 0.1 0.1
- link Pelvis: geometry collision mesh filename=package://pepper_robot_meshes/meshes/1.0/HipPitch_0.10.stl scale=0.1 0.1 0.1; visual mesh filename=package://pepper_robot_meshes/meshes/1.0/HipPitch.dae scale=0.1 0.1 0.1
- link RBicep: geometry collision mesh filename=package://pepper_robot_meshes/meshes/1.0/RShoulderRoll_0.10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 scale=0.1 0.1 0.1; visual mesh filename=package://pepper_robot_meshes/meshes/1.0/RShoulderRoll.dae scale=0.1 0.1 0.1
- link RElbow: geometry collision mesh filename=package://pepper_robot_meshes/meshes/1.0/RElbowYaw_0.10.stl scale=0.1 0.1 0.1; visual mesh filename=package://pepper_robot_meshes/meshes/1.0/RElbowYaw.dae scale=0.1 0.1 0.1
- link RFinger11_link: geometry collision mesh filename=package://pepper_robot_meshes/meshes/1.0/RFinger11_0.10.stl scale=0.1 0.1 0.1; visual mesh filename=package://pepper_robot_meshes/meshes/1.0/RFinger11.dae scale=0.1 0.1 0.1
- link RFinger12_link: geometry collision mesh filename=package://pepper_robot_meshes/meshes/1.0/RFinger12_0.10.stl scale=0.1 0.1 0.1; visual mesh filename=package://pepper_robot_meshes/meshes/1.0/RFinger12.dae scale=0.1 0.1 0.1
- link RFinger13_link: geometry collision mesh filename=package://pepper_robot_meshes/meshes/1.0/RFinger13_0.10.stl scale=0.1 0.1 0.1; visual mesh filename=package://pepper_robot_meshes/meshes/1.0/RFinger13.dae scale=0.1 0.1 0.1
- link RFinger21_link: geometry collision mesh filename=package://pepper_robot_meshes/meshes/1.0/RFinger21_0.10.stl scale=0.1 0.1 0.1; visual mesh filename=package://pepper_robot_meshes/meshes/1.0/RFinger21.dae scale=0.1 0.1 0.1
- link RFinger22_link: geometry collision mesh filename=package://pepper_robot_meshes/meshes/1.0/RFinger22_0.10.stl scale=0.1 0.1 0.1; visual mesh filename=package://pepper_robot_meshes/meshes/1.0/RFinger22.dae scale=0.1 0.1 0.1
- link RFinger23_link: geometry collision mesh filename=package://pepper_robot_meshes/meshes/1.0/RFinger23_0.10.stl scale=0.1 0.1 0.1; visual mesh filename=package://pepper_robot_meshes/meshes/1.0/RFinger23.dae scale=0.1 0.1 0.1
- link RFinger31_link: geometry collision mesh filename=package://pepper_robot_meshes/meshes/1.0/RFinger31_0.10.stl scale=0.1 0.1 0.1; visual mesh filename=package://pepper_robot_meshes/meshes/1.0/RFinger31.dae scale=0.1 0.1 0.1
- link RFinger32_link: geometry collision mesh filename=package://pepper_robot_meshes/meshes/1.0/RFinger32_0.10.stl scale=0.1 0.1 0.1; visual mesh filename=package://pepper_robot_meshes/meshes/1.0/RFinger32.dae scale=0.1 0.1 0.1
- link RFinger33_link: geometry collision mesh filename=package://pepper_robot_meshes/meshes/1.0/RFinger33_0.10.stl scale=0.1 0.1 0.1; visual mesh filename=package://pepper_robot_meshes/meshes/1.0/RFinger33.dae scale=0.1 0.1 0.1
- link RFinger41_link: geometry collision mesh filename=package://pepper_robot_meshes/meshes/1.0/RFinger41_0.10.stl scale=0.1 0.1 0.1; visual mesh filename=package://pepper_robot_meshes/meshes/1.0/RFinger41.dae scale=0.1 0.1 0.1
- link RFinger42_link: geometry collision mesh filename=package://pepper_robot_meshes/meshes/1.0/RFinger42_0.10.stl scale=0.1 0.1 0.1; visual mesh filename=package://pepper_robot_meshes/meshes/1.0/RFinger42.dae scale=0.1 0.1 0.1
- link RFinger43_link: geometry collision mesh filename=package://pepper_robot_meshes/meshes/1.0/RFinger43_0.10.stl scale=0.1 0.1 0.1; visual mesh filename=package://pepper_robot_meshes/meshes/1.0/RFinger43.dae scale=0.1 0.1 0.1
- link RForeArm: geometry collision mesh filename=package://pepper_robot_meshes/meshes/1.0/RElbowRoll_0.10.stl scale=0.1 0.1 0.1; visual mesh filename=package://pepper_robot_meshes/meshes/1.0/RElbowRoll.dae scale=0.1 0.1 0.1
- link RShoulder: geometry collision mesh filename=package://pepper_robot_meshes/meshes/1.0/RShoulderPitch_0.1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 scale=0.1 0.1 0.1; visual mesh filename=package://pepper_robot_meshes/meshes/1.0/RShoulderPitch.dae scale=0.1 0.1 0.1
- link RThumb1_link: geometry collision mesh filename=package://pepper_robot_meshes/meshes/1.0/RThumb1_0.10.stl scale=0.1 0.1 0.1; visual mesh filename=package://pepper_robot_meshes/meshes/1.0/RThumb1.dae scale=0.1 0.1 0.1
- link RThumb2_link: geometry collision mesh filename=package://pepper_robot_meshes/meshes/1.0/RThumb2_0.10.stl scale=0.1 0.1 0.1; visual mesh filename=package://pepper_robot_meshes/meshes/1.0/RThumb2.dae scale=0.1 0.1 0.1
- link Tibia: geometry collision mesh filename=package://pepper_robot_meshes/meshes/1.0/KneePitch_0.10.stl scale=0.1 0.1 0.1; visual mesh filename=package://pepper_robot_meshes/meshes/1.0/KneePitch.dae scale=0.1 0.1 0.1
- link WheelB_link: geometry collision mesh filename=package://pepper_robot_meshes/meshes/1.0/WheelB_0.10.stl scale=0.1 0.1 0.1; visual mesh filename=package://pepper_robot_meshes/meshes/1.0/WheelB.dae scale=0.1 0.1 0.1
- link WheelFL_link: geometry collision mesh filename=package://pepper_robot_meshes/meshes/1.0/WheelFL_0.10.stl scale=0.1 0.1 0.1; visual mesh filename=package://pepper_robot_meshes/meshes/1.0/WheelFL.dae scale=0.1 0.1 0.1
- link WheelFR_link: geometry collision mesh filename=package://pepper_robot_meshes/meshes/1.0/WheelFR_0.10.stl scale=0.1 0.1 0.1; visual mesh filename=package://pepper_robot_meshes/meshes/1.0/WheelFR.dae scale=0.1 0.1 0.1
- link l_wrist: geometry collision mesh filename=package://pepper_robot_meshes/meshes/1.0/LWristYaw_0.10.stl scale=0.1 0.1 0.1; visual mesh filename=package://pepper_robot_meshes/meshes/1.0/LWristYaw.dae scale=0.1 0.1 0.1
- link r_wrist: geometry collision mesh filename=package://pepper_robot_meshes/meshes/1.0/RWristYaw_0.10.stl scale=0.1 0.1 0.1; visual mesh filename=package://pepper_robot_meshes/meshes/1.0/RWristYaw.dae scale=0.1 0.1 0.1
- link torso: geometry collision mesh filename=package://pepper_robot_meshes/meshes/1.0/Torso_0.10.stl scale=0.1 0.1 0.1; visual mesh filename=package://pepper_robot_meshes/meshes/1.0/Torso.dae scale=0.1 0.1 0.1

File: pepper_robot_description/urdf/pepper_robot.xacro (robot description, xacro)
@@ -3,5 +3,5 @@
  ****** File automatically generated by generate_urdf.py script ******
  *********************************************************************-->
-<robot name="pepper" xmlns:xacro="http://www.ros.org/wiki/xacro">
+<robot name="pepper_robot" xmlns:xacro="http://www.ros.org/wiki/xacro">
 	<xacro:include filename="pepper_visual_collisions.xacro"/>
 	<xacro:include filename="pepper_head.xacro"/>

File: pepper_robot_description/urdf/pepper_sensors.xacro (robot description, xacro)
@@ -3,5 +3,5 @@
  ****** File automatically generated by generate_urdf.py script ******
  *********************************************************************-->
-<robot name="pepper" xmlns:xacro="http://www.ros.org/wiki/xacro">
+<robot name="pepper_robot" xmlns:xacro="http://www.ros.org/wiki/xacro">
 	<link name="SonarBack_frame"/>
 	<joint name="Sonar/Back_sensor_fixedjoint" type="fixed">

File: pepper_robot_description/urdf/pepper_wheels.xacro (robot description, xacro)
@@ -3,5 +3,5 @@
  ****** File automatically generated by generate_urdf.py script ******
  *********************************************************************-->
-<robot name="pepper" xmlns:xacro="http://www.ros.org/wiki/xacro">
+<robot name="pepper_robot" xmlns:xacro="http://www.ros.org/wiki/xacro">
 	<link name="WheelFL_link">
 		<inertial>
