Commit message: changed pepper_meshes to pepper_robot

File: pepper_robot_description/urdf/pepper_visual_collisions.xacro (robot description, xacro)
@@ -7,11 +7,11 @@
 		<visual>
 			<geometry>
-				<mesh filename="package://pepper_meshes/meshes/1.0/RFinger41.dae" scale="0.1 0.1 0.1"/>
-			</geometry>
-			<origin rpy="0 0 0" xyz="0 0 0"/>
-		</visual>
-		<collision>
-			<geometry>
-				<mesh filename="package://pepper_meshes/meshes/1.0/RFinger41_0.10.stl" scale="0.1 0.1 0.1"/>
+				<mesh filename="package://pepper_robot/meshes/1.0/RFinger41.dae" scale="0.1 0.1 0.1"/>
+			</geometry>
+			<origin rpy="0 0 0" xyz="0 0 0"/>
+		</visual>
+		<collision>
+			<geometry>
+				<mesh filename="package://pepper_robot/meshes/1.0/RFinger41_0.10.stl" scale="0.1 0.1 0.1"/>
 			</geometry>
 			<origin rpy="0 0 0" xyz="0 0 0"/>
@@ -21,11 +21,11 @@
 		<visual>
 			<geometry>
-				<mesh filename="package://pepper_meshes/meshes/1.0/LFinger42.dae" scale="0.1 0.1 0.1"/>
-			</geometry>
-			<origin rpy="0 0 0" xyz="0 0 0"/>
-		</visual>
-		<collision>
-			<geometry>
-				<mesh filename="package://pepper_meshes/meshes/1.0/LFinger42_0.10.stl" scale="0.1 0.1 0.1"/>
+				<mesh filename="package://pepper_robot/meshes/1.0/LFinger42.dae" scale="0.1 0.1 0.1"/>
+			</geometry>
+			<origin rpy="0 0 0" xyz="0 0 0"/>
+		</visual>
+		<collision>
+			<geometry>
+				<mesh filename="package://pepper_robot/meshes/1.0/LFinger42_0.10.stl" scale="0.1 0.1 0.1"/>
 			</geometry>
 			<origin rpy="0 0 0" xyz="0 0 0"/>
@@ -35,11 +35,11 @@
 		<visual>
 			<geometry>
-				<mesh filename="package://pepper_meshes/meshes/1.0/HipRoll.dae" scale="0.1 0.1 0.1"/>
-			</geometry>
-			<origin rpy="0 0 0" xyz="0 0 0"/>
-		</visual>
-		<collision>
-			<geometry>
-				<mesh filename="package://pepper_meshes/meshes/1.0/HipRoll_0.10.stl" scale="0.1 0.1 0.1"/>
+				<mesh filename="package://pepper_robot/meshes/1.0/HipRoll.dae" scale="0.1 0.1 0.1"/>
+			</geometry>
+			<origin rpy="0 0 0" xyz="0 0 0"/>
+		</visual>
+		<collision>
+			<geometry>
+				<mesh filename="package://pepper_robot/meshes/1.0/HipRoll_0.10.stl" scale="0.1 0.1 0.1"/>
 			</geometry>
 			<origin rpy="0 0 0" xyz="0 0 0"/>
@@ -49,11 +49,11 @@
 		<visual>
 			<geometry>
-				<mesh filename="package://pepper_meshes/meshes/1.0/LElbowYaw.dae" scale="0.1 0.1 0.1"/>
-			</geometry>
-			<origin rpy="0 0 0" xyz="0 0 0"/>
-		</visual>
-		<collision>
-			<geometry>
-				<mesh filename="package://pepper_meshes/meshes/1.0/LElbowYaw_0.10.stl" scale="0.1 0.1 0.1"/>
+				<mesh filename="package://pepper_robot/meshes/1.0/LElbowYaw.dae" scale="0.1 0.1 0.1"/>
+			</geometry>
+			<origin rpy="0 0 0" xyz="0 0 0"/>
+		</visual>
+		<collision>
+			<geometry>
+				<mesh filename="package://pepper_robot/meshes/1.0/LElbowYaw_0.10.stl" scale="0.1 0.1 0.1"/>
 			</geometry>
 			<origin rpy="0 0 0" xyz="0 0 0"/>
@@ -63,11 +63,11 @@
 		<visual>
 			<geometry>
-				<mesh filename="package://pepper_meshes/meshes/1.0/RFinger12.dae" scale="0.1 0.1 0.1"/>
-			</geometry>
-			<origin rpy="0 0 0" xyz="0 0 0"/>
-		</visual>
-		<collision>
-			<geometry>
-				<mesh filename="package://pepper_meshes/meshes/1.0/RFinger12_0.10.stl" scale="0.1 0.1 0.1"/>
+				<mesh filename="package://pepper_robot/meshes/1.0/RFinger12.dae" scale="0.1 0.1 0.1"/>
+			</geometry>
+			<origin rpy="0 0 0" xyz="0 0 0"/>
+		</visual>
+		<collision>
+			<geometry>
+				<mesh filename="package://pepper_robot/meshes/1.0/RFinger12_0.10.stl" scale="0.1 0.1 0.1"/>
 			</geometry>
 			<origin rpy="0 0 0" xyz="0 0 0"/>
@@ -77,11 +77,11 @@
 		<visual>
 			<geometry>
-				<mesh filename="package://pepper_meshes/meshes/1.0/LFinger33.dae" scale="0.1 0.1 0.1"/>
-			</geometry>
-			<origin rpy="0 0 0" xyz="0 0 0"/>
-		</visual>
-		<collision>
-			<geometry>
-				<mesh filename="package://pepper_meshes/meshes/1.0/LFinger33_0.10.stl" scale="0.1 0.1 0.1"/>
+				<mesh filename="package://pepper_robot/meshes/1.0/LFinger33.dae" scale="0.1 0.1 0.1"/>
+			</geometry>
+			<origin rpy="0 0 0" xyz="0 0 0"/>
+		</visual>
+		<collision>
+			<geometry>
+				<mesh filename="package://pepper_robot/meshes/1.0/LFinger33_0.10.stl" scale="0.1 0.1 0.1"/>
 			</geometry>
 			<origin rpy="0 0 0" xyz="0 0 0"/>
@@ -91,11 +91,11 @@
 		<visual>
 			<geometry>
-				<mesh filename="package://pepper_meshes/meshes/1.0/RFinger31.dae" scale="0.1 0.1 0.1"/>
-			</geometry>
-			<origin rpy="0 0 0" xyz="0 0 0"/>
-		</visual>
-		<collision>
-			<geometry>
-				<mesh filename="package://pepper_meshes/meshes/1.0/RFinger31_0.10.stl" scale="0.1 0.1 0.1"/>
+				<mesh filename="package://pepper_robot/meshes/1.0/RFinger31.dae" scale="0.1 0.1 0.1"/>
+			</geometry>
+			<origin rpy="0 0 0" xyz="0 0 0"/>
+		</visual>
+		<collision>
+			<geometry>
+				<mesh filename="package://pepper_robot/meshes/1.0/RFinger31_0.10.stl" scale="0.1 0.1 0.1"/>
 			</geometry>
 			<origin rpy="0 0 0" xyz="0 0 0"/>
@@ -105,11 +105,11 @@
 		<visual>
 			<geometry>
-				<mesh filename="package://pepper_meshes/meshes/1.0/WheelFL.dae" scale="0.1 0.1 0.1"/>
-			</geometry>
-			<origin rpy="0 0 0" xyz="0 0 0"/>
-		</visual>
-		<collision>
-			<geometry>
-				<mesh filename="package://pepper_meshes/meshes/1.0/WheelFL_0.10.stl" scale="0.1 0.1 0.1"/>
+				<mesh filename="package://pepper_robot/meshes/1.0/WheelFL.dae" scale="0.1 0.1 0.1"/>
+			</geometry>
+			<origin rpy="0 0 0" xyz="0 0 0"/>
+		</visual>
+		<collision>
+			<geometry>
+				<mesh filename="package://pepper_robot/meshes/1.0/WheelFL_0.10.stl" scale="0.1 0.1 0.1"/>
 			</geometry>
 			<origin rpy="0 0 0" xyz="0 0 0"/>
@@ -119,11 +119,11 @@
 		<visual>
 			<geometry>
-				<mesh filename="package://pepper_meshes/meshes/1.0/LFinger21.dae" scale="0.1 0.1 0.1"/>
-			</geometry>
-			<origin rpy="0 0 0" xyz="0 0 0"/>
-		</visual>
-		<collision>
-			<geometry>
-				<mesh filename="package://pepper_meshes/meshes/1.0/LFinger21_0.10.stl" scale="0.1 0.1 0.1"/>
+				<mesh filename="package://pepper_robot/meshes/1.0/LFinger21.dae" scale="0.1 0.1 0.1"/>
+			</geometry>
+			<origin rpy="0 0 0" xyz="0 0 0"/>
+		</visual>
+		<collision>
+			<geometry>
+				<mesh filename="package://pepper_robot/meshes/1.0/LFinger21_0.10.stl" scale="0.1 0.1 0.1"/>
 			</geometry>
 			<origin rpy="0 0 0" xyz="0 0 0"/>
@@ -133,11 +133,11 @@
 		<visual>
 			<geometry>
-				<mesh filename="package://pepper_meshes/meshes/1.0/RFinger32.dae" scale="0.1 0.1 0.1"/>
-			</geometry>
-			<origin rpy="0 0 0" xyz="0 0 0"/>
-		</visual>
-		<collision>
-			<geometry>
-				<mesh filename="package://pepper_meshes/meshes/1.0/RFinger32_0.10.stl" scale="0.1 0.1 0.1"/>
+				<mesh filename="package://pepper_robot/meshes/1.0/RFinger32.dae" scale="0.1 0.1 0.1"/>
+			</geometry>
+			<origin rpy="0 0 0" xyz="0 0 0"/>
+		</visual>
+		<collision>
+			<geometry>
+				<mesh filename="package://pepper_robot/meshes/1.0/RFinger32_0.10.stl" scale="0.1 0.1 0.1"/>
 			</geometry>
 			<origin rpy="0 0 0" xyz="0 0 0"/>
@@ -147,11 +147,11 @@
 		<visual>
 			<geometry>
-				<mesh filename="package://pepper_meshes/meshes/1.0/LFinger13.dae" scale="0.1 0.1 0.1"/>
-			</geometry>
-			<origin rpy="0 0 0" xyz="0 0 0"/>
-		</visual>
-		<collision>
-			<geometry>
-				<mesh filename="package://pepper_meshes/meshes/1.0/LFinger13_0.10.stl" scale="0.1 0.1 0.1"/>
+				<mesh filename="package://pepper_robot/meshes/1.0/LFinger13.dae" scale="0.1 0.1 0.1"/>
+			</geometry>
+			<origin rpy="0 0 0" xyz="0 0 0"/>
+		</visual>
+		<collision>
+			<geometry>
+				<mesh filename="package://pepper_robot/meshes/1.0/LFinger13_0.10.stl" scale="0.1 0.1 0.1"/>
 			</geometry>
 			<origin rpy="0 0 0" xyz="0 0 0"/>
@@ -161,11 +161,11 @@
 		<visual>
 			<geometry>
-				<mesh filename="package://pepper_meshes/meshes/1.0/LFinger32.dae" scale="0.1 0.1 0.1"/>
-			</geometry>
-			<origin rpy="0 0 0" xyz="0 0 0"/>
-		</visual>
-		<collision>
-			<geometry>
-				<mesh filename="package://pepper_meshes/meshes/1.0/LFinger32_0.10.stl" scale="0.1 0.1 0.1"/>
+				<mesh filename="package://pepper_robot/meshes/1.0/LFinger32.dae" scale="0.1 0.1 0.1"/>
+			</geometry>
+			<origin rpy="0 0 0" xyz="0 0 0"/>
+		</visual>
+		<collision>
+			<geometry>
+				<mesh filename="package://pepper_robot/meshes/1.0/LFinger32_0.10.stl" scale="0.1 0.1 0.1"/>
 			</geometry>
 			<origin rpy="0 0 0" xyz="0 0 0"/>
@@ -175,11 +175,11 @@
 		<visual>
 			<geometry>
-				<mesh filename="package://pepper_meshes/meshes/1.0/LThumb1.dae" scale="0.1 0.1 0.1"/>
-			</geometry>
-			<origin rpy="0 0 0" xyz="0 0 0"/>
-		</visual>
-		<collision>
-			<geometry>
-				<mesh filename="package://pepper_meshes/meshes/1.0/LThumb1_0.10.stl" scale="0.1 0.1 0.1"/>
+				<mesh filename="package://pepper_robot/meshes/1.0/LThumb1.dae" scale="0.1 0.1 0.1"/>
+			</geometry>
+			<origin rpy="0 0 0" xyz="0 0 0"/>
+		</visual>
+		<collision>
+			<geometry>
+				<mesh filename="package://pepper_robot/meshes/1.0/LThumb1_0.10.stl" scale="0.1 0.1 0.1"/>
 			</geometry>
 			<origin rpy="0 0 0" xyz="0 0 0"/>
@@ -189,11 +189,11 @@
 		<visual>
 			<geometry>
-				<mesh filename="package://pepper_meshes/meshes/1.0/LFinger11.dae" scale="0.1 0.1 0.1"/>
-			</geometry>
-			<origin rpy="0 0 0" xyz="0 0 0"/>
-		</visual>
-		<collision>
-			<geometry>
-				<mesh filename="package://pepper_meshes/meshes/1.0/LFinger11_0.10.stl" scale="0.1 0.1 0.1"/>
+				<mesh filename="package://pepper_robot/meshes/1.0/LFinger11.dae" scale="0.1 0.1 0.1"/>
+			</geometry>
+			<origin rpy="0 0 0" xyz="0 0 0"/>
+		</visual>
+		<collision>
+			<geometry>
+				<mesh filename="package://pepper_robot/meshes/1.0/LFinger11_0.10.stl" scale="0.1 0.1 0.1"/>
 			</geometry>
 			<origin rpy="0 0 0" xyz="0 0 0"/>
@@ -203,11 +203,11 @@
 		<visual>
 			<geometry>
-				<mesh filename="package://pepper_meshes/meshes/1.0/RFinger22.dae" scale="0.1 0.1 0.1"/>
-			</geometry>
-			<origin rpy="0 0 0" xyz="0 0 0"/>
-		</visual>
-		<collision>
-			<geometry>
-				<mesh filename="package://pepper_meshes/meshes/1.0/RFinger22_0.10.stl" scale="0.1 0.1 0.1"/>
+				<mesh filename="package://pepper_robot/meshes/1.0/RFinger22.dae" scale="0.1 0.1 0.1"/>
+			</geometry>
+			<origin rpy="0 0 0" xyz="0 0 0"/>
+		</visual>
+		<collision>
+			<geometry>
+				<mesh filename="package://pepper_robot/meshes/1.0/RFinger22_0.10.stl" scale="0.1 0.1 0.1"/>
 			</geometry>
 			<origin rpy="0 0 0" xyz="0 0 0"/>
@@ -217,11 +217,11 @@
 		<visual>
 			<geometry>
-				<mesh filename="package://pepper_meshes/meshes/1.0/RThumb2.dae" scale="0.1 0.1 0.1"/>
-			</geometry>
-			<origin rpy="0 0 0" xyz="0 0 0"/>
-		</visual>
-		<collision>
-			<geometry>
-				<mesh filename="package://pepper_meshes/meshes/1.0/RThumb2_0.10.stl" scale="0.1 0.1 0.1"/>
+				<mesh filename="package://pepper_robot/meshes/1.0/RThumb2.dae" scale="0.1 0.1 0.1"/>
+			</geometry>
+			<origin rpy="0 0 0" xyz="0 0 0"/>
+		</visual>
+		<collision>
+			<geometry>
+				<mesh filename="package://pepper_robot/meshes/1.0/RThumb2_0.10.stl" scale="0.1 0.1 0.1"/>
 			</geometry>
 			<origin rpy="0 0 0" xyz="0 0 0"/>
@@ -231,11 +231,11 @@
 		<visual>
 			<geometry>
-				<mesh filename="package://pepper_meshes/meshes/1.0/RFinger13.dae" scale="0.1 0.1 0.1"/>
-			</geometry>
-			<origin rpy="0 0 0" xyz="0 0 0"/>
-		</visual>
-		<collision>
-			<geometry>
-				<mesh filename="package://pepper_meshes/meshes/1.0/RFinger13_0.10.stl" scale="0.1 0.1 0.1"/>
+				<mesh filename="package://pepper_robot/meshes/1.0/RFinger13.dae" scale="0.1 0.1 0.1"/>
+			</geometry>
+			<origin rpy="0 0 0" xyz="0 0 0"/>
+		</visual>
+		<collision>
+			<geometry>
+				<mesh filename="package://pepper_robot/meshes/1.0/RFinger13_0.10.stl" scale="0.1 0.1 0.1"/>
 			</geometry>
 			<origin rpy="0 0 0" xyz="0 0 0"/>
@@ -245,11 +245,11 @@
 		<visual>
 			<geometry>
-				<mesh filename="package://pepper_meshes/meshes/1.0/KneePitch.dae" scale="0.1 0.1 0.1"/>
-			</geometry>
-			<origin rpy="0 0 0" xyz="0 0 0"/>
-		</visual>
-		<collision>
-			<geometry>
-				<mesh filename="package://pepper_meshes/meshes/1.0/KneePitch_0.10.stl" scale="0.1 0.1 0.1"/>
+				<mesh filename="package://pepper_robot/meshes/1.0/KneePitch.dae" scale="0.1 0.1 0.1"/>
+			</geometry>
+			<origin rpy="0 0 0" xyz="0 0 0"/>
+		</visual>
+		<collision>
+			<geometry>
+				<mesh filename="package://pepper_robot/meshes/1.0/KneePitch_0.10.stl" scale="0.1 0.1 0.1"/>
 			</geometry>
 			<origin rpy="0 0 0" xyz="0 0 0"/>
@@ -259,11 +259,11 @@
 		<visual>
 			<geometry>
-				<mesh filename="package://pepper_meshes/meshes/1.0/HeadPitch.dae" scale="0.1 0.1 0.1"/>
-			</geometry>
-			<origin rpy="0 0 0" xyz="0 0 0"/>
-		</visual>
-		<collision>
-			<geometry>
-				<mesh filename="package://pepper_meshes/meshes/1.0/HeadPitch_0.10.stl" scale="0.1 0.1 0.1"/>
+				<mesh filename="package://pepper_robot/meshes/1.0/HeadPitch.dae" scale="0.1 0.1 0.1"/>
+			</geometry>
+			<origin rpy="0 0 0" xyz="0 0 0"/>
+		</visual>
+		<collision>
+			<geometry>
+				<mesh filename="package://pepper_robot/meshes/1.0/HeadPitch_0.10.stl" scale="0.1 0.1 0.1"/>
 			</geometry>
 			<origin rpy="0 0 0" xyz="0 0 0"/>
@@ -273,11 +273,11 @@
 		<visual>
 			<geometry>
-				<mesh filename="package://pepper_meshes/meshes/1.0/LFinger22.dae" scale="0.1 0.1 0.1"/>
-			</geometry>
-			<origin rpy="0 0 0" xyz="0 0 0"/>
-		</visual>
-		<collision>
-			<geometry>
-				<mesh filename="package://pepper_meshes/meshes/1.0/LFinger22_0.10.stl" scale="0.1 0.1 0.1"/>
+				<mesh filename="package://pepper_robot/meshes/1.0/LFinger22.dae" scale="0.1 0.1 0.1"/>
+			</geometry>
+			<origin rpy="0 0 0" xyz="0 0 0"/>
+		</visual>
+		<collision>
+			<geometry>
+				<mesh filename="package://pepper_robot/meshes/1.0/LFinger22_0.10.stl" scale="0.1 0.1 0.1"/>
 			</geometry>
 			<origin rpy="0 0 0" xyz="0 0 0"/>
@@ -287,11 +287,11 @@
 		<visual>
 			<geometry>
-				<mesh filename="package://pepper_meshes/meshes/1.0/RFinger21.dae" scale="0.1 0.1 0.1"/>
-			</geometry>
-			<origin rpy="0 0 0" xyz="0 0 0"/>
-		</visual>
-		<collision>
-			<geometry>
-				<mesh filename="package://pepper_meshes/meshes/1.0/RFinger21_0.10.stl" scale="0.1 0.1 0.1"/>
+				<mesh filename="package://pepper_robot/meshes/1.0/RFinger21.dae" scale="0.1 0.1 0.1"/>
+			</geometry>
+			<origin rpy="0 0 0" xyz="0 0 0"/>
+		</visual>
+		<collision>
+			<geometry>
+				<mesh filename="package://pepper_robot/meshes/1.0/RFinger21_0.10.stl" scale="0.1 0.1 0.1"/>
 			</geometry>
 			<origin rpy="0 0 0" xyz="0 0 0"/>
@@ -301,11 +301,11 @@
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