Commit message: fix urdf files

File: pepper_robot_description/urdf/pepper_robot.urdf (robot description, URDF)
Before this commit: robot JulietteY20MP, 83 links, 82 joints
Links:
- link Head: geometry collision mesh filename=package://pepper_robot/meshes/HeadPitch_0.10.stl scale=0.1 0.1 0.1; visual mesh filename=package://pepper_robot/meshes/HeadPitch.dae scale=0.1 0.1 0.1
- link Hip: geometry collision mesh filename=package://pepper_robot/meshes/HipRoll_0.10.stl scale=0.1 0.1 0.1; visual mesh filename=package://pepper_robot/meshes/HipRoll.dae scale=0.1 0.1 0.1
- link LBicep: geometry collision mesh filename=package://pepper_robot/meshes/LShoulderRoll_0.10.stl scale=0.1 0.1 0.1; visual mesh filename=package://pepper_robot/meshes/LShoulderRoll.dae scale=0.1 0.1 0.1
- link LElbow: geometry collision mesh filename=package://pepper_robot/meshes/LElbowYaw_0.10.stl scale=0.1 0.1 0.1; visual mesh filename=package://pepper_robot/meshes/LElbowYaw.dae scale=0.1 0.1 0.1
- link LFinger11_link: geometry collision mesh filename=package://pepper_robot/meshes/LFinger11_0.10.stl scale=0.1 0.1 0.1; visual mesh filename=package://pepper_robot/meshes/LFinger11.dae scale=0.1 0.1 0.1
- link LFinger12_link: geometry collision mesh filename=package://pepper_robot/meshes/LFinger12_0.10.stl scale=0.1 0.1 0.1; visual mesh filename=package://pepper_robot/meshes/LFinger12.dae scale=0.1 0.1 0.1
- link LFinger13_link: geometry collision mesh filename=package://pepper_robot/meshes/LFinger13_0.10.stl scale=0.1 0.1 0.1; visual mesh filename=package://pepper_robot/meshes/LFinger13.dae scale=0.1 0.1 0.1
- link LFinger21_link: geometry collision mesh filename=package://pepper_robot/meshes/LFinger21_0.10.stl scale=0.1 0.1 0.1; visual mesh filename=package://pepper_robot/meshes/LFinger21.dae scale=0.1 0.1 0.1
- link LFinger22_link: geometry collision mesh filename=package://pepper_robot/meshes/LFinger22_0.10.stl scale=0.1 0.1 0.1; visual mesh filename=package://pepper_robot/meshes/LFinger22.dae scale=0.1 0.1 0.1
- link LFinger23_link: geometry collision mesh filename=package://pepper_robot/meshes/LFinger23_0.10.stl scale=0.1 0.1 0.1; visual mesh filename=package://pepper_robot/meshes/LFinger23.dae scale=0.1 0.1 0.1
- link LFinger31_link: geometry collision mesh filename=package://pepper_robot/meshes/LFinger31_0.10.stl scale=0.1 0.1 0.1; visual mesh filename=package://pepper_robot/meshes/LFinger31.dae scale=0.1 0.1 0.1
- link LFinger32_link: geometry collision mesh filename=package://pepper_robot/meshes/LFinger32_0.10.stl scale=0.1 0.1 0.1; visual mesh filename=package://pepper_robot/meshes/LFinger32.dae scale=0.1 0.1 0.1
- link LFinger33_link: geometry collision mesh filename=package://pepper_robot/meshes/LFinger33_0.10.stl scale=0.1 0.1 0.1; visual mesh filename=package://pepper_robot/meshes/LFinger33.dae scale=0.1 0.1 0.1
- link LFinger41_link: geometry collision mesh filename=package://pepper_robot/meshes/LFinger41_0.10.stl scale=0.1 0.1 0.1; visual mesh filename=package://pepper_robot/meshes/LFinger41.dae scale=0.1 0.1 0.1
- link LFinger42_link: geometry collision mesh filename=package://pepper_robot/meshes/LFinger42_0.10.stl scale=0.1 0.1 0.1; visual mesh filename=package://pepper_robot/meshes/LFinger42.dae scale=0.1 0.1 0.1
- link LFinger43_link: geometry collision mesh filename=package://pepper_robot/meshes/LFinger43_0.10.stl scale=0.1 0.1 0.1; visual mesh filename=package://pepper_robot/meshes/LFinger43.dae scale=0.1 0.1 0.1
- link LForeArm: geometry collision mesh filename=package://pepper_robot/meshes/LElbowRoll_0.10.stl scale=0.1 0.1 0.1; visual mesh filename=package://pepper_robot/meshes/LElbowRoll.dae scale=0.1 0.1 0.1
- link LShoulder: geometry collision mesh filename=package://pepper_robot/meshes/LShoulderPitch_0.10.stl scale=0.1 0.1 0.1; visual mesh filename=package://pepper_robot/meshes/LShoulderPitch.dae scale=0.1 0.1 0.1
- link LThumb1_link: geometry collision mesh filename=package://pepper_robot/meshes/LThumb1_0.10.stl scale=0.1 0.1 0.1; visual mesh filename=package://pepper_robot/meshes/LThumb1.dae scale=0.1 0.1 0.1
- link LThumb2_link: geometry collision mesh filename=package://pepper_robot/meshes/LThumb2_0.10.stl scale=0.1 0.1 0.1; visual mesh filename=package://pepper_robot/meshes/LThumb2.dae scale=0.1 0.1 0.1
- link Neck: geometry collision mesh filename=package://pepper_robot/meshes/HeadYaw_0.10.stl scale=0.1 0.1 0.1; visual mesh filename=package://pepper_robot/meshes/HeadYaw.dae scale=0.1 0.1 0.1
- link Pelvis: geometry collision mesh filename=package://pepper_robot/meshes/HipPitch_0.10.stl scale=0.1 0.1 0.1; visual mesh filename=package://pepper_robot/meshes/HipPitch.dae scale=0.1 0.1 0.1
- link RBicep: geometry collision mesh filename=package://pepper_robot/meshes/RShoulderRoll_0.10.stl scale=0.1 0.1 0.1; visual mesh filename=package://pepper_robot/meshes/RShoulderRoll.dae scale=0.1 0.1 0.1
- link RElbow: geometry collision mesh filename=package://pepper_robot/meshes/RElbowYaw_0.10.stl scale=0.1 0.1 0.1; visual mesh filename=package://pepper_robot/meshes/RElbowYaw.dae scale=0.1 0.1 0.1
- link RFinger11_link: geometry collision mesh filename=package://pepper_robot/meshes/RFinger11_0.10.stl scale=0.1 0.1 0.1; visual mesh filename=package://pepper_robot/meshes/RFinger11.dae scale=0.1 0.1 0.1
- link RFinger12_link: geometry collision mesh filename=package://pepper_robot/meshes/RFinger12_0.10.stl scale=0.1 0.1 0.1; visual mesh filename=package://pepper_robot/meshes/RFinger12.dae scale=0.1 0.1 0.1
- link RFinger13_link: geometry collision mesh filename=package://pepper_robot/meshes/RFinger13_0.10.stl scale=0.1 0.1 0.1; visual mesh filename=package://pepper_robot/meshes/RFinger13.dae scale=0.1 0.1 0.1
- link RFinger21_link: geometry collision mesh filename=package://pepper_robot/meshes/RFinger21_0.10.stl scale=0.1 0.1 0.1; visual mesh filename=package://pepper_robot/meshes/RFinger21.dae scale=0.1 0.1 0.1
- link RFinger22_link: geometry collision mesh filename=package://pepper_robot/meshes/RFinger22_0.10.stl scale=0.1 0.1 0.1; visual mesh filename=package://pepper_robot/meshes/RFinger22.dae scale=0.1 0.1 0.1
- link RFinger23_link: geometry collision mesh filename=package://pepper_robot/meshes/RFinger23_0.10.stl scale=0.1 0.1 0.1; visual mesh filename=package://pepper_robot/meshes/RFinger23.dae scale=0.1 0.1 0.1
- link RFinger31_link: geometry collision mesh filename=package://pepper_robot/meshes/RFinger31_0.10.stl scale=0.1 0.1 0.1; visual mesh filename=package://pepper_robot/meshes/RFinger31.dae scale=0.1 0.1 0.1
- link RFinger32_link: geometry collision mesh filename=package://pepper_robot/meshes/RFinger32_0.10.stl scale=0.1 0.1 0.1; visual mesh filename=package://pepper_robot/meshes/RFinger32.dae scale=0.1 0.1 0.1
- link RFinger33_link: geometry collision mesh filename=package://pepper_robot/meshes/RFinger33_0.10.stl scale=0.1 0.1 0.1; visual mesh filename=package://pepper_robot/meshes/RFinger33.dae scale=0.1 0.1 0.1
- link RFinger41_link: geometry collision mesh filename=package://pepper_robot/meshes/RFinger41_0.10.stl scale=0.1 0.1 0.1; visual mesh filename=package://pepper_robot/meshes/RFinger41.dae scale=0.1 0.1 0.1
- link RFinger42_link: geometry collision mesh filename=package://pepper_robot/meshes/RFinger42_0.10.stl scale=0.1 0.1 0.1; visual mesh filename=package://pepper_robot/meshes/RFinger42.dae scale=0.1 0.1 0.1
- link RFinger43_link: geometry collision mesh filename=package://pepper_robot/meshes/RFinger43_0.10.stl scale=0.1 0.1 0.1; visual mesh filename=package://pepper_robot/meshes/RFinger43.dae scale=0.1 0.1 0.1
- link RForeArm: geometry collision mesh filename=package://pepper_robot/meshes/RElbowRoll_0.10.stl scale=0.1 0.1 0.1; visual mesh filename=package://pepper_robot/meshes/RElbowRoll.dae scale=0.1 0.1 0.1
- link RShoulder: geometry collision mesh filename=package://pepper_robot/meshes/RShoulderPitch_0.10.stl scale=0.1 0.1 0.1; visual mesh filename=package://pepper_robot/meshes/RShoulderPitch.dae scale=0.1 0.1 0.1
- link RThumb1_link: geometry collision mesh filename=package://pepper_robot/meshes/RThumb1_0.10.stl scale=0.1 0.1 0.1; visual mesh filename=package://pepper_robot/meshes/RThumb1.dae scale=0.1 0.1 0.1
- link RThumb2_link: geometry collision mesh filename=package://pepper_robot/meshes/RThumb2_0.10.stl scale=0.1 0.1 0.1; visual mesh filename=package://pepper_robot/meshes/RThumb2.dae scale=0.1 0.1 0.1
- link Tibia: geometry collision mesh filename=package://pepper_robot/meshes/KneePitch_0.10.stl scale=0.1 0.1 0.1; visual mesh filename=package://pepper_robot/meshes/KneePitch.dae scale=0.1 0.1 0.1
- link WheelB_link: geometry collision mesh filename=package://pepper_robot/meshes/WheelB_0.10.stl scale=0.1 0.1 0.1; visual mesh filename=package://pepper_robot/meshes/WheelB.dae scale=0.1 0.1 0.1
- link WheelFL_link: geometry collision mesh filename=package://pepper_robot/meshes/WheelFL_0.10.stl scale=0.1 0.1 0.1; visual mesh filename=package://pepper_robot/meshes/WheelFL.dae scale=0.1 0.1 0.1
- link WheelFR_link: geometry collision mesh filename=package://pepper_robot/meshes/WheelFR_0.10.stl scale=0.1 0.1 0.1; visual mesh filename=package://pepper_robot/meshes/WheelFR.dae scale=0.1 0.1 0.1
- link l_wrist: geometry collision mesh filename=package://pepper_robot/meshes/LWristYaw_0.10.stl scale=0.1 0.1 0.1; visual mesh filename=package://pepper_robot/meshes/LWristYaw.dae scale=0.1 0.1 0.1
- link r_wrist: geometry collision mesh filename=package://pepper_robot/meshes/RWristYaw_0.10.stl scale=0.1 0.1 0.1; visual mesh filename=package://pepper_robot/meshes/RWristYaw.dae scale=0.1 0.1 0.1
- link torso: geometry collision mesh filename=package://pepper_robot/meshes/Torso_0.10.stl scale=0.1 0.1 0.1; visual mesh filename=package://pepper_robot/meshes/Torso.dae scale=0.1 0.1 0.1
