Commit message: fix the path in the urdf file

File: pepper_robot_description/urdf/pepper_visual_collisions.xacro (robot description, xacro)
@@ -7,11 +7,11 @@
 		<visual>
 			<geometry>
-				<mesh filename="package://pepper_robot/meshes/RFinger41.dae" scale="0.1 0.1 0.1"/>
-			</geometry>
-			<origin rpy="0 0 0" xyz="0 0 0"/>
-		</visual>
-		<collision>
-			<geometry>
-				<mesh filename="package://pepper_robot/meshes/RFinger41_0.10.stl" scale="0.1 0.1 0.1"/>
+				<mesh filename="package://pepper_robot_description/meshes/RFinger41.dae" scale="0.1 0.1 0.1"/>
+			</geometry>
+			<origin rpy="0 0 0" xyz="0 0 0"/>
+		</visual>
+		<collision>
+			<geometry>
+				<mesh filename="package://pepper_robot_description/meshes/RFinger41_0.10.stl" scale="0.1 0.1 0.1"/>
 			</geometry>
 			<origin rpy="0 0 0" xyz="0 0 0"/>
@@ -21,11 +21,11 @@
 		<visual>
 			<geometry>
-				<mesh filename="package://pepper_robot/meshes/LFinger42.dae" scale="0.1 0.1 0.1"/>
-			</geometry>
-			<origin rpy="0 0 0" xyz="0 0 0"/>
-		</visual>
-		<collision>
-			<geometry>
-				<mesh filename="package://pepper_robot/meshes/LFinger42_0.10.stl" scale="0.1 0.1 0.1"/>
+				<mesh filename="package://pepper_robot_description/meshes/LFinger42.dae" scale="0.1 0.1 0.1"/>
+			</geometry>
+			<origin rpy="0 0 0" xyz="0 0 0"/>
+		</visual>
+		<collision>
+			<geometry>
+				<mesh filename="package://pepper_robot_description/meshes/LFinger42_0.10.stl" scale="0.1 0.1 0.1"/>
 			</geometry>
 			<origin rpy="0 0 0" xyz="0 0 0"/>
@@ -35,11 +35,11 @@
 		<visual>
 			<geometry>
-				<mesh filename="package://pepper_robot/meshes/HipRoll.dae" scale="0.1 0.1 0.1"/>
-			</geometry>
-			<origin rpy="0 0 0" xyz="0 0 0"/>
-		</visual>
-		<collision>
-			<geometry>
-				<mesh filename="package://pepper_robot/meshes/HipRoll_0.10.stl" scale="0.1 0.1 0.1"/>
+				<mesh filename="package://pepper_robot_description/meshes/HipRoll.dae" scale="0.1 0.1 0.1"/>
+			</geometry>
+			<origin rpy="0 0 0" xyz="0 0 0"/>
+		</visual>
+		<collision>
+			<geometry>
+				<mesh filename="package://pepper_robot_description/meshes/HipRoll_0.10.stl" scale="0.1 0.1 0.1"/>
 			</geometry>
 			<origin rpy="0 0 0" xyz="0 0 0"/>
@@ -49,11 +49,11 @@
 		<visual>
 			<geometry>
-				<mesh filename="package://pepper_robot/meshes/LElbowYaw.dae" scale="0.1 0.1 0.1"/>
-			</geometry>
-			<origin rpy="0 0 0" xyz="0 0 0"/>
-		</visual>
-		<collision>
-			<geometry>
-				<mesh filename="package://pepper_robot/meshes/LElbowYaw_0.10.stl" scale="0.1 0.1 0.1"/>
+				<mesh filename="package://pepper_robot_description/meshes/LElbowYaw.dae" scale="0.1 0.1 0.1"/>
+			</geometry>
+			<origin rpy="0 0 0" xyz="0 0 0"/>
+		</visual>
+		<collision>
+			<geometry>
+				<mesh filename="package://pepper_robot_description/meshes/LElbowYaw_0.10.stl" scale="0.1 0.1 0.1"/>
 			</geometry>
 			<origin rpy="0 0 0" xyz="0 0 0"/>
@@ -63,11 +63,11 @@
 		<visual>
 			<geometry>
-				<mesh filename="package://pepper_robot/meshes/RFinger12.dae" scale="0.1 0.1 0.1"/>
-			</geometry>
-			<origin rpy="0 0 0" xyz="0 0 0"/>
-		</visual>
-		<collision>
-			<geometry>
-				<mesh filename="package://pepper_robot/meshes/RFinger12_0.10.stl" scale="0.1 0.1 0.1"/>
+				<mesh filename="package://pepper_robot_description/meshes/RFinger12.dae" scale="0.1 0.1 0.1"/>
+			</geometry>
+			<origin rpy="0 0 0" xyz="0 0 0"/>
+		</visual>
+		<collision>
+			<geometry>
+				<mesh filename="package://pepper_robot_description/meshes/RFinger12_0.10.stl" scale="0.1 0.1 0.1"/>
 			</geometry>
 			<origin rpy="0 0 0" xyz="0 0 0"/>
@@ -77,11 +77,11 @@
 		<visual>
 			<geometry>
-				<mesh filename="package://pepper_robot/meshes/LFinger33.dae" scale="0.1 0.1 0.1"/>
-			</geometry>
-			<origin rpy="0 0 0" xyz="0 0 0"/>
-		</visual>
-		<collision>
-			<geometry>
-				<mesh filename="package://pepper_robot/meshes/LFinger33_0.10.stl" scale="0.1 0.1 0.1"/>
+				<mesh filename="package://pepper_robot_description/meshes/LFinger33.dae" scale="0.1 0.1 0.1"/>
+			</geometry>
+			<origin rpy="0 0 0" xyz="0 0 0"/>
+		</visual>
+		<collision>
+			<geometry>
+				<mesh filename="package://pepper_robot_description/meshes/LFinger33_0.10.stl" scale="0.1 0.1 0.1"/>
 			</geometry>
 			<origin rpy="0 0 0" xyz="0 0 0"/>
@@ -91,11 +91,11 @@
 		<visual>
 			<geometry>
-				<mesh filename="package://pepper_robot/meshes/RFinger31.dae" scale="0.1 0.1 0.1"/>
-			</geometry>
-			<origin rpy="0 0 0" xyz="0 0 0"/>
-		</visual>
-		<collision>
-			<geometry>
-				<mesh filename="package://pepper_robot/meshes/RFinger31_0.10.stl" scale="0.1 0.1 0.1"/>
+				<mesh filename="package://pepper_robot_description/meshes/RFinger31.dae" scale="0.1 0.1 0.1"/>
+			</geometry>
+			<origin rpy="0 0 0" xyz="0 0 0"/>
+		</visual>
+		<collision>
+			<geometry>
+				<mesh filename="package://pepper_robot_description/meshes/RFinger31_0.10.stl" scale="0.1 0.1 0.1"/>
 			</geometry>
 			<origin rpy="0 0 0" xyz="0 0 0"/>
@@ -105,11 +105,11 @@
 		<visual>
 			<geometry>
-				<mesh filename="package://pepper_robot/meshes/WheelFL.dae" scale="0.1 0.1 0.1"/>
-			</geometry>
-			<origin rpy="0 0 0" xyz="0 0 0"/>
-		</visual>
-		<collision>
-			<geometry>
-				<mesh filename="package://pepper_robot/meshes/WheelFL_0.10.stl" scale="0.1 0.1 0.1"/>
+				<mesh filename="package://pepper_robot_description/meshes/WheelFL.dae" scale="0.1 0.1 0.1"/>
+			</geometry>
+			<origin rpy="0 0 0" xyz="0 0 0"/>
+		</visual>
+		<collision>
+			<geometry>
+				<mesh filename="package://pepper_robot_description/meshes/WheelFL_0.10.stl" scale="0.1 0.1 0.1"/>
 			</geometry>
 			<origin rpy="0 0 0" xyz="0 0 0"/>
@@ -119,11 +119,11 @@
 		<visual>
 			<geometry>
-				<mesh filename="package://pepper_robot/meshes/LFinger21.dae" scale="0.1 0.1 0.1"/>
-			</geometry>
-			<origin rpy="0 0 0" xyz="0 0 0"/>
-		</visual>
-		<collision>
-			<geometry>
-				<mesh filename="package://pepper_robot/meshes/LFinger21_0.10.stl" scale="0.1 0.1 0.1"/>
+				<mesh filename="package://pepper_robot_description/meshes/LFinger21.dae" scale="0.1 0.1 0.1"/>
+			</geometry>
+			<origin rpy="0 0 0" xyz="0 0 0"/>
+		</visual>
+		<collision>
+			<geometry>
+				<mesh filename="package://pepper_robot_description/meshes/LFinger21_0.10.stl" scale="0.1 0.1 0.1"/>
 			</geometry>
 			<origin rpy="0 0 0" xyz="0 0 0"/>
@@ -133,11 +133,11 @@
 		<visual>
 			<geometry>
-				<mesh filename="package://pepper_robot/meshes/RFinger32.dae" scale="0.1 0.1 0.1"/>
-			</geometry>
-			<origin rpy="0 0 0" xyz="0 0 0"/>
-		</visual>
-		<collision>
-			<geometry>
-				<mesh filename="package://pepper_robot/meshes/RFinger32_0.10.stl" scale="0.1 0.1 0.1"/>
+				<mesh filename="package://pepper_robot_description/meshes/RFinger32.dae" scale="0.1 0.1 0.1"/>
+			</geometry>
+			<origin rpy="0 0 0" xyz="0 0 0"/>
+		</visual>
+		<collision>
+			<geometry>
+				<mesh filename="package://pepper_robot_description/meshes/RFinger32_0.10.stl" scale="0.1 0.1 0.1"/>
 			</geometry>
 			<origin rpy="0 0 0" xyz="0 0 0"/>
@@ -147,11 +147,11 @@
 		<visual>
 			<geometry>
-				<mesh filename="package://pepper_robot/meshes/LFinger13.dae" scale="0.1 0.1 0.1"/>
-			</geometry>
-			<origin rpy="0 0 0" xyz="0 0 0"/>
-		</visual>
-		<collision>
-			<geometry>
-				<mesh filename="package://pepper_robot/meshes/LFinger13_0.10.stl" scale="0.1 0.1 0.1"/>
+				<mesh filename="package://pepper_robot_description/meshes/LFinger13.dae" scale="0.1 0.1 0.1"/>
+			</geometry>
+			<origin rpy="0 0 0" xyz="0 0 0"/>
+		</visual>
+		<collision>
+			<geometry>
+				<mesh filename="package://pepper_robot_description/meshes/LFinger13_0.10.stl" scale="0.1 0.1 0.1"/>
 			</geometry>
 			<origin rpy="0 0 0" xyz="0 0 0"/>
@@ -161,11 +161,11 @@
 		<visual>
 			<geometry>
-				<mesh filename="package://pepper_robot/meshes/LFinger32.dae" scale="0.1 0.1 0.1"/>
-			</geometry>
-			<origin rpy="0 0 0" xyz="0 0 0"/>
-		</visual>
-		<collision>
-			<geometry>
-				<mesh filename="package://pepper_robot/meshes/LFinger32_0.10.stl" scale="0.1 0.1 0.1"/>
+				<mesh filename="package://pepper_robot_description/meshes/LFinger32.dae" scale="0.1 0.1 0.1"/>
+			</geometry>
+			<origin rpy="0 0 0" xyz="0 0 0"/>
+		</visual>
+		<collision>
+			<geometry>
+				<mesh filename="package://pepper_robot_description/meshes/LFinger32_0.10.stl" scale="0.1 0.1 0.1"/>
 			</geometry>
 			<origin rpy="0 0 0" xyz="0 0 0"/>
@@ -175,11 +175,11 @@
 		<visual>
 			<geometry>
-				<mesh filename="package://pepper_robot/meshes/LThumb1.dae" scale="0.1 0.1 0.1"/>
-			</geometry>
-			<origin rpy="0 0 0" xyz="0 0 0"/>
-		</visual>
-		<collision>
-			<geometry>
-				<mesh filename="package://pepper_robot/meshes/LThumb1_0.10.stl" scale="0.1 0.1 0.1"/>
+				<mesh filename="package://pepper_robot_description/meshes/LThumb1.dae" scale="0.1 0.1 0.1"/>
+			</geometry>
+			<origin rpy="0 0 0" xyz="0 0 0"/>
+		</visual>
+		<collision>
+			<geometry>
+				<mesh filename="package://pepper_robot_description/meshes/LThumb1_0.10.stl" scale="0.1 0.1 0.1"/>
 			</geometry>
 			<origin rpy="0 0 0" xyz="0 0 0"/>
@@ -189,11 +189,11 @@
 		<visual>
 			<geometry>
-				<mesh filename="package://pepper_robot/meshes/LFinger11.dae" scale="0.1 0.1 0.1"/>
-			</geometry>
-			<origin rpy="0 0 0" xyz="0 0 0"/>
-		</visual>
-		<collision>
-			<geometry>
-				<mesh filename="package://pepper_robot/meshes/LFinger11_0.10.stl" scale="0.1 0.1 0.1"/>
+				<mesh filename="package://pepper_robot_description/meshes/LFinger11.dae" scale="0.1 0.1 0.1"/>
+			</geometry>
+			<origin rpy="0 0 0" xyz="0 0 0"/>
+		</visual>
+		<collision>
+			<geometry>
+				<mesh filename="package://pepper_robot_description/meshes/LFinger11_0.10.stl" scale="0.1 0.1 0.1"/>
 			</geometry>
 			<origin rpy="0 0 0" xyz="0 0 0"/>
@@ -203,11 +203,11 @@
 		<visual>
 			<geometry>
-				<mesh filename="package://pepper_robot/meshes/RFinger22.dae" scale="0.1 0.1 0.1"/>
-			</geometry>
-			<origin rpy="0 0 0" xyz="0 0 0"/>
-		</visual>
-		<collision>
-			<geometry>
-				<mesh filename="package://pepper_robot/meshes/RFinger22_0.10.stl" scale="0.1 0.1 0.1"/>
+				<mesh filename="package://pepper_robot_description/meshes/RFinger22.dae" scale="0.1 0.1 0.1"/>
+			</geometry>
+			<origin rpy="0 0 0" xyz="0 0 0"/>
+		</visual>
+		<collision>
+			<geometry>
+				<mesh filename="package://pepper_robot_description/meshes/RFinger22_0.10.stl" scale="0.1 0.1 0.1"/>
 			</geometry>
 			<origin rpy="0 0 0" xyz="0 0 0"/>
@@ -217,11 +217,11 @@
 		<visual>
 			<geometry>
-				<mesh filename="package://pepper_robot/meshes/RThumb2.dae" scale="0.1 0.1 0.1"/>
-			</geometry>
-			<origin rpy="0 0 0" xyz="0 0 0"/>
-		</visual>
-		<collision>
-			<geometry>
-				<mesh filename="package://pepper_robot/meshes/RThumb2_0.10.stl" scale="0.1 0.1 0.1"/>
+				<mesh filename="package://pepper_robot_description/meshes/RThumb2.dae" scale="0.1 0.1 0.1"/>
+			</geometry>
+			<origin rpy="0 0 0" xyz="0 0 0"/>
+		</visual>
+		<collision>
+			<geometry>
+				<mesh filename="package://pepper_robot_description/meshes/RThumb2_0.10.stl" scale="0.1 0.1 0.1"/>
 			</geometry>
 			<origin rpy="0 0 0" xyz="0 0 0"/>
@@ -231,11 +231,11 @@
 		<visual>
 			<geometry>
-				<mesh filename="package://pepper_robot/meshes/RFinger13.dae" scale="0.1 0.1 0.1"/>
-			</geometry>
-			<origin rpy="0 0 0" xyz="0 0 0"/>
-		</visual>
-		<collision>
-			<geometry>
-				<mesh filename="package://pepper_robot/meshes/RFinger13_0.10.stl" scale="0.1 0.1 0.1"/>
+				<mesh filename="package://pepper_robot_description/meshes/RFinger13.dae" scale="0.1 0.1 0.1"/>
+			</geometry>
+			<origin rpy="0 0 0" xyz="0 0 0"/>
+		</visual>
+		<collision>
+			<geometry>
+				<mesh filename="package://pepper_robot_description/meshes/RFinger13_0.10.stl" scale="0.1 0.1 0.1"/>
 			</geometry>
 			<origin rpy="0 0 0" xyz="0 0 0"/>
@@ -245,11 +245,11 @@
 		<visual>
 			<geometry>
-				<mesh filename="package://pepper_robot/meshes/KneePitch.dae" scale="0.1 0.1 0.1"/>
-			</geometry>
-			<origin rpy="0 0 0" xyz="0 0 0"/>
-		</visual>
-		<collision>
-			<geometry>
-				<mesh filename="package://pepper_robot/meshes/KneePitch_0.10.stl" scale="0.1 0.1 0.1"/>
+				<mesh filename="package://pepper_robot_description/meshes/KneePitch.dae" scale="0.1 0.1 0.1"/>
+			</geometry>
+			<origin rpy="0 0 0" xyz="0 0 0"/>
+		</visual>
+		<collision>
+			<geometry>
+				<mesh filename="package://pepper_robot_description/meshes/KneePitch_0.10.stl" scale="0.1 0.1 0.1"/>
 			</geometry>
 			<origin rpy="0 0 0" xyz="0 0 0"/>
@@ -259,11 +259,11 @@
 		<visual>
 			<geometry>
-				<mesh filename="package://pepper_robot/meshes/HeadPitch.dae" scale="0.1 0.1 0.1"/>
-			</geometry>
-			<origin rpy="0 0 0" xyz="0 0 0"/>
-		</visual>
-		<collision>
-			<geometry>
-				<mesh filename="package://pepper_robot/meshes/HeadPitch_0.10.stl" scale="0.1 0.1 0.1"/>
+				<mesh filename="package://pepper_robot_description/meshes/HeadPitch.dae" scale="0.1 0.1 0.1"/>
+			</geometry>
+			<origin rpy="0 0 0" xyz="0 0 0"/>
+		</visual>
+		<collision>
+			<geometry>
+				<mesh filename="package://pepper_robot_description/meshes/HeadPitch_0.10.stl" scale="0.1 0.1 0.1"/>
 			</geometry>
 			<origin rpy="0 0 0" xyz="0 0 0"/>
@@ -273,11 +273,11 @@
 		<visual>
 			<geometry>
-				<mesh filename="package://pepper_robot/meshes/LFinger22.dae" scale="0.1 0.1 0.1"/>
-			</geometry>
-			<origin rpy="0 0 0" xyz="0 0 0"/>
-		</visual>
-		<collision>
-			<geometry>
-				<mesh filename="package://pepper_robot/meshes/LFinger22_0.10.stl" scale="0.1 0.1 0.1"/>
+				<mesh filename="package://pepper_robot_description/meshes/LFinger22.dae" scale="0.1 0.1 0.1"/>
+			</geometry>
+			<origin rpy="0 0 0" xyz="0 0 0"/>
+		</visual>
+		<collision>
+			<geometry>
+				<mesh filename="package://pepper_robot_description/meshes/LFinger22_0.10.stl" scale="0.1 0.1 0.1"/>
 			</geometry>
 			<origin rpy="0 0 0" xyz="0 0 0"/>
@@ -287,11 +287,11 @@
 		<visual>
 			<geometry>
-				<mesh filename="package://pepper_robot/meshes/RFinger21.dae" scale="0.1 0.1 0.1"/>
-			</geometry>
-			<origin rpy="0 0 0" xyz="0 0 0"/>
-		</visual>
-		<collision>
-			<geometry>
-				<mesh filename="package://pepper_robot/meshes/RFinger21_0.10.stl" scale="0.1 0.1 0.1"/>
+				<mesh filename="package://pepper_robot_description/meshes/RFinger21.dae" scale="0.1 0.1 0.1"/>
+			</geometry>
+			<origin rpy="0 0 0" xyz="0 0 0"/>
+		</visual>
+		<collision>
+			<geometry>
+				<mesh filename="package://pepper_robot_description/meshes/RFinger21_0.10.stl" scale="0.1 0.1 0.1"/>
 			</geometry>
 			<origin rpy="0 0 0" xyz="0 0 0"/>
@@ -301,11 +301,11 @@
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