Commit message: fix urdf

File: pepper_robot_description/urdf/pepper_robot.urdf (robot description, URDF)
Before this commit: robot pepper_robot, 83 links, 83 joints
Links:
- link Tibia: mass None -> 11.6015; geometry collision mesh filename=package://pepper_robot_description/pepper_robot/meshes/Knee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 scale=0.1 0.1 0.1; visual mesh filename=package://pepper_robot_description/pepper_robot/meshes/Knee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 scale=0.1 0.1 0.1
Joints:
- removed joint torso_joint
- joint base_link_fixedjoint: child base_link -> torso; parent base_footprint -> base_link

Commit message: change base_link to the base of the robot

File: pepper_robot_description/urdf/pepper_robot.urdf (robot description, URDF)
Before this commit: robot pepper_robot, 83 links, 82 joints
Joints:
- joint base_link_fixedjoint: origin xyz=0 0 0 rpy=0 0 0 -> xyz=-0.038 0 -0.82 rpy=0 0 0

Commit message: change base_link to the base of the robot

File: pepper_robot_description/urdf/pepper_robot.urdf (robot description, URDF)
Before this commit: robot pepper_robot, 83 links, 82 joints
Joints:
- joint base_link_fixedjoint: origin xyz=-0.038 0 -0.82 rpy=0 0 0 -> xyz=0.038 0 0.82 rpy=0 0 0

Commit message: change base_link to the base of the robot

File: pepper_robot_description/urdf/pepper_robot.urdf (robot description, URDF)
Before this commit: robot pepper_robot, 83 links, 82 joints
Joints:
- joint base_link_fixedjoint: origin xyz=0.038 0 0.82 rpy=0 0 0 -> xyz=0 0 0.82 rpy=0 0 0

Commit message: change base_link to the base of the robot

File: pepper_robot_description/urdf/pepper_robot.urdf (robot description, URDF)
Before this commit: robot pepper_robot, 83 links, 82 joints
Joints:
- joint base_link_fixedjoint: origin xyz=0 0 0.82 rpy=0 0 0 -> xyz=0 0 0 rpy=0 0 0

Commit message: fix urdf root_link

File: pepper_robot_description/urdf/pepper_robot.urdf (robot description, URDF)
Before this commit: robot pepper_robot, 83 links, 82 joints
Links:
- removed link base_link
Joints:
- removed joint base_link_fixedjoint
- joint HipPitch: child Pelvis -> Hip; parent Hip -> Pelvis
- joint HipRoll: child Hip -> torso; parent torso -> Hip
- joint KneePitch: child Tibia -> Pelvis; parent Pelvis -> Tibia
- joint base_footprint_joint: child base_footprint -> Tibia; parent Tibia -> base_footprint

Commit message: fix urdf root_link

File: pepper_robot_description/urdf/pepper_robot.urdf (robot description, URDF)
Before this commit: robot pepper_robot, 82 links, 81 joints
Links:
- removed link base_footprint
- added link base_link
Joints:
- removed joint base_footprint_joint
- added joint base_link_fixedjoint: type fixed, parent base_link, child Tibia, origin xyz=0 0 0 rpy=0 0 0, axis 0 0 0

Commit message: fix urdf root_link

File: pepper_robot_description/urdf/pepper_robot.urdf (robot description, URDF)
Before this commit: robot pepper_robot, 82 links, 81 joints
Links:
- removed link BumperB_frame
- removed link BumperFL_frame
- removed link BumperFR_frame
- removed link CameraBottom_frame
- removed link CameraBottom_optical_frame
- removed link CameraDepth_frame
- removed link CameraDepth_optical_frame
- removed link CameraTop_frame
- removed link CameraTop_optical_frame
- removed link ChestButton_frame
- removed link HeadTouchFront_frame
- removed link HeadTouchMiddle_frame
- removed link HeadTouchRear_frame
- removed link ImuBaseAccelerometer_frame
- removed link ImuTorsoAccelerometer_frame
- removed link ImuTorsoGyrometer_frame
- removed link LHandTouchBack_frame
- removed link LSpeaker_frame
- removed link RHandTouchBack_frame
- removed link RSpeaker_frame
- removed link ShovelLaser_frame
- removed link SonarBack_frame
- removed link SonarFront_frame
- removed link SurroundingFrontLaser_device_frame
- removed link SurroundingFrontLaser_frame
- removed link SurroundingLeftLaser_device_frame
- removed link SurroundingLeftLaser_frame
- removed link SurroundingRightLaser_device_frame
- removed link SurroundingRightLaser_frame
- removed link Tablet_frame
- removed link VerticalLeftLaser_frame
- removed link VerticalRightLaser_frame
Joints:
- removed joint AccelerometerBase_sensor_fixedjoint
- removed joint Accelerometer_sensor_fixedjoint
- removed joint Bumper/Back_sensor_fixedjoint
- removed joint Bumper/FrontLeft_sensor_fixedjoint
- removed joint Bumper/FrontRight_sensor_fixedjoint
- removed joint CameraBottom_optical_frame_fixedjoint
- removed joint CameraBottom_sensor_fixedjoint
- removed joint CameraDepth_optical_frame_fixedjoint
- removed joint CameraDepth_sensor_fixedjoint
- removed joint CameraTop_optical_frame_fixedjoint
- removed joint CameraTop_sensor_fixedjoint
- removed joint ChestBoard/Button_sensor_fixedjoint
- removed joint Gyrometer_sensor_fixedjoint
- removed joint Head/Touch/Front_sensor_fixedjoint
- removed joint Head/Touch/Middle_sensor_fixedjoint
- removed joint Head/Touch/Rear_sensor_fixedjoint
- removed joint LHand/Touch/Back_sensor_fixedjoint
- removed joint LaserSensor/Front_projected_sensor_fixedjoint
- removed joint LaserSensor/Front_sensor_fixedjoint
- removed joint LaserSensor/Left_projected_sensor_fixedjoint
- removed joint LaserSensor/Left_sensor_fixedjoint
- removed joint LaserSensor/Right_projected_sensor_fixedjoint
- removed joint LaserSensor/Right_sensor_fixedjoint
- removed joint LaserSensor/Shovel_sensor_fixedjoint
- removed joint LaserSensor/VerticalLeft_sensor_fixedjoint
- removed joint LaserSensor/VerticalRight_sensor_fixedjoint
- removed joint RHand/Touch/Back_sensor_fixedjoint
- removed joint Sonar/Back_sensor_fixedjoint
- removed joint Sonar/Front_sensor_fixedjoint
- removed joint SpeakerLeft_sensor_fixedjoint
- removed joint SpeakerRight_sensor_fixedjoint
- removed joint Tablet_sensor_fixedjoint

Commit message: fix urdf root_link

File: pepper_robot_description/urdf/pepper_robot.urdf (robot description, URDF)
Before this commit: robot pepper_robot, 50 links, 49 joints
Joints:
- joint base_link_fixedjoint: origin xyz=0 0 0 rpy=0 0 0 -> xyz=0 0 0.334 rpy=0 0 0

Commit message: fix urdf root_link

File: pepper_robot_description/urdf/pepper_robot.urdf (robot description, URDF)
Before this commit: robot pepper_robot, 50 links, 49 joints
Joints:
- joint HeadYaw: origin xyz=-0.038 0 0.1699 rpy=0 0 0 -> xyz=-0.038 0 0.3089 rpy=0 0 0
- joint HipPitch: axis 0 1.0 0 -> 0 -1.0 0; origin xyz=0 0 -0.079 rpy=0 0 0 -> xyz=0 0 0.268 rpy=0 0 0
- joint HipRoll: axis 1.0 0 0 -> -1.0 0 0; origin xyz=2e-05 0 -0.139 rpy=0 0 0 -> xyz=2e-05 0 0.079 rpy=0 0 0
- joint KneePitch: axis 0 1.0 0 -> 0 -1.0 0; origin xyz=0 0 -0.268 rpy=0 0 0 -> xyz=0 0 0 rpy=0 0 0
- joint LShoulderPitch: origin xyz=-0.057 0.14974 0.08682 rpy=0 0 0 -> xyz=-0.057 0.14974 0.22582 rpy=0 0 0
- joint RShoulderPitch: origin xyz=-0.057 -0.14974 0.08682 rpy=0 0 0 -> xyz=-0.057 -0.14974 0.22582 rpy=0 0 0

Commit message: fix urdf root_link

File: pepper_robot_description/urdf/pepper_robot.urdf (robot description, URDF)
Before this commit: robot pepper_robot, 50 links, 49 joints
Joints:
- joint HipRoll: origin xyz=2e-05 0 0.079 rpy=0 0 0 -> xyz=0 0 0.079 rpy=0 0 0

Commit message: add base_footprint

File: pepper_robot_description/urdf/pepper_robot.urdf (robot description, URDF)
Before this commit: robot pepper_robot, 50 links, 49 joints
Links:
- added link base_footprint
Joints:
- added joint base_footprint_joint: type fixed, parent base_footprint, child base_link, origin xyz=0 0 0.334 rpy=0 0 0

Commit message: add base_footprint

File: pepper_robot_description/urdf/pepper_robot.urdf (robot description, URDF)
Before this commit: robot pepper_robot, 51 links, 50 joints
Joints:
- joint base_footprint_joint: child base_link -> Tibia; parent base_footprint -> base_link
- joint base_link_fixedjoint: child Tibia -> base_link; parent base_link -> base_footprint

Commit message: fix base_footprint

File: pepper_robot_description/urdf/pepper_robot.urdf (robot description, URDF)
Before this commit: robot pepper_robot, 51 links, 50 joints
Joints:
- joint base_footprint_joint: origin xyz=0 0 0.334 rpy=0 0 0 -> xyz=0 0 0 rpy=0 0 0

Commit message: fix base_footprint

File: pepper_robot_description/urdf/pepper_robot.urdf (robot description, URDF)
Before this commit: robot pepper_robot, 51 links, 50 joints
Joints:
- joint base_link_fixedjoint: origin xyz=0 0 0.334 rpy=0 0 0 -> xyz=0 0 0 rpy=0 0 0

Commit message: fix base_footprint

File: pepper_robot_description/urdf/pepper_robot.urdf (robot description, URDF)
Before this commit: robot pepper_robot, 51 links, 50 joints
Joints:
- joint base_footprint_joint: child Tibia -> base_link; parent base_link -> base_footprint
- joint base_link_fixedjoint: child base_link -> Tibia; parent base_footprint -> base_link

Commit message: fix base_footprint

File: pepper_robot_description/urdf/pepper_robot.urdf (robot description, URDF)
Before this commit: robot pepper_robot, 51 links, 50 joints
Joints:
- joint base_footprint_joint: origin xyz=0 0 0 rpy=0 0 0 -> xyz=0 0 0.334 rpy=0 0 0
- joint base_link_fixedjoint: origin xyz=0 0 0 rpy=0 0 0 -> xyz=0 0 0.334 rpy=0 0 0

Commit message: test mechanical stuff urdf

File: pepper_robot_description/urdf/pepper_robot.urdf (robot description, URDF)
Before this commit: robot pepper_robot, 51 links, 50 joints
Links:
- link Hip: mass 1.02338 -> 10.02338

Commit message: test inertia urdf

File: pepper_robot_description/urdf/pepper_robot.urdf (robot description, URDF)
Before this commit: robot pepper_robot, 51 links, 50 joints
Links:
- link Hip: mass 10.02338 -> 1.02338
