Commit message: test inertia

File: pepper_robot_description/urdf/pepper_robot.urdf (robot description, URDF)
Before this commit: robot pepper_robot, 51 links, 50 joints
Links:
- added link BumperB_frame
- added link BumperFL_frame
- added link BumperFR_frame
- added link CameraBottom_frame
- added link CameraBottom_optical_frame
- added link CameraDepth_frame
- added link CameraDepth_optical_frame
- added link CameraTop_frame
- added link CameraTop_optical_frame
- added link ChestButton_frame
- added link HeadTouchFront_frame
- added link HeadTouchMiddle_frame
- added link HeadTouchRear_frame
- added link ImuBaseAccelerometer_frame
- added link ImuTorsoAccelerometer_frame
- added link ImuTorsoGyrometer_frame
- added link LHandTouchBack_frame
- added link LSpeaker_frame
- added link RHandTouchBack_frame
- added link RSpeaker_frame
- added link ShovelLaser_frame
- added link SonarBack_frame
- added link SonarFront_frame
- added link SurroundingFrontLaser_device_frame
- added link SurroundingFrontLaser_frame
- added link SurroundingLeftLaser_device_frame
- added link SurroundingLeftLaser_frame
- added link SurroundingRightLaser_device_frame
- added link SurroundingRightLaser_frame
- added link Tablet_frame
- added link VerticalLeftLaser_frame
- added link VerticalRightLaser_frame
- link Head: geometry collision mesh filename=package://pepper_robot_description/pepper_robot/meshes/1.0/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 scale=0.1 0.1 0.1; visual mesh filename=package://pepper_robot_description/pepper_robot/meshes/1.0/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 scale=0.1 0.1 0.1
- link Hip: geometry collision mesh filename=package://pepper_robot_description/pepper_robot/meshes/1.0/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 scale=0.1 0.1 0.1; visual mesh filename=package://pepper_robot_description/pepper_robot/meshes/1.0/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 scale=0.1 0.1 0.1
- link LBicep: geometry collision mesh filename=package://pepper_robot_description/pepper_robot/meshes/1.0/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 scale=0.1 0.1 0.1; visual mesh filename=package://pepper_robot_description/pepper_robot/meshes/1.0/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 scale=0.1 0.1 0.1
- link LElbow: geometry collision mesh filename=package://pepper_robot_description/pepper_robot/meshes/1.0/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 scale=0.1 0.1 0.1; visual mesh filename=package://pepper_robot_description/pepper_robot/meshes/1.0/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 scale=0.1 0.1 0.1
- link LFinger11_link: geometry collision mesh filename=package://pepper_robot_description/pepper_robot/meshes/1.0/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 scale=0.1 0.1 0.1; visual mesh filename=package://pepper_robot_description/pepper_robot/meshes/1.0/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 scale=0.1 0.1 0.1
- link LFinger12_link: geometry collision mesh filename=package://pepper_robot_description/pepper_robot/meshes/1.0/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 scale=0.1 0.1 0.1; visual mesh filename=package://pepper_robot_description/pepper_robot/meshes/1.0/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 scale=0.1 0.1 0.1
- link LFinger13_link: geometry collision mesh filename=package://pepper_robot_description/pepper_robot/meshes/1.0/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 scale=0.1 0.1 0.1; visual mesh filename=package://pepper_robot_description/pepper_robot/meshes/1.0/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 scale=0.1 0.1 0.1
- link LFinger21_link: geometry collision mesh filename=package://pepper_robot_description/pepper_robot/meshes/1.0/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 scale=0.1 0.1 0.1; visual mesh filename=package://pepper_robot_description/pepper_robot/meshes/1.0/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 scale=0.1 0.1 0.1
- link LFinger22_link: geometry collision mesh filename=package://pepper_robot_description/pepper_robot/meshes/1.0/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 scale=0.1 0.1 0.1; visual mesh filename=package://pepper_robot_description/pepper_robot/meshes/1.0/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 scale=0.1 0.1 0.1
- link LFinger23_link: geometry collision mesh filename=package://pepper_robot_description/pepper_robot/meshes/1.0/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 scale=0.1 0.1 0.1; visual mesh filename=package://pepper_robot_description/pepper_robot/meshes/1.0/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 scale=0.1 0.1 0.1
- link LFinger31_link: geometry collision mesh filename=package://pepper_robot_description/pepper_robot/meshes/1.0/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 scale=0.1 0.1 0.1; visual mesh filename=package://pepper_robot_description/pepper_robot/meshes/1.0/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 scale=0.1 0.1 0.1
- link LFinger32_link: geometry collision mesh filename=package://pepper_robot_description/pepper_robot/meshes/1.0/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 scale=0.1 0.1 0.1; visual mesh filename=package://pepper_robot_description/pepper_robot/meshes/1.0/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 scale=0.1 0.1 0.1
- link LFinger33_link: geometry collision mesh filename=package://pepper_robot_description/pepper_robot/meshes/1.0/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 scale=0.1 0.1 0.1; visual mesh filename=package://pepper_robot_description/pepper_robot/meshes/1.0/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 scale=0.1 0.1 0.1
- link LFinger41_link: geometry collision mesh filename=package://pepper_robot_description/pepper_robot/meshes/1.0/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 scale=0.1 0.1 0.1; visual mesh filename=package://pepper_robot_description/pepper_robot/meshes/1.0/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 scale=0.1 0.1 0.1
- link LFinger42_link: geometry collision mesh filename=package://pepper_robot_description/pepper_robot/meshes/1.0/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 scale=0.1 0.1 0.1; visual mesh filename=package://pepper_robot_description/pepper_robot/meshes/1.0/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 scale=0.1 0.1 0.1
- link LFinger43_link: geometry collision mesh filename=package://pepper_robot_description/pepper_robot/meshes/1.0/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 scale=0.1 0.1 0.1; visual mesh filename=package://pepper_robot_description/pepper_robot/meshes/1.0/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 scale=0.1 0.1 0.1
- link LForeArm: geometry collision mesh filename=package://pepper_robot_description/pepper_robot/meshes/1.0/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 scale=0.1 0.1 0.1; visual mesh filename=package://pepper_robot_description/pepper_robot/meshes/1.0/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 scale=0.1 0.1 0.1
- link LShoulder: geometry collision mesh filename=package://pepper_robot_description/pepper_robot/meshes/1.0/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 scale=0.1 0.1 0.1; visual mesh filename=package://pepper_robot_description/pepper_robot/meshes/1.0/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 scale=0.1 0.1 0.1
- link LThumb1_link: geometry collision mesh filename=package://pepper_robot_description/pepper_robot/meshes/1.0/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 scale=0.1 0.1 0.1; visual mesh filename=package://pepper_robot_description/pepper_robot/meshes/1.0/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 scale=0.1 0.1 0.1
- link LThumb2_link: geometry collision mesh filename=package://pepper_robot_description/pepper_robot/meshes/1.0/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 scale=0.1 0.1 0.1; visual mesh filename=package://pepper_robot_description/pepper_robot/meshes/1.0/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 scale=0.1 0.1 0.1
- link Neck: geometry collision mesh filename=package://pepper_robot_description/pepper_robot/meshes/1.0/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 scale=0.1 0.1 0.1; visual mesh filename=package://pepper_robot_description/pepper_robot/meshes/1.0/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 scale=0.1 0.1 0.1
- link Pelvis: geometry collision mesh filename=package://pepper_robot_description/pepper_robot/meshes/1.0/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 scale=0.1 0.1 0.1; visual mesh filename=package://pepper_robot_description/pepper_robot/meshes/1.0/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 scale=0.1 0.1 0.1
- link RBicep: geometry collision mesh filename=package://pepper_robot_description/pepper_robot/meshes/1.0/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 scale=0.1 0.1 0.1; visual mesh filename=package://pepper_robot_description/pepper_robot/meshes/1.0/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 scale=0.1 0.1 0.1
- link RElbow: geometry collision mesh filename=package://pepper_robot_description/pepper_robot/meshes/1.0/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 scale=0.1 0.1 0.1; visual mesh filename=package://pepper_robot_description/pepper_robot/meshes/1.0/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 scale=0.1 0.1 0.1
- link RFinger11_link: geometry collision mesh filename=package://pepper_robot_description/pepper_robot/meshes/1.0/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 scale=0.1 0.1 0.1; visual mesh filename=package://pepper_robot_description/pepper_robot/meshes/1.0/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 scale=0.1 0.1 0.1
- link RFinger12_link: geometry collision mesh filename=package://pepper_robot_description/pepper_robot/meshes/1.0/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 scale=0.1 0.1 0.1; visual mesh filename=package://pepper_robot_description/pepper_robot/meshes/1.0/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 scale=0.1 0.1 0.1
- link RFinger13_link: geometry collision mesh filename=package://pepper_robot_description/pepper_robot/meshes/1.0/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 scale=0.1 0.1 0.1; visual mesh filename=package://pepper_robot_description/pepper_robot/meshes/1.0/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 scale=0.1 0.1 0.1
- link RFinger21_link: geometry collision mesh filename=package://pepper_robot_description/pepper_robot/meshes/1.0/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 scale=0.1 0.1 0.1; visual mesh filename=package://pepper_robot_description/pepper_robot/meshes/1.0/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 scale=0.1 0.1 0.1
- link RFinger22_link: geometry collision mesh filename=package://pepper_robot_description/pepper_robot/meshes/1.0/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 scale=0.1 0.1 0.1; visual mesh filename=package://pepper_robot_description/pepper_robot/meshes/1.0/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 scale=0.1 0.1 0.1
- link RFinger23_link: geometry collision mesh filename=package://pepper_robot_description/pepper_robot/meshes/1.0/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 scale=0.1 0.1 0.1; visual mesh filename=package://pepper_robot_description/pepper_robot/meshes/1.0/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 scale=0.1 0.1 0.1
- link RFinger31_link: geometry collision mesh filename=package://pepper_robot_description/pepper_robot/meshes/1.0/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 scale=0.1 0.1 0.1; visual mesh filename=package://pepper_robot_description/pepper_robot/meshes/1.0/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 scale=0.1 0.1 0.1
- link RFinger32_link: geometry collision mesh filename=package://pepper_robot_description/pepper_robot/meshes/1.0/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 scale=0.1 0.1 0.1; visual mesh filename=package://pepper_robot_description/pepper_robot/meshes/1.0/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 scale=0.1 0.1 0.1
- link RFinger33_link: geometry collision mesh filename=package://pepper_robot_description/pepper_robot/meshes/1.0/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 scale=0.1 0.1 0.1; visual mesh filename=package://pepper_robot_description/pepper_robot/meshes/1.0/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 scale=0.1 0.1 0.1
- link RFinger41_link: geometry collision mesh filename=package://pepper_robot_description/pepper_robot/meshes/1.0/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 scale=0.1 0.1 0.1; visual mesh filename=package://pepper_robot_description/pepper_robot/meshes/1.0/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 scale=0.1 0.1 0.1
- link RFinger42_link: geometry collision mesh filename=package://pepper_robot_description/pepper_robot/meshes/1.0/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 scale=0.1 0.1 0.1; visual mesh filename=package://pepper_robot_description/pepper_robot/meshes/1.0/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 scale=0.1 0.1 0.1
- link RFinger43_link: geometry collision mesh filename=package://pepper_robot_description/pepper_robot/meshes/1.0/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 scale=0.1 0.1 0.1; visual mesh filename=package://pepper_robot_description/pepper_robot/meshes/1.0/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 scale=0.1 0.1 0.1
- link RForeArm: geometry collision mesh filename=package://pepper_robot_description/pepper_robot/meshes/1.0/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 scale=0.1 0.1 0.1; visual mesh filename=package://pepper_robot_description/pepper_robot/meshes/1.0/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 scale=0.1 0.1 0.1
- link RShoulder: geometry collision mesh filename=package://pepper_robot_description/pepper_robot/meshes/1.0/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 scale=0.1 0.1 0.1; visual mesh filename=package://pepper_robot_description/pepper_robot/meshes/1.0/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 scale=0.1 0.1 0.1
- link RThumb1_link: geometry collision mesh filename=package://pepper_robot_description/pepper_robot/meshes/1.0/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 scale=0.1 0.1 0.1; visual mesh filename=package://pepper_robot_description/pepper_robot/meshes/1.0/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 scale=0.1 0.1 0.1
- link RThumb2_link: geometry collision mesh filename=package://pepper_robot_description/pepper_robot/meshes/1.0/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 scale=0.1 0.1 0.1; visual mesh filename=package://pepper_robot_description/pepper_robot/meshes/1.0/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 scale=0.1 0.1 0.1
- link Tibia: geometry collision mesh filename=package://pepper_robot_description/pepper_robot/meshes/1.0/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 scale=0.1 0.1 0.1; visual mesh filename=package://pepper_robot_description/pepper_robot/meshes/1.0/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 scale=0.1 0.1 0.1
- link WheelB_link: geometry collision mesh filename=package://pepper_robot_description/pepper_robot/meshes/1.0/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 scale=0.1 0.1 0.1; visual mesh filename=package://pepper_robot_description/pepper_robot/meshes/1.0/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 scale=0.1 0.1 0.1
- link WheelFL_link: geometry collision mesh filename=package://pepper_robot_description/pepper_robot/meshes/1.0/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 scale=0.1 0.1 0.1; visual mesh filename=package://pepper_robot_description/pepper_robot/meshes/1.0/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 scale=0.1 0.1 0.1
- link WheelFR_link: geometry collision mesh filename=package://pepper_robot_description/pepper_robot/meshes/1.0/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 scale=0.1 0.1 0.1; visual mesh filename=package://pepper_robot_description/pepper_robot/meshes/1.0/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 scale=0.1 0.1 0.1
- link l_wrist: geometry collision mesh filename=package://pepper_robot_description/pepper_robot/meshes/1.0/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 scale=0.1 0.1 0.1; visual mesh filename=package://pepper_robot_description/pepper_robot/meshes/1.0/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 scale=0.1 0.1 0.1
- link r_wrist: geometry collision mesh filename=package://pepper_robot_description/pepper_robot/meshes/1.0/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 scale=0.1 0.1 0.1; visual mesh filename=package://pepper_robot_description/pepper_robot/meshes/1.0/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 scale=0.1 0.1 0.1
- link torso: geometry collision mesh filename=package://pepper_robot_description/pepper_robot/meshes/1.0/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 scale=0.1 0.1 0.1; visual mesh filename=package://pepper_robot_description/pepper_robot/meshes/1.0/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 scale=0.1 0.1 0.1
Joints:
- added joint AccelerometerBase_sensor_fixedjoint: type fixed, parent Tibia, child ImuBaseAccelerometer_frame, origin xyz=0.0147 -0.0017 -0.26319 rpy=0 0 0, axis 0 0 0
- added joint Accelerometer_sensor_fixedjoint: type fixed, parent torso, child ImuTorsoAccelerometer_frame, origin xyz=0.00239 -0.03575 0.00626 rpy=0 0 0, axis 0 0 0
- added joint Bumper/Back_sensor_fixedjoint: type fixed, parent Tibia, child BumperB_frame, origin xyz=-0.251 0 -0.264 rpy=0 0 -3.14159, axis 0 0 0
- added joint Bumper/FrontLeft_sensor_fixedjoint: type fixed, parent Tibia, child BumperFL_frame, origin xyz=0.129 0.227 -0.264 rpy=0 0 0.48886, axis 0 0 0
- added joint Bumper/FrontRight_sensor_fixedjoint: type fixed, parent Tibia, child BumperFR_frame, origin xyz=0.129 -0.227 -0.264 rpy=0 0 -0.48886, axis 0 0 0
- added joint CameraBottom_optical_frame_fixedjoint: type fixed, parent CameraBottom_frame, child CameraBottom_optical_frame, origin xyz=0 0 0 rpy=-1.57079632679 0 -1.57079632679
- added joint CameraBottom_sensor_fixedjoint: type fixed, parent Head, child CameraBottom_frame, origin xyz=0.09262 0 0.06177 rpy=0 0.698132 0, axis 0 0 0
- added joint CameraDepth_optical_frame_fixedjoint: type fixed, parent CameraDepth_frame, child CameraDepth_optical_frame, origin xyz=0 0 0 rpy=-1.57079632679 0 -1.57079632679
- added joint CameraDepth_sensor_fixedjoint: type fixed, parent Head, child CameraDepth_frame, origin xyz=0.05138 0.039 0.1194 rpy=0 0 0, axis 0 0 0
- added joint CameraTop_optical_frame_fixedjoint: type fixed, parent CameraTop_frame, child CameraTop_optical_frame, origin xyz=0 0 0 rpy=-1.57079632679 0 -1.57079632679
- added joint CameraTop_sensor_fixedjoint: type fixed, parent Head, child CameraTop_frame, origin xyz=0.08601 0 0.16284 rpy=0 0 0, axis 0 0 0
- added joint ChestBoard/Button_sensor_fixedjoint: type fixed, parent torso, child ChestButton_frame, origin xyz=0.049871 0.001588 0.055163 rpy=0 0 0, axis 0 0 0
- added joint Gyrometer_sensor_fixedjoint: type fixed, parent torso, child ImuTorsoGyrometer_frame, origin xyz=0.00204 -0.03491 -0.00959 rpy=0 0 0, axis 0 0 0
- added joint Head/Touch/Front_sensor_fixedjoint: type fixed, parent Head, child HeadTouchFront_frame, origin xyz=0.028175 0 0.21267 rpy=0 0.20944 0, axis 0 0 0
- added joint Head/Touch/Middle_sensor_fixedjoint: type fixed, parent Head, child HeadTouchMiddle_frame, origin xyz=0.0041 0 0.2159 rpy=0 -0.0349066 0, axis 0 0 0
- added joint Head/Touch/Rear_sensor_fixedjoint: type fixed, parent Head, child HeadTouchRear_frame, origin xyz=-0.03376 0 0.21052 rpy=0 -0.314159 0, axis 0 0 0
- added joint LHand/Touch/Back_sensor_fixedjoint: type fixed, parent l_wrist, child LHandTouchBack_frame, origin xyz=0.0523 0 0.0304 rpy=1.5708 -1.5708 -3.14159, axis 0 0 0
- added joint LaserSensor/Front_projected_sensor_fixedjoint: type fixed, parent Tibia, child SurroundingFrontLaser_frame, origin xyz=0.0562 0 -0.334 rpy=0 0 0, axis 0 0 0
- added joint LaserSensor/Front_sensor_fixedjoint: type fixed, parent Tibia, child SurroundingFrontLaser_device_frame, origin xyz=0.0562 0 -0.0692 rpy=0 0.349066 0, axis 0 0 0
- added joint LaserSensor/Left_projected_sensor_fixedjoint: type fixed, parent Tibia, child SurroundingLeftLaser_frame, origin xyz=-0.018 0.0899 -0.334 rpy=0 0 1.75728, axis 0 0 0
- added joint LaserSensor/Left_sensor_fixedjoint: type fixed, parent Tibia, child SurroundingLeftLaser_device_frame, origin xyz=-0.018 0.0899 -0.0759 rpy=0 0.349066 1.5708, axis 0 0 0
- added joint LaserSensor/Right_projected_sensor_fixedjoint: type fixed, parent Tibia, child SurroundingRightLaser_frame, origin xyz=-0.018 -0.0899 -0.334 rpy=0 0 -1.75728, axis 0 0 0
- added joint LaserSensor/Right_sensor_fixedjoint: type fixed, parent Tibia, child SurroundingRightLaser_device_frame, origin xyz=-0.018 -0.0899 -0.0759 rpy=0 0.349066 -1.5708, axis 0 0 0
- added joint LaserSensor/Shovel_sensor_fixedjoint: type fixed, parent Tibia, child ShovelLaser_frame, origin xyz=0.0562 0 -0.0692 rpy=0 0.349066 0, axis 0 0 0
- added joint LaserSensor/VerticalLeft_sensor_fixedjoint: type fixed, parent Tibia, child VerticalLeftLaser_frame, origin xyz=0.0562 0 -0.0692 rpy=0 0.349066 0, axis 0 0 0
- added joint LaserSensor/VerticalRight_sensor_fixedjoint: type fixed, parent Tibia, child VerticalRightLaser_frame, origin xyz=0.0562 0 -0.0692 rpy=0 0.349066 0, axis 0 0 0
- added joint RHand/Touch/Back_sensor_fixedjoint: type fixed, parent r_wrist, child RHandTouchBack_frame, origin xyz=0.0523 0 0.0304 rpy=1.5708 -1.5708 -3.14159, axis 0 0 0
- added joint Sonar/Back_sensor_fixedjoint: type fixed, parent Tibia, child SonarBack_frame, origin xyz=-0.0718 0 -0.0534 rpy=-1.81761e-08 -0.209438 -3.14159, axis 0 0 0
- added joint Sonar/Front_sensor_fixedjoint: type fixed, parent Tibia, child SonarFront_frame, origin xyz=0.0699 0 -0.1023 rpy=0 -0.322858 0, axis 0 0 0
- added joint SpeakerLeft_sensor_fixedjoint: type fixed, parent Head, child LSpeaker_frame, origin xyz=0 0 0 rpy=0 0 0, axis 0 0 0
- added joint SpeakerRight_sensor_fixedjoint: type fixed, parent Head, child RSpeaker_frame, origin xyz=0 0 0 rpy=0 0 0, axis 0 0 0
- added joint Tablet_sensor_fixedjoint: type fixed, parent torso, child Tablet_frame, origin xyz=0.0839249 0 0.06251 rpy=0 -0.523599 0, axis 0 0 0
- joint HeadPitch: limit lower=-0.706858 upper=0.4451 effort=2.666 velocity=9.22756 -> lower=-0.706858 upper=0.637045 effort=2.666 velocity=9.22756
- joint HeadYaw: origin xyz=-0.038 0 0.3089 rpy=0 0 0 -> xyz=-0.038 0 0.1699 rpy=0 0 0
- joint HipPitch: axis 0 -1.0 0 -> 0 1.0 0; child Hip -> Pelvis; origin xyz=0 0 0.268 rpy=0 0 0 -> xyz=0 0 -0.079 rpy=0 0 0; parent Pelvis -> Hip
- joint HipRoll: axis -1.0 0 0 -> 1.0 0 0; child torso -> Hip; origin xyz=0 0 0.079 rpy=0 0 0 -> xyz=2e-05 0 -0.139 rpy=0 0 0; parent Hip -> torso
- joint KneePitch: axis 0 -1.0 0 -> 0 1.0 0; child Pelvis -> Tibia; origin xyz=0 0 0 rpy=0 0 0 -> xyz=0 0 -0.268 rpy=0 0 0; parent Tibia -> Pelvis
- joint LShoulderPitch: origin xyz=-0.057 0.14974 0.22582 rpy=0 0 0 -> xyz=-0.057 0.14974 0.08682 rpy=0 0 0
- joint RShoulderPitch: origin xyz=-0.057 -0.14974 0.22582 rpy=0 0 0 -> xyz=-0.057 -0.14974 0.08682 rpy=0 0 0
- joint base_footprint_joint: child base_link -> base_footprint; origin xyz=0 0 0 rpy=0 0 0 -> xyz=0 0 -0.334 rpy=0 0 0; parent base_footprint -> Tibia
- joint base_link_fixedjoint: child Tibia -> torso; origin xyz=0 0 0.334 rpy=0 0 0 -> xyz=0 0 0 rpy=0 0 0

Commit message: test inertia

File: pepper_robot_description/urdf/pepper_robot.urdf (robot description, URDF)
Before this commit: robot pepper_robot, 83 links, 82 joints
Links:
- removed link BumperB_frame
- removed link BumperFL_frame
- removed link BumperFR_frame
- removed link CameraBottom_frame
- removed link CameraBottom_optical_frame
- removed link CameraDepth_frame
- removed link CameraDepth_optical_frame
- removed link CameraTop_frame
- removed link CameraTop_optical_frame
- removed link ChestButton_frame
- removed link HeadTouchFront_frame
- removed link HeadTouchMiddle_frame
- removed link HeadTouchRear_frame
- removed link ImuBaseAccelerometer_frame
- removed link ImuTorsoAccelerometer_frame
- removed link ImuTorsoGyrometer_frame
- removed link LHandTouchBack_frame
- removed link LSpeaker_frame
- removed link RHandTouchBack_frame
- removed link RSpeaker_frame
- removed link ShovelLaser_frame
- removed link SonarBack_frame
- removed link SonarFront_frame
- removed link SurroundingFrontLaser_device_frame
- removed link SurroundingFrontLaser_frame
- removed link SurroundingLeftLaser_device_frame
- removed link SurroundingLeftLaser_frame
- removed link SurroundingRightLaser_device_frame
- removed link SurroundingRightLaser_frame
- removed link Tablet_frame
- removed link VerticalLeftLaser_frame
- removed link VerticalRightLaser_frame
Joints:
- removed joint AccelerometerBase_sensor_fixedjoint
- removed joint Accelerometer_sensor_fixedjoint
- removed joint Bumper/Back_sensor_fixedjoint
- removed joint Bumper/FrontLeft_sensor_fixedjoint
- removed joint Bumper/FrontRight_sensor_fixedjoint
- removed joint CameraBottom_optical_frame_fixedjoint
- removed joint CameraBottom_sensor_fixedjoint
- removed joint CameraDepth_optical_frame_fixedjoint
- removed joint CameraDepth_sensor_fixedjoint
- removed joint CameraTop_optical_frame_fixedjoint
- removed joint CameraTop_sensor_fixedjoint
- removed joint ChestBoard/Button_sensor_fixedjoint
- removed joint Gyrometer_sensor_fixedjoint
- removed joint Head/Touch/Front_sensor_fixedjoint
- removed joint Head/Touch/Middle_sensor_fixedjoint
- removed joint Head/Touch/Rear_sensor_fixedjoint
- removed joint LHand/Touch/Back_sensor_fixedjoint
- removed joint LaserSensor/Front_projected_sensor_fixedjoint
- removed joint LaserSensor/Front_sensor_fixedjoint
- removed joint LaserSensor/Left_projected_sensor_fixedjoint
- removed joint LaserSensor/Left_sensor_fixedjoint
- removed joint LaserSensor/Right_projected_sensor_fixedjoint
- removed joint LaserSensor/Right_sensor_fixedjoint
- removed joint LaserSensor/Shovel_sensor_fixedjoint
- removed joint LaserSensor/VerticalLeft_sensor_fixedjoint
- removed joint LaserSensor/VerticalRight_sensor_fixedjoint
- removed joint RHand/Touch/Back_sensor_fixedjoint
- removed joint Sonar/Back_sensor_fixedjoint
- removed joint Sonar/Front_sensor_fixedjoint
- removed joint SpeakerLeft_sensor_fixedjoint
- removed joint SpeakerRight_sensor_fixedjoint
- removed joint Tablet_sensor_fixedjoint
- joint HeadPitch: limit lower=-0.706858 upper=0.637045 effort=2.666 velocity=9.22756 -> lower=-0.706858 upper=0.4451 effort=2.666 velocity=9.22756
- joint HeadYaw: origin xyz=-0.038 0 0.1699 rpy=0 0 0 -> xyz=-0.038 0 0.3089 rpy=0 0 0
- joint HipPitch: axis 0 1.0 0 -> 0 -1.0 0; child Pelvis -> Hip; origin xyz=0 0 -0.079 rpy=0 0 0 -> xyz=0 0 0.268 rpy=0 0 0; parent Hip -> Pelvis
- joint HipRoll: axis 1.0 0 0 -> -1.0 0 0; child Hip -> torso; origin xyz=2e-05 0 -0.139 rpy=0 0 0 -> xyz=0 0 0.079 rpy=0 0 0; parent torso -> Hip
- joint KneePitch: axis 0 1.0 0 -> 0 -1.0 0; child Tibia -> Pelvis; origin xyz=0 0 -0.268 rpy=0 0 0 -> xyz=0 0 0 rpy=0 0 0; parent Pelvis -> Tibia
- joint LShoulderPitch: origin xyz=-0.057 0.14974 0.08682 rpy=0 0 0 -> xyz=-0.057 0.14974 0.22582 rpy=0 0 0
- joint RShoulderPitch: origin xyz=-0.057 -0.14974 0.08682 rpy=0 0 0 -> xyz=-0.057 -0.14974 0.22582 rpy=0 0 0
- joint base_footprint_joint: child base_footprint -> base_link; origin xyz=0 0 -0.334 rpy=0 0 0 -> xyz=0 0 0 rpy=0 0 0; parent Tibia -> base_footprint
- joint base_link_fixedjoint: child torso -> Tibia; origin xyz=0 0 0 rpy=0 0 0 -> xyz=0 0 0.334 rpy=0 0 0
