Commit message: change urdf test

File: pepper_robot_description/urdf/pepper_robot.urdf (robot description, URDF)
Before this commit: robot pepper_robot, 50 links, 49 joints
Links:
- removed link LShoulder
- removed link RElbow
- removed link RShoulder
- removed link l_gripper
- removed link r_gripper
- removed link torso
- added link BumperB
- added link BumperFL
- added link BumperFR
- added link CameraBottom
- added link CameraDepth
- added link CameraTop
- added link Gaze
- added link HeadPitch
- added link HeadPitchSphereCollision_shape; collision sphere radius=0.11
- added link HeadYaw
- added link HipPitch
- added link HipPitchPillCollision_shape; collision cylinder length=0.355 radius=0.1275
- added link HipPitchSphereCollision_shape; collision sphere radius=0.095
- added link HipRoll
- added link KneePitch
- added link LArm
- added link LArmFuse
- added link LElbowRoll
- added link LElbowRollDynamicCollision_shape; collision cylinder length=0.27 radius=0.035
- added link LElbowRollPillCollision_shape; collision cylinder length=0.2 radius=0.035
- added link LElbowRollSphereACollision_shape; collision sphere radius=0.035
- added link LElbowRollSphereBCollision_shape; collision sphere radius=0.035
- added link LElbowRollSphereCCollision_shape; collision sphere radius=0.035
- added link LElbowRollSphereDCollision_shape; collision sphere radius=0.035
- added link LElbowYaw
- added link LShoulderPitch, mass 0.3125; visual mesh filename=package://pepper_robot_description/pepper_robot/meshes/LSho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 scale=1 1 1
- added link LShoulderRoll
- added link LWristYaw
- added link LWristYawSphereCollision_shape; collision sphere radius=0.052
- added link RElbowRoll
- added link RElbowRollDynamicCollision_shape; collision cylinder length=0.27 radius=0.035
- added link RElbowRollPillCollision_shape; collision cylinder length=0.2 radius=0.035
- added link RElbowRollSphereACollision_shape; collision sphere radius=0.035
- added link RElbowRollSphereBCollision_shape; collision sphere radius=0.035
- added link RElbowRollSphereCCollision_shape; collision sphere radius=0.035
- added link RElbowRollSphereDCollision_shape; collision sphere radius=0.035
- added link RElbowYaw, mass 0.27495; visual mesh filename=package://pepper_robot_description/pepper_robot/meshes/RElb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 scale=1 1 1
- added link RShoulderPitch, mass 0.3125; visual mesh filename=package://pepper_robot_description/pepper_robot/meshes/RSho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 scale=1 1 1
- added link RShoulderRoll
- added link RWristYaw
- added link RWristYawSphereCollision_shape; collision sphere radius=0.052
- added link SonarBack
- added link SonarFront
- added link TorsoBackLeftSphereCollision_shape; collision sphere radius=0.08
- added link TorsoBackRightSphereCollision_shape; collision sphere radius=0.08
- added link TorsoSphereBackCollision_shape; collision sphere radius=0.1
- added link TorsoSphereLeftCollision_shape; collision sphere radius=0.07
- added link TorsoSphereRightCollision_shape; collision sphere radius=0.07
- added link TorsoTabCollision_shape; collision box size=0.2 0.256 0.1
- added link torso_link, mass 3.99533; visual mesh filename=package://pepper_robot_description/pepper_robot/meshes/Tors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 scale=1 1 1
- link Head: geometry visual mesh filename=package://pepper_robot_description/pepper_robot/meshes/Head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 scale=1 1 1
- link Hip: geometry visual mesh filename=package://pepper_robot_description/pepper_robot/meshes/HipR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 scale=1 1 1
- link LBicep: geometry visual mesh filename=package://pepper_robot_description/pepper_robot/meshes/LSho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 scale=1 1 1
- link LElbow: geometry visual mesh filename=package://pepper_robot_description/pepper_robot/meshes/LElb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 scale=1 1 1
- link LFinger11_link: mass 2e-06 -> None; geometry visual mesh filename=package://pepper_robot_description/pepper_robot/meshes/LFin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 scale=1 1 1
- link LFinger12_link: mass 2e-06 -> None; geometry visual mesh filename=package://pepper_robot_description/pepper_robot/meshes/LFin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 scale=1 1 1
- link LFinger13_link: mass 2e-06 -> None; geometry visual mesh filename=package://pepper_robot_description/pepper_robot/meshes/LFin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 scale=1 1 1
- link LFinger21_link: mass 2e-06 -> None; geometry visual mesh filename=package://pepper_robot_description/pepper_robot/meshes/LFin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 scale=1 1 1
- link LFinger22_link: mass 2e-06 -> None; geometry visual mesh filename=package://pepper_robot_description/pepper_robot/meshes/LFin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 scale=1 1 1
- link LFinger23_link: mass 2e-06 -> None; geometry visual mesh filename=package://pepper_robot_description/pepper_robot/meshes/LFin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 scale=1 1 1
- link LFinger31_link: mass 2e-06 -> None; geometry visual mesh filename=package://pepper_robot_description/pepper_robot/meshes/LFin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 scale=1 1 1
- link LFinger32_link: mass 2e-06 -> None; geometry visual mesh filename=package://pepper_robot_description/pepper_robot/meshes/LFin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 scale=1 1 1
- link LFinger33_link: mass 2e-06 -> None; geometry visual mesh filename=package://pepper_robot_description/pepper_robot/meshes/LFin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 scale=1 1 1
- link LFinger41_link: mass 2e-06 -> None; geometry visual mesh filename=package://pepper_robot_description/pepper_robot/meshes/LFin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 scale=1 1 1
- link LFinger42_link: mass 2e-06 -> None; geometry visual mesh filename=package://pepper_robot_description/pepper_robot/meshes/LFin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 scale=1 1 1
- link LFinger43_link: mass 2e-06 -> None; geometry visual mesh filename=package://pepper_robot_description/pepper_robot/meshes/LFin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 scale=1 1 1
- link LForeArm: geometry visual mesh filename=package://pepper_robot_description/pepper_robot/meshes/LElb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 scale=1 1 1
- link LThumb1_link: mass 2e-06 -> None; geometry visual mesh filename=package://pepper_robot_description/pepper_robot/meshes/LThu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 scale=1 1 1
- link LThumb2_link: mass 2e-06 -> None; geometry visual mesh filename=package://pepper_robot_description/pepper_robot/meshes/LThu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 scale=1 1 1
- link Neck: geometry visual mesh filename=package://pepper_robot_description/pepper_robot/meshes/Head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 scale=1 1 1
- link Pelvis: geometry visual mesh filename=package://pepper_robot_description/pepper_robot/meshes/HipP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 scale=1 1 1
- link RBicep: geometry visual mesh filename=package://pepper_robot_description/pepper_robot/meshes/RSho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 scale=1 1 1
- link RFinger11_link: mass 2e-06 -> None; geometry visual mesh filename=package://pepper_robot_description/pepper_robot/meshes/RFin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 scale=1 1 1
- link RFinger12_link: mass 2e-06 -> None; geometry visual mesh filename=package://pepper_robot_description/pepper_robot/meshes/RFin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 scale=1 1 1
- link RFinger13_link: mass 2e-06 -> None; geometry visual mesh filename=package://pepper_robot_description/pepper_robot/meshes/RFin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 scale=1 1 1
- link RFinger21_link: mass 2e-06 -> None; geometry visual mesh filename=package://pepper_robot_description/pepper_robot/meshes/RFin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 scale=1 1 1
- link RFinger22_link: mass 2e-06 -> None; geometry visual mesh filename=package://pepper_robot_description/pepper_robot/meshes/RFin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 scale=1 1 1
- link RFinger23_link: mass 2e-06 -> None; geometry visual mesh filename=package://pepper_robot_description/pepper_robot/meshes/RFin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 scale=1 1 1
- link RFinger31_link: mass 2e-06 -> None; geometry visual mesh filename=package://pepper_robot_description/pepper_robot/meshes/RFin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 scale=1 1 1
- link RFinger32_link: mass 2e-06 -> None; geometry visual mesh filename=package://pepper_robot_description/pepper_robot/meshes/RFin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 scale=1 1 1
- link RFinger33_link: mass 2e-06 -> None; geometry visual mesh filename=package://pepper_robot_description/pepper_robot/meshes/RFin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 scale=1 1 1
- link RFinger41_link: mass 2e-06 -> None; geometry visual mesh filename=package://pepper_robot_description/pepper_robot/meshes/RFin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 scale=1 1 1
- link RFinger42_link: mass 2e-06 -> None; geometry visual mesh filename=package://pepper_robot_description/pepper_robot/meshes/RFin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 scale=1 1 1
- link RFinger43_link: mass 2e-06 -> None; geometry visual mesh filename=package://pepper_robot_description/pepper_robot/meshes/RFin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 scale=1 1 1
- link RForeArm: geometry visual mesh filename=package://pepper_robot_description/pepper_robot/meshes/RElb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 scale=1 1 1
- link RThumb1_link: mass 2e-06 -> None; geometry visual mesh filename=package://pepper_robot_description/pepper_robot/meshes/RThu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 scale=1 1 1
- link RThumb2_link: mass 2e-06 -> None; geometry visual mesh filename=package://pepper_robot_description/pepper_robot/meshes/RThu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 scale=1 1 1
- link Tibia: geometry visual mesh filename=package://pepper_robot_description/pepper_robot/meshes/Knee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 scale=1 1 1
- link WheelB_link: geometry visual mesh filename=package://pepper_robot_description/pepper_robot/meshes/Whee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 scale=1 1 1
- link WheelFL_link: geometry visual mesh filename=package://pepper_robot_description/pepper_robot/meshes/Whee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 scale=1 1 1
- link WheelFR_link: geometry visual mesh filename=package://pepper_robot_description/pepper_robot/meshes/Whee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 scale=1 1 1
- link l_wrist: geometry visual mesh filename=package://pepper_robot_description/pepper_robot/meshes/LWri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 scale=1 1 1
- link r_wrist: geometry visual mesh filename=package://pepper_robot_description/pepper_robot/meshes/RWri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 scale=1 1 1
Joints:
- added joint BumperB_fixedjoint: type fixed, parent Tibia, child BumperB, origin xyz=-0.251 0.264 0 rpy=-1.5708 -0 3.14159, axis 0 0 0
- added joint BumperFL_fixedjoint: type fixed, parent Tibia, child BumperFL, origin xyz=0.129 0.264 0.227 rpy=1.5708 -0.48886 0, axis 0 0 0
- added joint BumperFR_fixedjoint: type fixed, parent Tibia, child BumperFR, origin xyz=0.129 0.264 -0.227 rpy=1.5708 0.48886 0, axis 0 0 0
- added joint CameraBottom_fixedjoint: type fixed, parent Head, child CameraBottom, origin xyz=0.06177 0.09262 0 rpy=1.5708 5.55112e-17 2.26893, axis 0 0 0
- added joint CameraDepth_fixedjoint: type fixed, parent Head, child CameraDepth, origin xyz=0.1194 0.05138 0.039 rpy=1.5708 5.55112e-17 1.5708, axis 0 0 0
- added joint CameraTop_fixedjoint: type fixed, parent Head, child CameraTop, origin xyz=0.16284 0.08601 0 rpy=1.5708 5.55112e-17 1.5708, axis 0 0 0
- added joint Gaze_fixedjoint: type fixed, parent Head, child Gaze, origin xyz=0.1189 0.0657 0 rpy=1.5708 5.55112e-17 1.5708, axis 0 0 0
- added joint HeadPitchSphereCollision_shape_fixedjoint: type fixed, parent Head, child HeadPitchSphereCollision_shape, origin xyz=0.12 0.004 0 rpy=1.5708 5.55112e-17 1.5708, axis 0 0 0
- added joint HeadPitch_fixedjoint: type fixed, parent Head, child HeadPitch, origin xyz=0 0 0 rpy=1.5708 5.55112e-17 1.5708, axis 0 0 0
- added joint HeadYaw_fixedjoint: type fixed, parent Neck, child HeadYaw, origin xyz=0 0 0 rpy=0 -0 0, axis 0 0 0
- added joint Head_fixedjoint: type fixed, parent Head, child Head, origin xyz=0 0 0 rpy=1.5708 5.55112e-17 1.5708, axis 0 0 0
- added joint HipPitchPillCollision_shape_fixedjoint: type fixed, parent Pelvis, child HipPitchPillCollision_shape, origin xyz=-0.0075 0.07 0 rpy=1.5708 -0 -3.14159, axis 0 0 0
- added joint HipPitchSphereCollision_shape_fixedjoint: type fixed, parent Pelvis, child HipPitchSphereCollision_shape, origin xyz=-0.005 -0.05 0 rpy=1.5708 -0 0, axis 0 0 0
- added joint HipPitch_fixedjoint: type fixed, parent Pelvis, child HipPitch, origin xyz=0 0 0 rpy=1.5708 -0 0, axis 0 0 0
- added joint HipRoll_fixedjoint: type fixed, parent Hip, child HipRoll, origin xyz=0 0 0 rpy=3.14159 -1.5708 3.14159, axis 0 0 0
- added joint KneePitch_fixedjoint: type fixed, parent Tibia, child KneePitch, origin xyz=0 0 0 rpy=1.5708 -0 0, axis 0 0 0
- added joint LArmFuse_fixedjoint: type fixed, parent torso, child LArmFuse, origin xyz=0 0 0 rpy=0 -0 0, axis 0 0 0
- added joint LArm_fixedjoint: type fixed, parent l_wrist, child LArm, origin xyz=0 -0.0303 0.0695 rpy=1.5708 -1.5708 -3.14159, axis 0 0 0
- added joint LElbowRollDynamicCollision_shape_fixedjoint: type fixed, parent LForeArm, child LElbowRollDynamicCollision_shape, origin xyz=0 -0.15 0 rpy=1.5708 -0 0, axis 0 0 0
- added joint LElbowRollPillCollision_shape_fixedjoint: type fixed, parent LForeArm, child LElbowRollPillCollision_shape, origin xyz=0 -0.115 0 rpy=1.5708 -0 0, axis 0 0 0
- added joint LElbowRollSphereACollision_shape_fixedjoint: type fixed, parent LForeArm, child LElbowRollSphereACollision_shape, origin xyz=0 -0.1875 0 rpy=0 -0 -1.5708, axis 0 0 0
- added joint LElbowRollSphereBCollision_shape_fixedjoint: type fixed, parent LForeArm, child LElbowRollSphereBCollision_shape, origin xyz=0 -0.125 0 rpy=0 -0 -1.5708, axis 0 0 0
- added joint LElbowRollSphereCCollision_shape_fixedjoint: type fixed, parent LForeArm, child LElbowRollSphereCCollision_shape, origin xyz=0 -0.0625 0 rpy=0 -0 -1.5708, axis 0 0 0
- added joint LElbowRollSphereDCollision_shape_fixedjoint: type fixed, parent LForeArm, child LElbowRollSphereDCollision_shape, origin xyz=0 0 0 rpy=0 -0 -1.5708, axis 0 0 0
- added joint LElbowRoll_fixedjoint: type fixed, parent LForeArm, child LElbowRoll, origin xyz=0 0 0 rpy=0 -0 -1.5708, axis 0 0 0
- added joint LElbowYaw_fixedjoint: type fixed, parent LElbow, child LElbowYaw, origin xyz=0 0 0 rpy=-1.5708 -1.5708 8.76263e-08, axis 0 0 0
- added joint LShoulderPitch_fixedjoint: type fixed, parent LShoulderPitch, child LShoulderPitch, origin xyz=0 0 0 rpy=1.5708 -0 0, axis 0 0 0
- added joint LShoulderRoll_fixedjoint: type fixed, parent LBicep, child LShoulderRoll, origin xyz=0 0 0 rpy=0 -0 -1.5708, axis 0 0 0
- added joint LWristYawSphereCollision_shape_fixedjoint: type fixed, parent l_wrist, child LWristYawSphereCollision_shape, origin xyz=-0.01 -0.015 0.055 rpy=1.5708 -1.5708 -3.14159, axis 0 0 0
- added joint LWristYaw_fixedjoint: type fixed, parent l_wrist, child LWristYaw, origin xyz=0 0 0 rpy=-1.5708 -1.5708 8.76263e-08, axis 0 0 0
- added joint RArm_fixedjoint: type fixed, parent r_wrist, child RArm, origin xyz=0 -0.0303 0.0695 rpy=1.5708 -1.5708 -3.14159, axis 0 0 0
- added joint RElbowRollDynamicCollision_shape_fixedjoint: type fixed, parent RForeArm, child RElbowRollDynamicCollision_shape, origin xyz=0 -0.15 0 rpy=1.5708 -0 0, axis 0 0 0
- added joint RElbowRollPillCollision_shape_fixedjoint: type fixed, parent RForeArm, child RElbowRollPillCollision_shape, origin xyz=0 -0.115 0 rpy=1.5708 -0 0, axis 0 0 0
- added joint RElbowRollSphereACollision_shape_fixedjoint: type fixed, parent RForeArm, child RElbowRollSphereACollision_shape, origin xyz=0 -0.1875 0 rpy=0 -0 -1.5708, axis 0 0 0
- added joint RElbowRollSphereBCollision_shape_fixedjoint: type fixed, parent RForeArm, child RElbowRollSphereBCollision_shape, origin xyz=0 -0.125 0 rpy=0 -0 -1.5708, axis 0 0 0
- added joint RElbowRollSphereCCollision_shape_fixedjoint: type fixed, parent RForeArm, child RElbowRollSphereCCollision_shape, origin xyz=0 -0.0625 0 rpy=0 -0 -1.5708, axis 0 0 0
- added joint RElbowRollSphereDCollision_shape_fixedjoint: type fixed, parent RForeArm, child RElbowRollSphereDCollision_shape, origin xyz=0 0 0 rpy=0 -0 -1.5708, axis 0 0 0
- added joint RElbowRoll_fixedjoint: type fixed, parent RForeArm, child RElbowRoll, origin xyz=0 0 0 rpy=0 -0 -1.5708, axis 0 0 0
- added joint RElbowYaw_fixedjoint: type fixed, parent RElbowYaw, child RElbowYaw, origin xyz=0 0 0 rpy=-1.5708 -1.5708 8.76263e-08, axis 0 0 0
- added joint RHand/Touch/Back_fixedjoint: type fixed, parent r_wrist, child RHand/Touch/Back, origin xyz=0 0.0304 0.0523 rpy=1.5708 5.55112e-17 1.5708, axis 0 0 0
- added joint RShoulderPitch_fixedjoint: type fixed, parent RShoulderPitch, child RShoulderPitch, origin xyz=0 0 0 rpy=1.5708 -0 0, axis 0 0 0
- added joint RShoulderRoll_fixedjoint: type fixed, parent RBicep, child RShoulderRoll, origin xyz=0 0 0 rpy=0 -0 -1.5708, axis 0 0 0
- added joint RWristYawSphereCollision_shape_fixedjoint: type fixed, parent r_wrist, child RWristYawSphereCollision_shape, origin xyz=0.01 -0.015 0.055 rpy=1.5708 -1.5708 -3.14159, axis 0 0 0
- added joint RWristYaw_fixedjoint: type fixed, parent r_wrist, child RWristYaw, origin xyz=0 0 0 rpy=-1.5708 -1.5708 8.76263e-08, axis 0 0 0
- added joint SonarBack_fixedjoint: type fixed, parent Tibia, child SonarBack, origin xyz=-0.0718 0.0534 0 rpy=-1.5708 1.38778e-17 -2.93215, axis 0 0 0
- added joint SonarFront_fixedjoint: type fixed, parent Tibia, child SonarFront, origin xyz=0.0699 0.1023 0 rpy=1.5708 -0 -0.322858, axis 0 0 0
- added joint TorsoBackLeftSphereCollision_shape_fixedjoint: type fixed, parent torso, child TorsoBackLeftSphereCollision_shape, origin xyz=-0.08 0.055 -0.06 rpy=0 -0 0, axis 0 0 0
- added joint TorsoBackRightSphereCollision_shape_fixedjoint: type fixed, parent torso, child TorsoBackRightSphereCollision_shape, origin xyz=-0.08 -0.055 -0.06 rpy=0 -0 0, axis 0 0 0
- added joint TorsoSphereBackCollision_shape_fixedjoint: type fixed, parent torso, child TorsoSphereBackCollision_shape, origin xyz=0 0 -0.08 rpy=0 -0 0, axis 0 0 0
- added joint TorsoSphereLeftCollision_shape_fixedjoint: type fixed, parent torso, child TorsoSphereLeftCollision_shape, origin xyz=0.08 0.05 0 rpy=0 -0 0, axis 0 0 0
- added joint TorsoSphereRightCollision_shape_fixedjoint: type fixed, parent torso, child TorsoSphereRightCollision_shape, origin xyz=0.08 -0.05 0 rpy=0 -0 0, axis 0 0 0
- added joint TorsoTabCollision_shape_fixedjoint: type fixed, parent torso, child TorsoTabCollision_shape, origin xyz=0.08 0 0.04 rpy=0 1.0472 0, axis 0 0 0
- joint HeadPitch: axis 0 1.0 0 -> 0 0 1; limit lower=-0.706858 upper=0.4451 effort=2.666 velocity=9.22756 -> lower=-0.706858 upper=0.445059 effort=2.66575 velocity=9.22756; origin xyz=0 0 0 rpy=0 0 0 -> xyz=0 0 0 rpy=1.5708 -1.5708 -3.14159
- joint HeadYaw: axis 0 0 1.0 -> 0 0 1; limit lower=-2.08567 upper=2.08567 effort=5.428 velocity=7.33998 -> lower=-2.08567 upper=2.08567 effort=1.8721 velocity=7.33998; origin xyz=-0.038 0 0.3089 rpy=0 0 0 -> xyz=-0.038 0 0.1699 rpy=0 -0 0
- joint HipPitch: axis 0 -1.0 0 -> 0 0 1; child Hip -> Pelvis; origin xyz=0 0 0.268 rpy=0 0 0 -> xyz=0.079 0 0 rpy=1.5708 -1.5708 -3.14159; parent Pelvis -> Hip
- joint HipRoll: axis -1.0 0 0 -> 0 0 1; child torso -> Hip; origin xyz=0 0 0.079 rpy=0 0 0 -> xyz=2e-05 0 -0.139 rpy=3.14159 1.5708 3.14159; parent Hip -> torso
- joint KneePitch: axis 0 -1.0 0 -> 0 0 1; child Pelvis -> Tibia; origin xyz=0 0 0 rpy=0 0 0 -> xyz=0 0.268 0 rpy=0 -0 0; parent Tibia -> Pelvis
- joint LElbowRoll: axis 0 0 1.0 -> 0 0 1; limit lower=-1.56207 upper=-0.00872665 effort=2.666 velocity=9.22756 -> lower=-1.56207 upper=-0.00872665 effort=2.22146 velocity=9.22756; origin xyz=0 0 0 rpy=0 0 0 -> xyz=0 0 0 rpy=-1.5708 -0 0
- joint LElbowYaw: axis 1.0 0 0 -> 0 0 1; limit lower=-2.08567 upper=2.08567 effort=5.428 velocity=7.33998 -> lower=-2.08567 upper=2.08567 effort=2.80815 velocity=7.33998; origin xyz=0.1812 0.015 0.00013 rpy=0 -0.157079 0 -> xyz=0.015 -0.1812 0.00013 rpy=1.41372 -0 0
- joint LFinger11: axis 0 0 1.0 -> 0 0 1; origin xyz=0.0821 -0.0268 0.004 rpy=1.74402 1.04064 -0.0334335 -> xyz=-0.0268 0.004 0.0821 rpy=1.78277 -0.529825 -1.59039
- joint LFinger12: axis 0 0 1.0 -> 0 0 1; origin xyz=0.018 0 0 rpy=0 0 -1.0472 -> xyz=0.018 0 0 rpy=-0 -0 -1.0472
- joint LFinger13: axis 0 0 1.0 -> 0 0 1; origin xyz=0.018 0 0 rpy=0 0 -1.0472 -> xyz=0.018 0 0 rpy=-0 -0 -1.0472
- joint LFinger21: axis 0 0 1.0 -> 0 0 1; origin xyz=0.0873 -0.0073 0.006 rpy=1.5708 1.0472 -0.061086 -> xyz=-0.0073 0.006 0.0873 rpy=1.6413 -0.522522 -1.60603
- joint LFinger22: axis 0 0 1.0 -> 0 0 1; origin xyz=0.018 0 0 rpy=0 0 -1.0472 -> xyz=0.018 0 0 rpy=-0 -0 -1.0472
- joint LFinger23: axis 0 0 1.0 -> 0 0 1; origin xyz=0.018 0 0 rpy=0 0 -1.0472 -> xyz=0.018 0 0 rpy=-0 -0 -1.0472
- joint LFinger31: axis 0 0 1.0 -> 0 0 1; origin xyz=0.0833 0.0123 0.004 rpy=1.46636 1.04483 -0.029314 -> xyz=0.0123 0.004 0.0833 rpy=1.50025 -0.525718 -1.58781
- joint LFinger32: axis 0 0 1.0 -> 0 0 1; origin xyz=0.018 0 0 rpy=0 0 -1.0472 -> xyz=0.018 0 0 rpy=-0 -0 -1.0472
- joint LFinger33: axis 0 0 1.0 -> 0 0 1; origin xyz=0.018 0 0 rpy=0 0 -1.0472 -> xyz=0.018 0 0 rpy=-0 -0 -1.0472
- joint LFinger41: axis 0 0 1.0 -> 0 0 1; origin xyz=0.074 0.0309 0 rpy=1.39757 1.04064 0.0683394 -> xyz=0.0309 0 0.074 rpy=1.3184 -0.528785 -1.53079
- joint LFinger42: axis 0 0 1.0 -> 0 0 1; origin xyz=0.018 0 0 rpy=0 0 -1.0472 -> xyz=0.018 0 0 rpy=-0 -0 -1.0472
- joint LFinger43: axis 0 0 1.0 -> 0 0 1; origin xyz=0.018 0 0 rpy=0 0 -1.0472 -> xyz=0.018 0 0 rpy=-0 -0 -1.0472
- joint LHand: axis 1.0 0 0 -> 1 0 0; child l_gripper -> LHand_actuator_frame; limit lower=0.02 upper=0.98 effort=0.144 velocity=12.56 -> lower=0.02 upper=0.98 effort=0.096152 velocity=12.56; origin xyz=0.025 0 0 rpy=0 0 0 -> xyz=0 0 0.025 rpy=1.5708 -1.5708 -3.14159
- joint LShoulderPitch: axis 0 1.0 0 -> 0 0 1; child LShoulder -> LShoulderPitch; limit lower=-2.08567 upper=2.08567 effort=5.428 velocity=7.33998 -> lower=-2.08567 upper=2.08567 effort=4.11862 velocity=7.33998; origin xyz=-0.057 0.14974 0.22582 rpy=0 0 0 -> xyz=-0.057 0.14974 0.08682 rpy=-1.5708 -0 0
- joint LShoulderRoll: axis 0 0 1.0 -> 0 0 1; limit lower=0.00872665 upper=1.56207 effort=2.666 velocity=9.22756 -> lower=0.00872665 upper=1.56207 effort=3.70244 velocity=9.22756; origin xyz=0 0 0 rpy=0 0 0 -> xyz=0 0 0 rpy=-1.5708 -1.5708 3.14159; parent LShoulder -> LShoulderPitch
- joint LThumb1: axis 0 0 1.0 -> 0 0 1; origin xyz=0.0482 -0.0357 -0.0199 rpy=-1.95836 0.60626 0.533978 -> xyz=-0.0357 -0.0199 0.0482 rpy=-2.76225 -0.785789 -0.937585
- joint LThumb2: axis 0 0 1.0 -> 0 0 1; origin xyz=0.022 0 0 rpy=0 0 -1.0472 -> xyz=0.022 0 0 rpy=-0 -0 -1.0472
- joint LWristYaw: axis 1.0 0 0 -> 0 0 1; limit lower=-1.82387 upper=1.82387 effort=0.2014 velocity=17.3835 -> lower=-1.82387 upper=1.82387 effort=0.134278 velocity=17.3835; origin xyz=0.15 0 0 rpy=0 0 0 -> xyz=0 -0.15 0 rpy=1.5708 -0 0
- joint RElbowRoll: axis 0 0 1.0 -> 0 0 1; limit lower=0.00872665 upper=1.56207 effort=2.666 velocity=9.22756 -> lower=0.00872665 upper=1.56207 effort=2.22146 velocity=9.22756; origin xyz=0 0 0 rpy=0 0 0 -> xyz=0 0 0 rpy=-1.5708 -0 0; parent RElbow -> RElbowYaw
- joint RElbowYaw: axis 1.0 0 0 -> 0 0 1; child RElbow -> RElbowYaw; limit lower=-2.08567 upper=2.08567 effort=5.428 velocity=7.33998 -> lower=-2.08567 upper=2.08567 effort=2.80815 velocity=7.33998; origin xyz=0.1812 -0.015 0.00013 rpy=0 -0.157079 0 -> xyz=-0.015 -0.1812 0.00013 rpy=1.41372 -0 0
- joint RFinger11: axis 0 0 1.0 -> 0 0 1; origin xyz=0.0821 0.0268 0.004 rpy=1.39757 1.04064 0.0334335 -> xyz=0.0268 0.004 0.0821 rpy=1.35882 -0.529825 -1.55121
- joint RFinger12: axis 0 0 1.0 -> 0 0 1; origin xyz=0.018 0 0 rpy=0 0 -1.0472 -> xyz=0.018 0 0 rpy=-0 -0 -1.0472
- joint RFinger13: axis 0 0 1.0 -> 0 0 1; origin xyz=0.018 0 0 rpy=0 0 -1.0472 -> xyz=0.018 0 0 rpy=-0 -0 -1.0472
- joint RFinger21: axis 0 0 1.0 -> 0 0 1; origin xyz=0.0873 0.0073 0.006 rpy=1.5708 1.0472 0.061086 -> xyz=0.0073 0.006 0.0873 rpy=1.50029 -0.522522 -1.53556
- joint RFinger22: axis 0 0 1.0 -> 0 0 1; origin xyz=0.018 0 0 rpy=0 0 -1.0472 -> xyz=0.018 0 0 rpy=-0 -0 -1.0472
- joint RFinger23: axis 0 0 1.0 -> 0 0 1; origin xyz=0.018 0 0 rpy=0 0 -1.0472 -> xyz=0.018 0 0 rpy=-0 -0 -1.0472
- joint RFinger31: axis 0 0 1.0 -> 0 0 1; origin xyz=0.0833 -0.0123 0.004 rpy=1.67523 1.04483 0.029316 -> xyz=-0.0123 0.004 0.0833 rpy=1.64134 -0.525718 -1.55378
- joint RFinger32: axis 0 0 1.0 -> 0 0 1; origin xyz=0.018 0 0 rpy=0 0 -1.0472 -> xyz=0.018 0 0 rpy=-0 -0 -1.0472
- joint RFinger33: axis 0 0 1.0 -> 0 0 1; origin xyz=0.018 0 0 rpy=0 0 -1.0472 -> xyz=0.018 0 0 rpy=-0 -0 -1.0472
- joint RFinger41: axis 0 0 1.0 -> 0 0 1; origin xyz=0.074 -0.0309 0 rpy=1.74402 1.04064 -0.0683394 -> xyz=-0.0309 0 0.074 rpy=1.82319 -0.528785 -1.6108
- joint RFinger42: axis 0 0 1.0 -> 0 0 1; origin xyz=0.018 0 0 rpy=0 0 -1.0472 -> xyz=0.018 0 0 rpy=-0 -0 -1.0472
- joint RFinger43: axis 0 0 1.0 -> 0 0 1; origin xyz=0.018 0 0 rpy=0 0 -1.0472 -> xyz=0.018 0 0 rpy=-0 -0 -1.0472
- joint RHand: axis 1.0 0 0 -> 1 0 0; child r_gripper -> RHand_actuator_frame; limit lower=0.02 upper=0.98 effort=0.144 velocity=12.56 -> lower=0.02 upper=0.98 effort=0.096152 velocity=12.56; origin xyz=0.025 0 0 rpy=0 0 0 -> xyz=0 0 0.025 rpy=1.5708 -1.5708 -3.14159
- joint RShoulderPitch: axis 0 1.0 0 -> 0 0 1; child RShoulder -> RShoulderPitch; limit lower=-2.08567 upper=2.08567 effort=5.428 velocity=7.33998 -> lower=-2.08567 upper=2.08567 effort=4.11862 velocity=7.33998; origin xyz=-0.057 -0.14974 0.22582 rpy=0 0 0 -> xyz=-0.057 -0.14974 0.08682 rpy=-1.5708 -0 0
- joint RShoulderRoll: axis 0 0 1.0 -> 0 0 1; limit lower=-1.56207 upper=-0.00872665 effort=2.666 velocity=9.22756 -> lower=-1.56207 upper=-0.00872665 effort=3.70244 velocity=9.22756; origin xyz=0 0 0 rpy=0 0 0 -> xyz=0 0 0 rpy=-1.5708 -1.5708 3.14159; parent RShoulder -> RShoulderPitch
- joint RThumb1: axis 0 0 1.0 -> 0 0 1; origin xyz=0.0482 0.0357 -0.0199 rpy=-1.18323 0.60626 -0.533978 -> xyz=0.0357 -0.0199 0.0482 rpy=-0.379338 -0.785789 -2.20401
- joint RThumb2: axis 0 0 1.0 -> 0 0 1; origin xyz=0.022 0 0 rpy=0 0 -1.0472 -> xyz=0.022 0 0 rpy=-0 -0 -1.0472
- joint RWristYaw: axis 1.0 0 0 -> 0 0 1; limit lower=-1.82387 upper=1.82387 effort=0.2014 velocity=17.3835 -> lower=-1.82387 upper=1.82387 effort=0.134278 velocity=17.3835; origin xyz=0.15 0 0 rpy=0 0 0 -> xyz=0 -0.15 0 rpy=1.5708 -0 0
- joint WheelB: axis 1.0 0 0 -> 1 0 0; origin xyz=-0.17 0 -0.264 rpy=0 0 -3.14159 -> xyz=-0.17 0.264 0 rpy=-1.5708 -0 -3.14159
- joint WheelFL: axis 1.0 0 0 -> 1 0 0; origin xyz=0.09 0.155 -0.264 rpy=0 0 1.07517 -> xyz=0.09 0.264 0.155 rpy=1.5708 -1.07517 -1.16723e-16
- joint WheelFR: axis 1.0 0 0 -> 1 0 0; origin xyz=0.09 -0.155 -0.264 rpy=0 0 -1.07517 -> xyz=0.09 0.264 -0.155 rpy=1.5708 1.07517 1.16723e-16
- joint base_link_fixedjoint: child Tibia -> torso; origin xyz=0 0 0.334 rpy=0 0 0 -> xyz=0 0 0 rpy=0 -0 0
