Commit message: change urdf test failed

File: pepper_robot_description/urdf/pepper_robot.urdf (robot description, URDF)
Before this commit: robot pepper_robot, 94 links, 101 joints
Links:
- removed link BumperB
- removed link BumperFL
- removed link BumperFR
- removed link CameraBottom
- removed link CameraDepth
- removed link CameraTop
- removed link Gaze
- removed link HeadPitch
- removed link HeadPitchSphereCollision_shape
- removed link HeadYaw
- removed link HipPitch
- removed link HipPitchPillCollision_shape
- removed link HipPitchSphereCollision_shape
- removed link HipRoll
- removed link KneePitch
- removed link LArm
- removed link LArmFuse
- removed link LElbowRoll
- removed link LElbowRollDynamicCollision_shape
- removed link LElbowRollPillCollision_shape
- removed link LElbowRollSphereACollision_shape
- removed link LElbowRollSphereBCollision_shape
- removed link LElbowRollSphereCCollision_shape
- removed link LElbowRollSphereDCollision_shape
- removed link LElbowYaw
- removed link LShoulderPitch
- removed link LShoulderRoll
- removed link LWristYaw
- removed link LWristYawSphereCollision_shape
- removed link RElbowRoll
- removed link RElbowRollDynamicCollision_shape
- removed link RElbowRollPillCollision_shape
- removed link RElbowRollSphereACollision_shape
- removed link RElbowRollSphereBCollision_shape
- removed link RElbowRollSphereCCollision_shape
- removed link RElbowRollSphereDCollision_shape
- removed link RElbowYaw
- removed link RShoulderPitch
- removed link RShoulderRoll
- removed link RWristYaw
- removed link RWristYawSphereCollision_shape
- removed link SonarBack
- removed link SonarFront
- removed link TorsoBackLeftSphereCollision_shape
- removed link TorsoBackRightSphereCollision_shape
- removed link TorsoSphereBackCollision_shape
- removed link TorsoSphereLeftCollision_shape
- removed link TorsoSphereRightCollision_shape
- removed link TorsoTabCollision_shape
- removed link torso_link
- added link LShoulder, mass 0.3125; collision mesh filename=package://pepper_robot_description/pepper_robot/meshes/LSho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 scale=0.1 0.1 0.1; visual mesh filename=package://pepper_robot_description/pepper_robot/meshes/LSho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 scale=0.1 0.1 0.1
- added link RElbow, mass 0.27495; collision mesh filename=package://pepper_robot_description/pepper_robot/meshes/RElb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 scale=0.1 0.1 0.1; visual mesh filename=package://pepper_robot_description/pepper_robot/meshes/RElb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 scale=0.1 0.1 0.1
- added link RShoulder, mass 0.3125; collision mesh filename=package://pepper_robot_description/pepper_robot/meshes/RSho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 scale=0.1 0.1 0.1; visual mesh filename=package://pepper_robot_description/pepper_robot/meshes/RSho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 scale=0.1 0.1 0.1
- added link l_gripper, mass 2e-06
- added link r_gripper, mass 2e-06
- added link torso, mass 3.99533; collision mesh filename=package://pepper_robot_description/pepper_robot/meshes/Tors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 scale=0.1 0.1 0.1; visual mesh filename=package://pepper_robot_description/pepper_robot/meshes/Tors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 scale=0.1 0.1 0.1
- link Head: geometry collision mesh filename=package://pepper_robot_description/pepper_robot/meshes/Head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 scale=0.1 0.1 0.1; visual mesh filename=package://pepper_robot_description/pepper_robot/meshes/Head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 scale=0.1 0.1 0.1
- link Hip: geometry collision mesh filename=package://pepper_robot_description/pepper_robot/meshes/HipR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 scale=0.1 0.1 0.1; visual mesh filename=package://pepper_robot_description/pepper_robot/meshes/HipR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 scale=0.1 0.1 0.1
- link LBicep: geometry collision mesh filename=package://pepper_robot_description/pepper_robot/meshes/LSho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 scale=0.1 0.1 0.1; visual mesh filename=package://pepper_robot_description/pepper_robot/meshes/LSho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 scale=0.1 0.1 0.1
- link LElbow: geometry collision mesh filename=package://pepper_robot_description/pepper_robot/meshes/LElb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 scale=0.1 0.1 0.1; visual mesh filename=package://pepper_robot_description/pepper_robot/meshes/LElb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 scale=0.1 0.1 0.1
- link LFinger11_link: mass None -> 2e-06; geometry collision mesh filename=package://pepper_robot_description/pepper_robot/meshes/LFin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 scale=0.1 0.1 0.1; visual mesh filename=package://pepper_robot_description/pepper_robot/meshes/LFin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 scale=0.1 0.1 0.1
- link LFinger12_link: mass None -> 2e-06; geometry collision mesh filename=package://pepper_robot_description/pepper_robot/meshes/LFin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 scale=0.1 0.1 0.1; visual mesh filename=package://pepper_robot_description/pepper_robot/meshes/LFin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 scale=0.1 0.1 0.1
- link LFinger13_link: mass None -> 2e-06; geometry collision mesh filename=package://pepper_robot_description/pepper_robot/meshes/LFin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 scale=0.1 0.1 0.1; visual mesh filename=package://pepper_robot_description/pepper_robot/meshes/LFin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 scale=0.1 0.1 0.1
- link LFinger21_link: mass None -> 2e-06; geometry collision mesh filename=package://pepper_robot_description/pepper_robot/meshes/LFin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 scale=0.1 0.1 0.1; visual mesh filename=package://pepper_robot_description/pepper_robot/meshes/LFin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 scale=0.1 0.1 0.1
- link LFinger22_link: mass None -> 2e-06; geometry collision mesh filename=package://pepper_robot_description/pepper_robot/meshes/LFin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 scale=0.1 0.1 0.1; visual mesh filename=package://pepper_robot_description/pepper_robot/meshes/LFin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 scale=0.1 0.1 0.1
- link LFinger23_link: mass None -> 2e-06; geometry collision mesh filename=package://pepper_robot_description/pepper_robot/meshes/LFin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 scale=0.1 0.1 0.1; visual mesh filename=package://pepper_robot_description/pepper_robot/meshes/LFin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 scale=0.1 0.1 0.1
- link LFinger31_link: mass None -> 2e-06; geometry collision mesh filename=package://pepper_robot_description/pepper_robot/meshes/LFin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 scale=0.1 0.1 0.1; visual mesh filename=package://pepper_robot_description/pepper_robot/meshes/LFin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 scale=0.1 0.1 0.1
- link LFinger32_link: mass None -> 2e-06; geometry collision mesh filename=package://pepper_robot_description/pepper_robot/meshes/LFin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 scale=0.1 0.1 0.1; visual mesh filename=package://pepper_robot_description/pepper_robot/meshes/LFin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 scale=0.1 0.1 0.1
- link LFinger33_link: mass None -> 2e-06; geometry collision mesh filename=package://pepper_robot_description/pepper_robot/meshes/LFin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 scale=0.1 0.1 0.1; visual mesh filename=package://pepper_robot_description/pepper_robot/meshes/LFin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 scale=0.1 0.1 0.1
- link LFinger41_link: mass None -> 2e-06; geometry collision mesh filename=package://pepper_robot_description/pepper_robot/meshes/LFin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 scale=0.1 0.1 0.1; visual mesh filename=package://pepper_robot_description/pepper_robot/meshes/LFin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 scale=0.1 0.1 0.1
- link LFinger42_link: mass None -> 2e-06; geometry collision mesh filename=package://pepper_robot_description/pepper_robot/meshes/LFin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 scale=0.1 0.1 0.1; visual mesh filename=package://pepper_robot_description/pepper_robot/meshes/LFin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 scale=0.1 0.1 0.1
- link LFinger43_link: mass None -> 2e-06; geometry collision mesh filename=package://pepper_robot_description/pepper_robot/meshes/LFin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 scale=0.1 0.1 0.1; visual mesh filename=package://pepper_robot_description/pepper_robot/meshes/LFin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 scale=0.1 0.1 0.1
- link LForeArm: geometry collision mesh filename=package://pepper_robot_description/pepper_robot/meshes/LElb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 scale=0.1 0.1 0.1; visual mesh filename=package://pepper_robot_description/pepper_robot/meshes/LElb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 scale=0.1 0.1 0.1
- link LThumb1_link: mass None -> 2e-06; geometry collision mesh filename=package://pepper_robot_description/pepper_robot/meshes/LThu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 scale=0.1 0.1 0.1; visual mesh filename=package://pepper_robot_description/pepper_robot/meshes/LThu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 scale=0.1 0.1 0.1
- link LThumb2_link: mass None -> 2e-06; geometry collision mesh filename=package://pepper_robot_description/pepper_robot/meshes/LThu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 scale=0.1 0.1 0.1; visual mesh filename=package://pepper_robot_description/pepper_robot/meshes/LThu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 scale=0.1 0.1 0.1
- link Neck: geometry collision mesh filename=package://pepper_robot_description/pepper_robot/meshes/Head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 scale=0.1 0.1 0.1; visual mesh filename=package://pepper_robot_description/pepper_robot/meshes/Head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 scale=0.1 0.1 0.1
- link Pelvis: geometry collision mesh filename=package://pepper_robot_description/pepper_robot/meshes/HipP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 scale=0.1 0.1 0.1; visual mesh filename=package://pepper_robot_description/pepper_robot/meshes/HipP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 scale=0.1 0.1 0.1
- link RBicep: geometry collision mesh filename=package://pepper_robot_description/pepper_robot/meshes/RSho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 scale=0.1 0.1 0.1; visual mesh filename=package://pepper_robot_description/pepper_robot/meshes/RSho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 scale=0.1 0.1 0.1
- link RFinger11_link: mass None -> 2e-06; geometry collision mesh filename=package://pepper_robot_description/pepper_robot/meshes/RFin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 scale=0.1 0.1 0.1; visual mesh filename=package://pepper_robot_description/pepper_robot/meshes/RFin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 scale=0.1 0.1 0.1
- link RFinger12_link: mass None -> 2e-06; geometry collision mesh filename=package://pepper_robot_description/pepper_robot/meshes/RFin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 scale=0.1 0.1 0.1; visual mesh filename=package://pepper_robot_description/pepper_robot/meshes/RFin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 scale=0.1 0.1 0.1
- link RFinger13_link: mass None -> 2e-06; geometry collision mesh filename=package://pepper_robot_description/pepper_robot/meshes/RFin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 scale=0.1 0.1 0.1; visual mesh filename=package://pepper_robot_description/pepper_robot/meshes/RFin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 scale=0.1 0.1 0.1
- link RFinger21_link: mass None -> 2e-06; geometry collision mesh filename=package://pepper_robot_description/pepper_robot/meshes/RFin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 scale=0.1 0.1 0.1; visual mesh filename=package://pepper_robot_description/pepper_robot/meshes/RFin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 scale=0.1 0.1 0.1
- link RFinger22_link: mass None -> 2e-06; geometry collision mesh filename=package://pepper_robot_description/pepper_robot/meshes/RFin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 scale=0.1 0.1 0.1; visual mesh filename=package://pepper_robot_description/pepper_robot/meshes/RFin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 scale=0.1 0.1 0.1
- link RFinger23_link: mass None -> 2e-06; geometry collision mesh filename=package://pepper_robot_description/pepper_robot/meshes/RFin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 scale=0.1 0.1 0.1; visual mesh filename=package://pepper_robot_description/pepper_robot/meshes/RFin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 scale=0.1 0.1 0.1
- link RFinger31_link: mass None -> 2e-06; geometry collision mesh filename=package://pepper_robot_description/pepper_robot/meshes/RFin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 scale=0.1 0.1 0.1; visual mesh filename=package://pepper_robot_description/pepper_robot/meshes/RFin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 scale=0.1 0.1 0.1
- link RFinger32_link: mass None -> 2e-06; geometry collision mesh filename=package://pepper_robot_description/pepper_robot/meshes/RFin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 scale=0.1 0.1 0.1; visual mesh filename=package://pepper_robot_description/pepper_robot/meshes/RFin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 scale=0.1 0.1 0.1
- link RFinger33_link: mass None -> 2e-06; geometry collision mesh filename=package://pepper_robot_description/pepper_robot/meshes/RFin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 scale=0.1 0.1 0.1; visual mesh filename=package://pepper_robot_description/pepper_robot/meshes/RFin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 scale=0.1 0.1 0.1
- link RFinger41_link: mass None -> 2e-06; geometry collision mesh filename=package://pepper_robot_description/pepper_robot/meshes/RFin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 scale=0.1 0.1 0.1; visual mesh filename=package://pepper_robot_description/pepper_robot/meshes/RFin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 scale=0.1 0.1 0.1
- link RFinger42_link: mass None -> 2e-06; geometry collision mesh filename=package://pepper_robot_description/pepper_robot/meshes/RFin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 scale=0.1 0.1 0.1; visual mesh filename=package://pepper_robot_description/pepper_robot/meshes/RFin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 scale=0.1 0.1 0.1
- link RFinger43_link: mass None -> 2e-06; geometry collision mesh filename=package://pepper_robot_description/pepper_robot/meshes/RFin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 scale=0.1 0.1 0.1; visual mesh filename=package://pepper_robot_description/pepper_robot/meshes/RFin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 scale=0.1 0.1 0.1
- link RForeArm: geometry collision mesh filename=package://pepper_robot_description/pepper_robot/meshes/RElb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 scale=0.1 0.1 0.1; visual mesh filename=package://pepper_robot_description/pepper_robot/meshes/RElb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 scale=0.1 0.1 0.1
- link RThumb1_link: mass None -> 2e-06; geometry collision mesh filename=package://pepper_robot_description/pepper_robot/meshes/RThu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 scale=0.1 0.1 0.1; visual mesh filename=package://pepper_robot_description/pepper_robot/meshes/RThu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 scale=0.1 0.1 0.1
- link RThumb2_link: mass None -> 2e-06; geometry collision mesh filename=package://pepper_robot_description/pepper_robot/meshes/RThu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 scale=0.1 0.1 0.1; visual mesh filename=package://pepper_robot_description/pepper_robot/meshes/RThu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 scale=0.1 0.1 0.1
- link Tibia: geometry collision mesh filename=package://pepper_robot_description/pepper_robot/meshes/Knee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 scale=0.1 0.1 0.1; visual mesh filename=package://pepper_robot_description/pepper_robot/meshes/Knee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 scale=0.1 0.1 0.1
- link WheelB_link: geometry collision mesh filename=package://pepper_robot_description/pepper_robot/meshes/Whee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 scale=0.1 0.1 0.1; visual mesh filename=package://pepper_robot_description/pepper_robot/meshes/Whee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 scale=0.1 0.1 0.1
- link WheelFL_link: geometry collision mesh filename=package://pepper_robot_description/pepper_robot/meshes/Whee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 scale=0.1 0.1 0.1; visual mesh filename=package://pepper_robot_description/pepper_robot/meshes/Whee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 scale=0.1 0.1 0.1
- link WheelFR_link: geometry collision mesh filename=package://pepper_robot_description/pepper_robot/meshes/Whee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 scale=0.1 0.1 0.1; visual mesh filename=package://pepper_robot_description/pepper_robot/meshes/Whee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 scale=0.1 0.1 0.1
- link l_wrist: geometry collision mesh filename=package://pepper_robot_description/pepper_robot/meshes/LWri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 scale=0.1 0.1 0.1; visual mesh filename=package://pepper_robot_description/pepper_robot/meshes/LWri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 scale=0.1 0.1 0.1
- link r_wrist: geometry collision mesh filename=package://pepper_robot_description/pepper_robot/meshes/RWri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 scale=0.1 0.1 0.1; visual mesh filename=package://pepper_robot_description/pepper_robot/meshes/RWri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 scale=0.1 0.1 0.1
Joints:
- removed joint BumperB_fixedjoint
- removed joint BumperFL_fixedjoint
- removed joint BumperFR_fixedjoint
- removed joint CameraBottom_fixedjoint
- removed joint CameraDepth_fixedjoint
- removed joint CameraTop_fixedjoint
- removed joint Gaze_fixedjoint
- removed joint HeadPitchSphereCollision_shape_fixedjoint
- removed joint HeadPitch_fixedjoint
- removed joint HeadYaw_fixedjoint
- removed joint Head_fixedjoint
- removed joint HipPitchPillCollision_shape_fixedjoint
- removed joint HipPitchSphereCollision_shape_fixedjoint
- removed joint HipPitch_fixedjoint
- removed joint HipRoll_fixedjoint
- removed joint KneePitch_fixedjoint
- removed joint LArmFuse_fixedjoint
- removed joint LArm_fixedjoint
- removed joint LElbowRollDynamicCollision_shape_fixedjoint
- removed joint LElbowRollPillCollision_shape_fixedjoint
- removed joint LElbowRollSphereACollision_shape_fixedjoint
- removed joint LElbowRollSphereBCollision_shape_fixedjoint
- removed joint LElbowRollSphereCCollision_shape_fixedjoint
- removed joint LElbowRollSphereDCollision_shape_fixedjoint
- removed joint LElbowRoll_fixedjoint
- removed joint LElbowYaw_fixedjoint
- removed joint LShoulderPitch_fixedjoint
- removed joint LShoulderRoll_fixedjoint
- removed joint LWristYawSphereCollision_shape_fixedjoint
- removed joint LWristYaw_fixedjoint
- removed joint RArm_fixedjoint
- removed joint RElbowRollDynamicCollision_shape_fixedjoint
- removed joint RElbowRollPillCollision_shape_fixedjoint
- removed joint RElbowRollSphereACollision_shape_fixedjoint
- removed joint RElbowRollSphereBCollision_shape_fixedjoint
- removed joint RElbowRollSphereCCollision_shape_fixedjoint
- removed joint RElbowRollSphereDCollision_shape_fixedjoint
- removed joint RElbowRoll_fixedjoint
- removed joint RElbowYaw_fixedjoint
- removed joint RHand/Touch/Back_fixedjoint
- removed joint RShoulderPitch_fixedjoint
- removed joint RShoulderRoll_fixedjoint
- removed joint RWristYawSphereCollision_shape_fixedjoint
- removed joint RWristYaw_fixedjoint
- removed joint SonarBack_fixedjoint
- removed joint SonarFront_fixedjoint
- removed joint TorsoBackLeftSphereCollision_shape_fixedjoint
- removed joint TorsoBackRightSphereCollision_shape_fixedjoint
- removed joint TorsoSphereBackCollision_shape_fixedjoint
- removed joint TorsoSphereLeftCollision_shape_fixedjoint
- removed joint TorsoSphereRightCollision_shape_fixedjoint
- removed joint TorsoTabCollision_shape_fixedjoint
- joint HeadPitch: axis 0 0 1 -> 0 1.0 0; limit lower=-0.706858 upper=0.445059 effort=2.66575 velocity=9.22756 -> lower=-0.706858 upper=0.4451 effort=2.666 velocity=9.22756; origin xyz=0 0 0 rpy=1.5708 -1.5708 -3.14159 -> xyz=0 0 0 rpy=0 0 0
- joint HeadYaw: axis 0 0 1 -> 0 0 1.0; limit lower=-2.08567 upper=2.08567 effort=1.8721 velocity=7.33998 -> lower=-2.08567 upper=2.08567 effort=5.428 velocity=7.33998; origin xyz=-0.038 0 0.1699 rpy=0 -0 0 -> xyz=-0.038 0 0.3089 rpy=0 0 0
- joint HipPitch: axis 0 0 1 -> 0 -1.0 0; child Pelvis -> Hip; origin xyz=0.079 0 0 rpy=1.5708 -1.5708 -3.14159 -> xyz=0 0 0.268 rpy=0 0 0; parent Hip -> Pelvis
- joint HipRoll: axis 0 0 1 -> -1.0 0 0; child Hip -> torso; origin xyz=2e-05 0 -0.139 rpy=3.14159 1.5708 3.14159 -> xyz=0 0 0.079 rpy=0 0 0; parent torso -> Hip
- joint KneePitch: axis 0 0 1 -> 0 -1.0 0; child Tibia -> Pelvis; origin xyz=0 0.268 0 rpy=0 -0 0 -> xyz=0 0 0 rpy=0 0 0; parent Pelvis -> Tibia
- joint LElbowRoll: axis 0 0 1 -> 0 0 1.0; limit lower=-1.56207 upper=-0.00872665 effort=2.22146 velocity=9.22756 -> lower=-1.56207 upper=-0.00872665 effort=2.666 velocity=9.22756; origin xyz=0 0 0 rpy=-1.5708 -0 0 -> xyz=0 0 0 rpy=0 0 0
- joint LElbowYaw: axis 0 0 1 -> 1.0 0 0; limit lower=-2.08567 upper=2.08567 effort=2.80815 velocity=7.33998 -> lower=-2.08567 upper=2.08567 effort=5.428 velocity=7.33998; origin xyz=0.015 -0.1812 0.00013 rpy=1.41372 -0 0 -> xyz=0.1812 0.015 0.00013 rpy=0 -0.157079 0
- joint LFinger11: axis 0 0 1 -> 0 0 1.0; origin xyz=-0.0268 0.004 0.0821 rpy=1.78277 -0.529825 -1.59039 -> xyz=0.0821 -0.0268 0.004 rpy=1.74402 1.04064 -0.0334335
- joint LFinger12: axis 0 0 1 -> 0 0 1.0; origin xyz=0.018 0 0 rpy=-0 -0 -1.0472 -> xyz=0.018 0 0 rpy=0 0 -1.0472
- joint LFinger13: axis 0 0 1 -> 0 0 1.0; origin xyz=0.018 0 0 rpy=-0 -0 -1.0472 -> xyz=0.018 0 0 rpy=0 0 -1.0472
- joint LFinger21: axis 0 0 1 -> 0 0 1.0; origin xyz=-0.0073 0.006 0.0873 rpy=1.6413 -0.522522 -1.60603 -> xyz=0.0873 -0.0073 0.006 rpy=1.5708 1.0472 -0.061086
- joint LFinger22: axis 0 0 1 -> 0 0 1.0; origin xyz=0.018 0 0 rpy=-0 -0 -1.0472 -> xyz=0.018 0 0 rpy=0 0 -1.0472
- joint LFinger23: axis 0 0 1 -> 0 0 1.0; origin xyz=0.018 0 0 rpy=-0 -0 -1.0472 -> xyz=0.018 0 0 rpy=0 0 -1.0472
- joint LFinger31: axis 0 0 1 -> 0 0 1.0; origin xyz=0.0123 0.004 0.0833 rpy=1.50025 -0.525718 -1.58781 -> xyz=0.0833 0.0123 0.004 rpy=1.46636 1.04483 -0.029314
- joint LFinger32: axis 0 0 1 -> 0 0 1.0; origin xyz=0.018 0 0 rpy=-0 -0 -1.0472 -> xyz=0.018 0 0 rpy=0 0 -1.0472
- joint LFinger33: axis 0 0 1 -> 0 0 1.0; origin xyz=0.018 0 0 rpy=-0 -0 -1.0472 -> xyz=0.018 0 0 rpy=0 0 -1.0472
- joint LFinger41: axis 0 0 1 -> 0 0 1.0; origin xyz=0.0309 0 0.074 rpy=1.3184 -0.528785 -1.53079 -> xyz=0.074 0.0309 0 rpy=1.39757 1.04064 0.0683394
- joint LFinger42: axis 0 0 1 -> 0 0 1.0; origin xyz=0.018 0 0 rpy=-0 -0 -1.0472 -> xyz=0.018 0 0 rpy=0 0 -1.0472
- joint LFinger43: axis 0 0 1 -> 0 0 1.0; origin xyz=0.018 0 0 rpy=-0 -0 -1.0472 -> xyz=0.018 0 0 rpy=0 0 -1.0472
- joint LHand: axis 1 0 0 -> 1.0 0 0; child LHand_actuator_frame -> l_gripper; limit lower=0.02 upper=0.98 effort=0.096152 velocity=12.56 -> lower=0.02 upper=0.98 effort=0.144 velocity=12.56; origin xyz=0 0 0.025 rpy=1.5708 -1.5708 -3.14159 -> xyz=0.025 0 0 rpy=0 0 0
- joint LShoulderPitch: axis 0 0 1 -> 0 1.0 0; child LShoulderPitch -> LShoulder; limit lower=-2.08567 upper=2.08567 effort=4.11862 velocity=7.33998 -> lower=-2.08567 upper=2.08567 effort=5.428 velocity=7.33998; origin xyz=-0.057 0.14974 0.08682 rpy=-1.5708 -0 0 -> xyz=-0.057 0.14974 0.22582 rpy=0 0 0
- joint LShoulderRoll: axis 0 0 1 -> 0 0 1.0; limit lower=0.00872665 upper=1.56207 effort=3.70244 velocity=9.22756 -> lower=0.00872665 upper=1.56207 effort=2.666 velocity=9.22756; origin xyz=0 0 0 rpy=-1.5708 -1.5708 3.14159 -> xyz=0 0 0 rpy=0 0 0; parent LShoulderPitch -> LShoulder
- joint LThumb1: axis 0 0 1 -> 0 0 1.0; origin xyz=-0.0357 -0.0199 0.0482 rpy=-2.76225 -0.785789 -0.937585 -> xyz=0.0482 -0.0357 -0.0199 rpy=-1.95836 0.60626 0.533978
- joint LThumb2: axis 0 0 1 -> 0 0 1.0; origin xyz=0.022 0 0 rpy=-0 -0 -1.0472 -> xyz=0.022 0 0 rpy=0 0 -1.0472
- joint LWristYaw: axis 0 0 1 -> 1.0 0 0; limit lower=-1.82387 upper=1.82387 effort=0.134278 velocity=17.3835 -> lower=-1.82387 upper=1.82387 effort=0.2014 velocity=17.3835; origin xyz=0 -0.15 0 rpy=1.5708 -0 0 -> xyz=0.15 0 0 rpy=0 0 0
- joint RElbowRoll: axis 0 0 1 -> 0 0 1.0; limit lower=0.00872665 upper=1.56207 effort=2.22146 velocity=9.22756 -> lower=0.00872665 upper=1.56207 effort=2.666 velocity=9.22756; origin xyz=0 0 0 rpy=-1.5708 -0 0 -> xyz=0 0 0 rpy=0 0 0; parent RElbowYaw -> RElbow
- joint RElbowYaw: axis 0 0 1 -> 1.0 0 0; child RElbowYaw -> RElbow; limit lower=-2.08567 upper=2.08567 effort=2.80815 velocity=7.33998 -> lower=-2.08567 upper=2.08567 effort=5.428 velocity=7.33998; origin xyz=-0.015 -0.1812 0.00013 rpy=1.41372 -0 0 -> xyz=0.1812 -0.015 0.00013 rpy=0 -0.157079 0
- joint RFinger11: axis 0 0 1 -> 0 0 1.0; origin xyz=0.0268 0.004 0.0821 rpy=1.35882 -0.529825 -1.55121 -> xyz=0.0821 0.0268 0.004 rpy=1.39757 1.04064 0.0334335
- joint RFinger12: axis 0 0 1 -> 0 0 1.0; origin xyz=0.018 0 0 rpy=-0 -0 -1.0472 -> xyz=0.018 0 0 rpy=0 0 -1.0472
- joint RFinger13: axis 0 0 1 -> 0 0 1.0; origin xyz=0.018 0 0 rpy=-0 -0 -1.0472 -> xyz=0.018 0 0 rpy=0 0 -1.0472
- joint RFinger21: axis 0 0 1 -> 0 0 1.0; origin xyz=0.0073 0.006 0.0873 rpy=1.50029 -0.522522 -1.53556 -> xyz=0.0873 0.0073 0.006 rpy=1.5708 1.0472 0.061086
- joint RFinger22: axis 0 0 1 -> 0 0 1.0; origin xyz=0.018 0 0 rpy=-0 -0 -1.0472 -> xyz=0.018 0 0 rpy=0 0 -1.0472
- joint RFinger23: axis 0 0 1 -> 0 0 1.0; origin xyz=0.018 0 0 rpy=-0 -0 -1.0472 -> xyz=0.018 0 0 rpy=0 0 -1.0472
- joint RFinger31: axis 0 0 1 -> 0 0 1.0; origin xyz=-0.0123 0.004 0.0833 rpy=1.64134 -0.525718 -1.55378 -> xyz=0.0833 -0.0123 0.004 rpy=1.67523 1.04483 0.029316
- joint RFinger32: axis 0 0 1 -> 0 0 1.0; origin xyz=0.018 0 0 rpy=-0 -0 -1.0472 -> xyz=0.018 0 0 rpy=0 0 -1.0472
- joint RFinger33: axis 0 0 1 -> 0 0 1.0; origin xyz=0.018 0 0 rpy=-0 -0 -1.0472 -> xyz=0.018 0 0 rpy=0 0 -1.0472
- joint RFinger41: axis 0 0 1 -> 0 0 1.0; origin xyz=-0.0309 0 0.074 rpy=1.82319 -0.528785 -1.6108 -> xyz=0.074 -0.0309 0 rpy=1.74402 1.04064 -0.0683394
- joint RFinger42: axis 0 0 1 -> 0 0 1.0; origin xyz=0.018 0 0 rpy=-0 -0 -1.0472 -> xyz=0.018 0 0 rpy=0 0 -1.0472
- joint RFinger43: axis 0 0 1 -> 0 0 1.0; origin xyz=0.018 0 0 rpy=-0 -0 -1.0472 -> xyz=0.018 0 0 rpy=0 0 -1.0472
- joint RHand: axis 1 0 0 -> 1.0 0 0; child RHand_actuator_frame -> r_gripper; limit lower=0.02 upper=0.98 effort=0.096152 velocity=12.56 -> lower=0.02 upper=0.98 effort=0.144 velocity=12.56; origin xyz=0 0 0.025 rpy=1.5708 -1.5708 -3.14159 -> xyz=0.025 0 0 rpy=0 0 0
- joint RShoulderPitch: axis 0 0 1 -> 0 1.0 0; child RShoulderPitch -> RShoulder; limit lower=-2.08567 upper=2.08567 effort=4.11862 velocity=7.33998 -> lower=-2.08567 upper=2.08567 effort=5.428 velocity=7.33998; origin xyz=-0.057 -0.14974 0.08682 rpy=-1.5708 -0 0 -> xyz=-0.057 -0.14974 0.22582 rpy=0 0 0
- joint RShoulderRoll: axis 0 0 1 -> 0 0 1.0; limit lower=-1.56207 upper=-0.00872665 effort=3.70244 velocity=9.22756 -> lower=-1.56207 upper=-0.00872665 effort=2.666 velocity=9.22756; origin xyz=0 0 0 rpy=-1.5708 -1.5708 3.14159 -> xyz=0 0 0 rpy=0 0 0; parent RShoulderPitch -> RShoulder
- joint RThumb1: axis 0 0 1 -> 0 0 1.0; origin xyz=0.0357 -0.0199 0.0482 rpy=-0.379338 -0.785789 -2.20401 -> xyz=0.0482 0.0357 -0.0199 rpy=-1.18323 0.60626 -0.533978
- joint RThumb2: axis 0 0 1 -> 0 0 1.0; origin xyz=0.022 0 0 rpy=-0 -0 -1.0472 -> xyz=0.022 0 0 rpy=0 0 -1.0472
- joint RWristYaw: axis 0 0 1 -> 1.0 0 0; limit lower=-1.82387 upper=1.82387 effort=0.134278 velocity=17.3835 -> lower=-1.82387 upper=1.82387 effort=0.2014 velocity=17.3835; origin xyz=0 -0.15 0 rpy=1.5708 -0 0 -> xyz=0.15 0 0 rpy=0 0 0
- joint WheelB: axis 1 0 0 -> 1.0 0 0; origin xyz=-0.17 0.264 0 rpy=-1.5708 -0 -3.14159 -> xyz=-0.17 0 -0.264 rpy=0 0 -3.14159
- joint WheelFL: axis 1 0 0 -> 1.0 0 0; origin xyz=0.09 0.264 0.155 rpy=1.5708 -1.07517 -1.16723e-16 -> xyz=0.09 0.155 -0.264 rpy=0 0 1.07517
- joint WheelFR: axis 1 0 0 -> 1.0 0 0; origin xyz=0.09 0.264 -0.155 rpy=1.5708 1.07517 1.16723e-16 -> xyz=0.09 -0.155 -0.264 rpy=0 0 -1.07517
- joint base_link_fixedjoint: child torso -> Tibia; origin xyz=0 0 0 rpy=0 -0 0 -> xyz=0 0 0.334 rpy=0 0 0
