Commit message: remove l_gripper

File: pepper_robot_description/urdf/pepper_robot.urdf (robot description, URDF)
Before this commit: robot pepper_robot, 50 links, 49 joints
Links:
- link l_gripper: mass 2e-06 -> None
- link r_gripper: mass 2e-06 -> None

Commit message: remove l_gripper

File: pepper_robot_description/urdf/pepper_robot.urdf (robot description, URDF)
Before this commit: robot pepper_robot, 50 links, 49 joints
Links:
- removed link l_gripper
- removed link r_gripper
- added link LHand
- added link RHand
Joints:
- joint LHand: child l_gripper -> LHand
- joint RHand: child r_gripper -> RHand

Commit message: remove l_gripper failed

File: pepper_robot_description/urdf/pepper_robot.urdf (robot description, URDF)
Before this commit: robot pepper_robot, 50 links, 49 joints
Links:
- removed link LHand
- removed link RHand
- added link l_gripper, mass 2e-06
- added link r_gripper, mass 2e-06
Joints:
- joint LHand: child LHand -> l_gripper
- joint RHand: child RHand -> r_gripper

Commit message: fix total volume

File: pepper_robot_description/urdf/pepper_robot.urdf (robot description, URDF)
Before this commit: robot pepper_robot, 50 links, 49 joints
Links:
- link Head: mass 1.51893 -> 3.7955398538315377
- link Hip: mass 1.02338 -> 1.007402858772892
- link LBicep: mass 0.50527 -> 1e-10
- link LElbow: mass 0.27495 -> 0.07380464672624755
- link LForeArm: mass 0.16579 -> 0.13321114815783727
- link LShoulder: mass 0.3125 -> 0.1407150721615769
- link Neck: mass 0.27391 -> 0.09146568603258816
- link Pelvis: mass 2.45917 -> 3.7955398538315377
- link RBicep: mass 0.50527 -> 0.3137032437994389
- link RElbow: mass 0.27495 -> 0.07380464672624755
- link RForeArm: mass 0.16579 -> 0.13321114815783727
- link RShoulder: mass 0.3125 -> 0.1407150721615769
- link Tibia: mass 11.6015 -> 12.344158152172728
- link WheelB_link: mass 1.58028 -> 0.7575690266305116
- link WheelFL_link: mass 1.58028 -> 0.7575690379154867
- link WheelFR_link: mass 1.58028 -> 0.75756900450011
- link l_wrist: mass 0.27555 -> 0.207591874180564
- link r_wrist: mass 0.27555 -> 0.20759187418056393
- link torso: mass 3.99533 -> 4.89481724014063

Commit message: fix total volume

File: pepper_robot_description/urdf/pepper_robot.urdf (robot description, URDF)
Before this commit: robot pepper_robot, 50 links, 49 joints
Links:
- link LBicep: mass 1e-10 -> 0.3137032437994389

Commit message: fix inertial values in urdf

File: pepper_robot_description/urdf/pepper_robot.urdf (robot description, URDF)
Before this commit: robot pepper_robot, 50 links, 49 joints
Links:
- link LFinger11_link: mass 2e-06 -> 0.0017342022611750378
- link LFinger12_link: mass 2e-06 -> 0.001734202280194698
- link LFinger13_link: mass 2e-06 -> 0.001211966381471568
- link LFinger21_link: mass 2e-06 -> 0.0017342022480607796
- link LFinger22_link: mass 2e-06 -> 0.001734202428057582
- link LFinger23_link: mass 2e-06 -> 0.0012119663699255415
- link LFinger31_link: mass 2e-06 -> 0.001734202271258544
- link LFinger32_link: mass 2e-06 -> 0.0017342022235830492
- link LFinger33_link: mass 2e-06 -> 0.0012119665608007826
- link LFinger41_link: mass 2e-06 -> 0.0017342022888397826
- link LFinger42_link: mass 2e-06 -> 0.0017342022167828866
- link LFinger43_link: mass 2e-06 -> 0.0012119663070476055
- link LThumb1_link: mass 2e-06 -> 0.0017342022979805805
- link LThumb2_link: mass 2e-06 -> 0.001211966381471568
- link RFinger11_link: mass 2e-06 -> 0.0017342022611750378
- link RFinger12_link: mass 2e-06 -> 0.001734202280194698
- link RFinger13_link: mass 2e-06 -> 0.001211966381471568
- link RFinger21_link: mass 2e-06 -> 0.0017342022480607796
- link RFinger22_link: mass 2e-06 -> 0.001734202428057582
- link RFinger23_link: mass 2e-06 -> 0.0012119663699255415
- link RFinger31_link: mass 2e-06 -> 0.001734202271258544
- link RFinger32_link: mass 2e-06 -> 0.0017342022235830492
- link RFinger33_link: mass 2e-06 -> 0.0012119665608007826
- link RFinger41_link: mass 2e-06 -> 0.0017342022888397826
- link RFinger42_link: mass 2e-06 -> 0.0017342022167828866
- link RFinger43_link: mass 2e-06 -> 0.0012119663070476055
- link RThumb1_link: mass 2e-06 -> 0.0017342022979805805
- link RThumb2_link: mass 2e-06 -> 0.001211966381471568
- link l_gripper: mass 2e-06 -> 0.207591874180564
- link r_gripper: mass 2e-06 -> 0.20759187418056393

Commit message: test please work

File: pepper_robot_description/urdf/pepper_robot.urdf (robot description, URDF)
Before this commit: robot pepper_robot, 50 links, 49 joints
Links:
- added link BumperB_frame
- added link BumperFL_frame
- added link BumperFR_frame
- added link CameraBottom_frame
- added link CameraBottom_optical_frame
- added link CameraDepth_frame
- added link CameraDepth_optical_frame
- added link CameraTop_frame
- added link CameraTop_optical_frame
- added link ChestButton_frame
- added link HeadTouchFront_frame
- added link HeadTouchMiddle_frame
- added link HeadTouchRear_frame
- added link ImuBaseAccelerometer_frame
- added link ImuTorsoAccelerometer_frame
- added link ImuTorsoGyrometer_frame
- added link LHandTouchBack_frame
- added link LSpeaker_frame
- added link RHandTouchBack_frame
- added link RSpeaker_frame
- added link ShovelLaser_frame
- added link SonarBack_frame
- added link SonarFront_frame
- added link SurroundingFrontLaser_device_frame
- added link SurroundingFrontLaser_frame
- added link SurroundingLeftLaser_device_frame
- added link SurroundingLeftLaser_frame
- added link SurroundingRightLaser_device_frame
- added link SurroundingRightLaser_frame
- added link Tablet_frame
- added link VerticalLeftLaser_frame
- added link VerticalRightLaser_frame
- added link base_footprint
Joints:
- added joint AccelerometerBase_sensor_fixedjoint: type fixed, parent Tibia, child ImuBaseAccelerometer_frame, origin xyz=0.0147 -0.0017 -0.26319 rpy=0 0 0, axis 0 0 0
- added joint Accelerometer_sensor_fixedjoint: type fixed, parent torso, child ImuTorsoAccelerometer_frame, origin xyz=0.00239 -0.03575 0.00626 rpy=0 0 0, axis 0 0 0
- added joint Bumper/Back_sensor_fixedjoint: type fixed, parent Tibia, child BumperB_frame, origin xyz=-0.251 0 -0.264 rpy=0 0 -3.14159, axis 0 0 0
- added joint Bumper/FrontLeft_sensor_fixedjoint: type fixed, parent Tibia, child BumperFL_frame, origin xyz=0.129 0.227 -0.264 rpy=0 0 0.48886, axis 0 0 0
- added joint Bumper/FrontRight_sensor_fixedjoint: type fixed, parent Tibia, child BumperFR_frame, origin xyz=0.129 -0.227 -0.264 rpy=0 0 -0.48886, axis 0 0 0
- added joint CameraBottom_optical_frame_fixedjoint: type fixed, parent CameraBottom_frame, child CameraBottom_optical_frame, origin xyz=0 0 0 rpy=-1.57079632679 0 -1.57079632679
- added joint CameraBottom_sensor_fixedjoint: type fixed, parent Head, child CameraBottom_frame, origin xyz=0.09262 0 0.06177 rpy=0 0.698132 0, axis 0 0 0
- added joint CameraDepth_optical_frame_fixedjoint: type fixed, parent CameraDepth_frame, child CameraDepth_optical_frame, origin xyz=0 0 0 rpy=-1.57079632679 0 -1.57079632679
- added joint CameraDepth_sensor_fixedjoint: type fixed, parent Head, child CameraDepth_frame, origin xyz=0.05138 0.039 0.1194 rpy=0 0 0, axis 0 0 0
- added joint CameraTop_optical_frame_fixedjoint: type fixed, parent CameraTop_frame, child CameraTop_optical_frame, origin xyz=0 0 0 rpy=-1.57079632679 0 -1.57079632679
- added joint CameraTop_sensor_fixedjoint: type fixed, parent Head, child CameraTop_frame, origin xyz=0.08601 0 0.16284 rpy=0 0 0, axis 0 0 0
- added joint ChestBoard/Button_sensor_fixedjoint: type fixed, parent torso, child ChestButton_frame, origin xyz=0.049871 0.001588 0.055163 rpy=0 0 0, axis 0 0 0
- added joint Gyrometer_sensor_fixedjoint: type fixed, parent torso, child ImuTorsoGyrometer_frame, origin xyz=0.00204 -0.03491 -0.00959 rpy=0 0 0, axis 0 0 0
- added joint Head/Touch/Front_sensor_fixedjoint: type fixed, parent Head, child HeadTouchFront_frame, origin xyz=0.028175 0 0.21267 rpy=0 0.20944 0, axis 0 0 0
- added joint Head/Touch/Middle_sensor_fixedjoint: type fixed, parent Head, child HeadTouchMiddle_frame, origin xyz=0.0041 0 0.2159 rpy=0 -0.0349066 0, axis 0 0 0
- added joint Head/Touch/Rear_sensor_fixedjoint: type fixed, parent Head, child HeadTouchRear_frame, origin xyz=-0.03376 0 0.21052 rpy=0 -0.314159 0, axis 0 0 0
- added joint LHand/Touch/Back_sensor_fixedjoint: type fixed, parent l_wrist, child LHandTouchBack_frame, origin xyz=0.0523 0 0.0304 rpy=1.5708 -1.5708 -3.14159, axis 0 0 0
- added joint LaserSensor/Front_projected_sensor_fixedjoint: type fixed, parent Tibia, child SurroundingFrontLaser_frame, origin xyz=0.0562 0 -0.334 rpy=0 0 0, axis 0 0 0
- added joint LaserSensor/Front_sensor_fixedjoint: type fixed, parent Tibia, child SurroundingFrontLaser_device_frame, origin xyz=0.0562 0 -0.0692 rpy=0 0.349066 0, axis 0 0 0
- added joint LaserSensor/Left_projected_sensor_fixedjoint: type fixed, parent Tibia, child SurroundingLeftLaser_frame, origin xyz=-0.018 0.0899 -0.334 rpy=0 0 1.75728, axis 0 0 0
- added joint LaserSensor/Left_sensor_fixedjoint: type fixed, parent Tibia, child SurroundingLeftLaser_device_frame, origin xyz=-0.018 0.0899 -0.0759 rpy=0 0.349066 1.5708, axis 0 0 0
- added joint LaserSensor/Right_projected_sensor_fixedjoint: type fixed, parent Tibia, child SurroundingRightLaser_frame, origin xyz=-0.018 -0.0899 -0.334 rpy=0 0 -1.75728, axis 0 0 0
- added joint LaserSensor/Right_sensor_fixedjoint: type fixed, parent Tibia, child SurroundingRightLaser_device_frame, origin xyz=-0.018 -0.0899 -0.0759 rpy=0 0.349066 -1.5708, axis 0 0 0
- added joint LaserSensor/Shovel_sensor_fixedjoint: type fixed, parent Tibia, child ShovelLaser_frame, origin xyz=0.0562 0 -0.0692 rpy=0 0.349066 0, axis 0 0 0
- added joint LaserSensor/VerticalLeft_sensor_fixedjoint: type fixed, parent Tibia, child VerticalLeftLaser_frame, origin xyz=0.0562 0 -0.0692 rpy=0 0.349066 0, axis 0 0 0
- added joint LaserSensor/VerticalRight_sensor_fixedjoint: type fixed, parent Tibia, child VerticalRightLaser_frame, origin xyz=0.0562 0 -0.0692 rpy=0 0.349066 0, axis 0 0 0
- added joint RHand/Touch/Back_sensor_fixedjoint: type fixed, parent r_wrist, child RHandTouchBack_frame, origin xyz=0.0523 0 0.0304 rpy=1.5708 -1.5708 -3.14159, axis 0 0 0
- added joint Sonar/Back_sensor_fixedjoint: type fixed, parent Tibia, child SonarBack_frame, origin xyz=-0.0718 0 -0.0534 rpy=-1.81761e-08 -0.209438 -3.14159, axis 0 0 0
- added joint Sonar/Front_sensor_fixedjoint: type fixed, parent Tibia, child SonarFront_frame, origin xyz=0.0699 0 -0.1023 rpy=0 -0.322858 0, axis 0 0 0
- added joint SpeakerLeft_sensor_fixedjoint: type fixed, parent Head, child LSpeaker_frame, origin xyz=0 0 0 rpy=0 0 0, axis 0 0 0
- added joint SpeakerRight_sensor_fixedjoint: type fixed, parent Head, child RSpeaker_frame, origin xyz=0 0 0 rpy=0 0 0, axis 0 0 0
- added joint Tablet_sensor_fixedjoint: type fixed, parent torso, child Tablet_frame, origin xyz=0.0839249 0 0.06251 rpy=0 -0.523599 0, axis 0 0 0
- added joint base_footprint_joint: type fixed, parent Tibia, child base_footprint, origin xyz=0 0 -0.334 rpy=0 0 0
- joint HeadPitch: limit lower=-0.706858 upper=0.4451 effort=2.666 velocity=9.22756 -> lower=-0.706858 upper=0.637045 effort=2.666 velocity=9.22756
- joint HeadYaw: origin xyz=-0.038 0 0.3089 rpy=0 0 0 -> xyz=-0.038 0 0.1699 rpy=0 0 0
- joint HipPitch: axis 0 -1.0 0 -> 0 1.0 0; child Hip -> Pelvis; origin xyz=0 0 0.268 rpy=0 0 0 -> xyz=0 0 -0.079 rpy=0 0 0; parent Pelvis -> Hip
- joint HipRoll: axis -1.0 0 0 -> 1.0 0 0; child torso -> Hip; origin xyz=0 0 0.079 rpy=0 0 0 -> xyz=2e-05 0 -0.139 rpy=0 0 0; parent Hip -> torso
- joint KneePitch: axis 0 -1.0 0 -> 0 1.0 0; child Pelvis -> Tibia; origin xyz=0 0 0 rpy=0 0 0 -> xyz=0 0 -0.268 rpy=0 0 0; parent Tibia -> Pelvis
- joint LShoulderPitch: origin xyz=-0.057 0.14974 0.22582 rpy=0 0 0 -> xyz=-0.057 0.14974 0.08682 rpy=0 0 0
- joint RShoulderPitch: origin xyz=-0.057 -0.14974 0.22582 rpy=0 0 0 -> xyz=-0.057 -0.14974 0.08682 rpy=0 0 0
- joint base_link_fixedjoint: child Tibia -> torso; origin xyz=0 0 0.334 rpy=0 0 0 -> xyz=0 0 0 rpy=0 0 0

Commit message: test please work

File: pepper_robot_description/urdf/pepper_robot.urdf (robot description, URDF)
Before this commit: robot pepper_robot, 83 links, 82 joints
Links:
- removed link BumperB_frame
- removed link BumperFL_frame
- removed link BumperFR_frame
- removed link CameraBottom_frame
- removed link CameraBottom_optical_frame
- removed link CameraDepth_frame
- removed link CameraDepth_optical_frame
- removed link CameraTop_frame
- removed link CameraTop_optical_frame
- removed link ChestButton_frame
- removed link HeadTouchFront_frame
- removed link HeadTouchMiddle_frame
- removed link HeadTouchRear_frame
- removed link ImuBaseAccelerometer_frame
- removed link ImuTorsoAccelerometer_frame
- removed link ImuTorsoGyrometer_frame
- removed link LHandTouchBack_frame
- removed link LSpeaker_frame
- removed link RHandTouchBack_frame
- removed link RSpeaker_frame
- removed link ShovelLaser_frame
- removed link SonarBack_frame
- removed link SonarFront_frame
- removed link SurroundingFrontLaser_device_frame
- removed link SurroundingFrontLaser_frame
- removed link SurroundingLeftLaser_device_frame
- removed link SurroundingLeftLaser_frame
- removed link SurroundingRightLaser_device_frame
- removed link SurroundingRightLaser_frame
- removed link Tablet_frame
- removed link VerticalLeftLaser_frame
- removed link VerticalRightLaser_frame
- removed link base_footprint
Joints:
- removed joint AccelerometerBase_sensor_fixedjoint
- removed joint Accelerometer_sensor_fixedjoint
- removed joint Bumper/Back_sensor_fixedjoint
- removed joint Bumper/FrontLeft_sensor_fixedjoint
- removed joint Bumper/FrontRight_sensor_fixedjoint
- removed joint CameraBottom_optical_frame_fixedjoint
- removed joint CameraBottom_sensor_fixedjoint
- removed joint CameraDepth_optical_frame_fixedjoint
- removed joint CameraDepth_sensor_fixedjoint
- removed joint CameraTop_optical_frame_fixedjoint
- removed joint CameraTop_sensor_fixedjoint
- removed joint ChestBoard/Button_sensor_fixedjoint
- removed joint Gyrometer_sensor_fixedjoint
- removed joint Head/Touch/Front_sensor_fixedjoint
- removed joint Head/Touch/Middle_sensor_fixedjoint
- removed joint Head/Touch/Rear_sensor_fixedjoint
- removed joint LHand/Touch/Back_sensor_fixedjoint
- removed joint LaserSensor/Front_projected_sensor_fixedjoint
- removed joint LaserSensor/Front_sensor_fixedjoint
- removed joint LaserSensor/Left_projected_sensor_fixedjoint
- removed joint LaserSensor/Left_sensor_fixedjoint
- removed joint LaserSensor/Right_projected_sensor_fixedjoint
- removed joint LaserSensor/Right_sensor_fixedjoint
- removed joint LaserSensor/Shovel_sensor_fixedjoint
- removed joint LaserSensor/VerticalLeft_sensor_fixedjoint
- removed joint LaserSensor/VerticalRight_sensor_fixedjoint
- removed joint RHand/Touch/Back_sensor_fixedjoint
- removed joint Sonar/Back_sensor_fixedjoint
- removed joint Sonar/Front_sensor_fixedjoint
- removed joint SpeakerLeft_sensor_fixedjoint
- removed joint SpeakerRight_sensor_fixedjoint
- removed joint Tablet_sensor_fixedjoint
- removed joint base_footprint_joint
- joint HeadPitch: limit lower=-0.706858 upper=0.637045 effort=2.666 velocity=9.22756 -> lower=-0.706858 upper=0.4451 effort=2.666 velocity=9.22756
- joint HeadYaw: origin xyz=-0.038 0 0.1699 rpy=0 0 0 -> xyz=-0.038 0 0.3089 rpy=0 0 0
- joint HipPitch: axis 0 1.0 0 -> 0 -1.0 0; child Pelvis -> Hip; origin xyz=0 0 -0.079 rpy=0 0 0 -> xyz=0 0 0.268 rpy=0 0 0; parent Hip -> Pelvis
- joint HipRoll: axis 1.0 0 0 -> -1.0 0 0; child Hip -> torso; origin xyz=2e-05 0 -0.139 rpy=0 0 0 -> xyz=0 0 0.079 rpy=0 0 0; parent torso -> Hip
- joint KneePitch: axis 0 1.0 0 -> 0 -1.0 0; child Tibia -> Pelvis; origin xyz=0 0 -0.268 rpy=0 0 0 -> xyz=0 0 0 rpy=0 0 0; parent Pelvis -> Tibia
- joint LShoulderPitch: origin xyz=-0.057 0.14974 0.08682 rpy=0 0 0 -> xyz=-0.057 0.14974 0.22582 rpy=0 0 0
- joint RShoulderPitch: origin xyz=-0.057 -0.14974 0.08682 rpy=0 0 0 -> xyz=-0.057 -0.14974 0.22582 rpy=0 0 0
- joint base_link_fixedjoint: child torso -> Tibia; origin xyz=0 0 0 rpy=0 0 0 -> xyz=0 0 0.334 rpy=0 0 0

Commit message: change initial_joint_positions

File: pepper_robot_description/urdf/pepper_robot.urdf (robot description, URDF)
Before this commit: robot pepper_robot, 50 links, 49 joints
Joints:
- joint HipRoll: type revolute -> fixed

Commit message: change initial_joint_positions

File: pepper_robot_description/urdf/pepper_robot.urdf (robot description, URDF)
Before this commit: robot pepper_robot, 50 links, 49 joints
Joints:
- joint HipRoll: type fixed -> continuous

Commit message: test

File: pepper_robot_description/urdf/pepper_robot.urdf (robot description, URDF)
Before this commit: robot pepper_robot, 50 links, 49 joints
Joints:
- joint HipRoll: limit lower=-0.514872 upper=0.514872 effort=10.1884 velocity=2.27032 -> lower=0.214872 upper=0.514872 effort=10.1884 velocity=2.27032; type continuous -> revolute

Commit message: test

File: pepper_robot_description/urdf/pepper_robot.urdf (robot description, URDF)
Before this commit: robot pepper_robot, 50 links, 49 joints
Joints:
- joint HipRoll: limit lower=0.214872 upper=0.514872 effort=10.1884 velocity=2.27032 -> lower=-0.514872 upper=0.514872 effort=10.1884 velocity=2.27032

Commit message: test

File: pepper_robot_description/urdf/pepper_robot.urdf (robot description, URDF)
Before this commit: robot pepper_robot, 50 links, 49 joints
Joints:
- joint HipRoll: limit lower=-0.514872 upper=0.514872 effort=10.1884 velocity=2.27032 -> lower=-0.514872 upper=0.514872 effort=2.1884 velocity=2.27032

Commit message: test

File: pepper_robot_description/urdf/pepper_robot.urdf (robot description, URDF)
Before this commit: robot pepper_robot, 50 links, 49 joints
Joints:
- joint HipRoll: limit lower=-0.514872 upper=0.514872 effort=2.1884 velocity=2.27032 -> lower=-0.514872 upper=0.514872 effort=10.1884 velocity=2.27032

Commit message: test

File: pepper_robot_description/urdf/pepper_robot.urdf (robot description, URDF)
Before this commit: robot pepper_robot, 50 links, 49 joints
Joints:
- joint HipRoll: limit lower=-0.514872 upper=0.514872 effort=10.1884 velocity=2.27032 -> lower=-15 upper=15 effort=10.1884 velocity=2.27032
- joint LShoulderPitch: limit lower=-2.08567 upper=2.08567 effort=5.428 velocity=7.33998 -> lower=-10 upper=10 effort=5.428 velocity=2
- joint RShoulderPitch: limit lower=-2.08567 upper=2.08567 effort=5.428 velocity=7.33998 -> lower=-10 upper=10 effort=5.428 velocity=2

Commit message: test

File: pepper_robot_description/urdf/pepper_robot.urdf (robot description, URDF)
Before this commit: robot pepper_robot, 50 links, 49 joints
Joints:
- joint HipRoll: limit lower=-15 upper=15 effort=10.1884 velocity=2.27032 -> lower=-0.514872 upper=0.514872 effort=10.1884 velocity=2.27032
- joint LShoulderPitch: limit lower=-10 upper=10 effort=5.428 velocity=2 -> lower=-0.08567 upper=0.08567 effort=5.428 velocity=7.33998
- joint RShoulderPitch: limit lower=-10 upper=10 effort=5.428 velocity=2 -> lower=-0.08567 upper=0.08567 effort=5.428 velocity=7.33998

Commit message: test

File: pepper_robot_description/urdf/pepper_robot.urdf (robot description, URDF)
Before this commit: robot pepper_robot, 50 links, 49 joints
Joints:
- joint HipPitch: limit lower=-1.03847 upper=1.03847 effort=19.787 velocity=2.93276 -> lower=-1.03847 upper=1.03847 effort=0 velocity=2.93276
- joint HipRoll: limit lower=-0.514872 upper=0.514872 effort=10.1884 velocity=2.27032 -> lower=-0.514872 upper=0.514872 effort=0 velocity=2.27032
- joint LShoulderPitch: limit lower=-0.08567 upper=0.08567 effort=5.428 velocity=7.33998 -> lower=-2.08567 upper=2.08567 effort=0 velocity=7.33998
- joint RShoulderPitch: limit lower=-0.08567 upper=0.08567 effort=5.428 velocity=7.33998 -> lower=-2.08567 upper=2.08567 effort=0 velocity=7.33998

Commit message: test

File: pepper_robot_description/urdf/pepper_robot.urdf (robot description, URDF)
Before this commit: robot pepper_robot, 50 links, 49 joints
Links:
- link Hip: mass 1.007402858772892 -> 3
Joints:
- joint HipPitch: limit lower=-1.03847 upper=1.03847 effort=0 velocity=2.93276 -> lower=-1.03847 upper=1.03847 effort=19.787 velocity=2.93276
- joint HipRoll: limit lower=-0.514872 upper=0.514872 effort=0 velocity=2.27032 -> lower=-0.514872 upper=0.514872 effort=10.1884 velocity=2.27032
- joint LShoulderPitch: limit lower=-2.08567 upper=2.08567 effort=0 velocity=7.33998 -> lower=-2.08567 upper=2.08567 effort=5.428 velocity=7.33998
- joint RShoulderPitch: limit lower=-2.08567 upper=2.08567 effort=0 velocity=7.33998 -> lower=-2.08567 upper=2.08567 effort=5.428 velocity=7.33998

Commit message: test

File: pepper_robot_description/urdf/pepper_robot.urdf (robot description, URDF)
Before this commit: robot pepper_robot, 50 links, 49 joints
Links:
- link Hip: mass 3 -> 5

Commit message: test

File: pepper_robot_description/urdf/pepper_robot.urdf (robot description, URDF)
Before this commit: robot pepper_robot, 50 links, 49 joints
Links:
- link Hip: mass 5 -> 7
- link Pelvis: mass 3.7955398538315377 -> 5

Commit message: test

File: pepper_robot_description/urdf/pepper_robot.urdf (robot description, URDF)
Before this commit: robot pepper_robot, 50 links, 49 joints
Links:
- link Hip: mass 7 -> 10
Joints:
- joint HipPitch: limit lower=-1.03847 upper=1.03847 effort=19.787 velocity=2.93276 -> lower=-1.03847 upper=1.03847 effort=19.787 velocity=0
- joint HipRoll: limit lower=-0.514872 upper=0.514872 effort=10.1884 velocity=2.27032 -> lower=-0.514872 upper=0.514872 effort=10.1884 velocity=0

Commit message: test

File: pepper_robot_description/urdf/pepper_robot.urdf (robot description, URDF)
Before this commit: robot pepper_robot, 50 links, 49 joints
Links:
- link Hip: mass 10 -> 1.007402858772892
- link Pelvis: mass 5 -> 3.7955398538315377
Joints:
- joint HipPitch: limit lower=-1.03847 upper=1.03847 effort=19.787 velocity=0 -> lower=-1.03847 upper=1.03847 effort=19.787 velocity=2.93276
- joint HipRoll: limit lower=-0.514872 upper=0.514872 effort=10.1884 velocity=0 -> lower=-0.514872 upper=0.514872 effort=10.1884 velocity=2.27032
