Commit message: test

File: pepper_robot_description/urdf/pepper_robot.urdf (robot description, URDF)
Before this commit: robot pepper_robot, 50 links, 49 joints
Joints:
- joint HeadPitch: limit lower=-0.706858 upper=0.4451 effort=2.666 velocity=0 -> lower=-0.706858 upper=0.4451 effort=0 velocity=0
- joint HeadYaw: limit lower=-2.08567 upper=2.08567 effort=5.428 velocity=0 -> lower=-2.08567 upper=2.08567 effort=0 velocity=0
- joint HipPitch: limit lower=-1.03847 upper=1.03847 effort=19.787 velocity=0 -> lower=-1.03847 upper=1.03847 effort=0 velocity=0
- joint HipRoll: limit lower=-0.514872 upper=0.514872 effort=10.1884 velocity=0 -> lower=-0.514872 upper=0.514872 effort=0 velocity=0
- joint KneePitch: limit lower=-0.514872 upper=0.514872 effort=27.702 velocity=0 -> lower=-0.514872 upper=0.514872 effort=0 velocity=0
- joint LElbowRoll: limit lower=-1.56207 upper=-0.00872665 effort=2.666 velocity=0 -> lower=-1.56207 upper=-0.00872665 effort=0 velocity=0
- joint LElbowYaw: limit lower=-2.08567 upper=2.08567 effort=5.428 velocity=0 -> lower=-2.08567 upper=2.08567 effort=0 velocity=0
- joint LHand: limit lower=0.02 upper=0.98 effort=0.144 velocity=0 -> lower=0.02 upper=0.98 effort=0 velocity=0
- joint LShoulderPitch: limit lower=-2.08567 upper=2.08567 effort=5.428 velocity=0 -> lower=-2.08567 upper=2.08567 effort=0 velocity=0
- joint LShoulderRoll: limit lower=0.00872665 upper=1.56207 effort=2.666 velocity=0 -> lower=0.00872665 upper=1.56207 effort=0 velocity=0
- joint LWristYaw: limit lower=-1.82387 upper=1.82387 effort=0.2014 velocity=0 -> lower=-1.82387 upper=1.82387 effort=0 velocity=0
- joint RElbowRoll: limit lower=0.00872665 upper=1.56207 effort=2.666 velocity=0 -> lower=0.00872665 upper=1.56207 effort=0 velocity=0
- joint RElbowYaw: limit lower=-2.08567 upper=2.08567 effort=5.428 velocity=0 -> lower=-2.08567 upper=2.08567 effort=0 velocity=0
- joint RHand: limit lower=0.02 upper=0.98 effort=0.144 velocity=0 -> lower=0.02 upper=0.98 effort=0 velocity=0
- joint RShoulderPitch: limit lower=-2.08567 upper=2.08567 effort=5.428 velocity=0 -> lower=-2.08567 upper=2.08567 effort=0 velocity=0
- joint RShoulderRoll: limit lower=-1.56207 upper=-0.00872665 effort=2.666 velocity=0 -> lower=-1.56207 upper=-0.00872665 effort=0 velocity=0
- joint RWristYaw: limit lower=-1.82387 upper=1.82387 effort=0.2014 velocity=0 -> lower=-1.82387 upper=1.82387 effort=0 velocity=0
- joint WheelB: limit lower=0 upper=0 effort=3.25 velocity=0 -> lower=0 upper=0 effort=0 velocity=0
- joint WheelFL: limit lower=0 upper=0 effort=3.25 velocity=0 -> lower=0 upper=0 effort=0 velocity=0
- joint WheelFR: limit lower=0 upper=0 effort=3.25 velocity=0 -> lower=0 upper=0 effort=0 velocity=0

Commit message: test

File: pepper_robot_description/urdf/pepper_robot.urdf (robot description, URDF)
Before this commit: robot pepper_robot, 50 links, 49 joints
Joints:
- joint HeadPitch: limit lower=-0.706858 upper=0.4451 effort=0 velocity=0 -> lower=-0.706858 upper=0.4451 effort=2.666 velocity=9.22756
- joint HeadYaw: limit lower=-2.08567 upper=2.08567 effort=0 velocity=0 -> lower=-2.08567 upper=2.08567 effort=5.428 velocity=7.33998
- joint HipPitch: limit lower=-1.03847 upper=1.03847 effort=0 velocity=0 -> lower=-1.03847 upper=1.03847 effort=19.787 velocity=2.93276
- joint HipRoll: limit lower=-0.514872 upper=0.514872 effort=0 velocity=0 -> lower=-0.514872 upper=0.514872 effort=10.1884 velocity=2.27032
- joint KneePitch: limit lower=-0.514872 upper=0.514872 effort=0 velocity=0 -> lower=-0.514872 upper=0.514872 effort=27.702 velocity=2.93276
- joint LElbowRoll: limit lower=-1.56207 upper=-0.00872665 effort=0 velocity=0 -> lower=-1.56207 upper=-0.00872665 effort=2.666 velocity=9.22756
- joint LElbowYaw: limit lower=-2.08567 upper=2.08567 effort=0 velocity=0 -> lower=-2.08567 upper=2.08567 effort=5.428 velocity=7.33998
- joint LHand: limit lower=0.02 upper=0.98 effort=0 velocity=0 -> lower=0.02 upper=0.98 effort=0.144 velocity=12.56
- joint LShoulderPitch: limit lower=-2.08567 upper=2.08567 effort=0 velocity=0 -> lower=-2.08567 upper=2.08567 effort=5.428 velocity=7.33998
- joint LShoulderRoll: limit lower=0.00872665 upper=1.56207 effort=0 velocity=0 -> lower=0.00872665 upper=1.56207 effort=2.666 velocity=9.22756
- joint LWristYaw: limit lower=-1.82387 upper=1.82387 effort=0 velocity=0 -> lower=-1.82387 upper=1.82387 effort=0.2014 velocity=17.3835
- joint RElbowRoll: limit lower=0.00872665 upper=1.56207 effort=0 velocity=0 -> lower=0.00872665 upper=1.56207 effort=2.666 velocity=9.22756
- joint RElbowYaw: limit lower=-2.08567 upper=2.08567 effort=0 velocity=0 -> lower=-2.08567 upper=2.08567 effort=5.428 velocity=7.33998
- joint RHand: limit lower=0.02 upper=0.98 effort=0 velocity=0 -> lower=0.02 upper=0.98 effort=0.144 velocity=12.56
- joint RShoulderPitch: limit lower=-2.08567 upper=2.08567 effort=0 velocity=0 -> lower=-2.08567 upper=2.08567 effort=5.428 velocity=7.33998
- joint RShoulderRoll: limit lower=-1.56207 upper=-0.00872665 effort=0 velocity=0 -> lower=-1.56207 upper=-0.00872665 effort=2.666 velocity=9.22756
- joint RWristYaw: limit lower=-1.82387 upper=1.82387 effort=0 velocity=0 -> lower=-1.82387 upper=1.82387 effort=0.2014 velocity=17.3835
- joint WheelB: limit lower=0 upper=0 effort=0 velocity=0 -> lower=0 upper=0 effort=3.25 velocity=6.28319
- joint WheelFL: limit lower=0 upper=0 effort=0 velocity=0 -> lower=0 upper=0 effort=3.25 velocity=6.28319
- joint WheelFR: limit lower=0 upper=0 effort=0 velocity=0 -> lower=0 upper=0 effort=3.25 velocity=6.28319

Commit message: test

File: pepper_robot_description/urdf/pepper_robot.urdf (robot description, URDF)
Before this commit: robot pepper_robot, 50 links, 49 joints
Links:
- link Head: mass 3.7955398538315377 -> 1.5189
- link Hip: mass 1.007402858772892 -> 1.0234
- link LBicep: mass 0.3137032437994389 -> 0.50527
- link LElbow: mass 0.07380464672624755 -> 0.27495
- link LFinger11_link: mass 0.0017342022611750378 -> 2e-06
- link LFinger12_link: mass 0.001734202280194698 -> 2e-06
- link LFinger13_link: mass 0.001211966381471568 -> 2e-06
- link LFinger21_link: mass 0.0017342022480607796 -> 2e-06
- link LFinger22_link: mass 0.001734202428057582 -> 2e-06
- link LFinger23_link: mass 0.0012119663699255415 -> 2e-06
- link LFinger31_link: mass 0.001734202271258544 -> 2e-06
- link LFinger32_link: mass 0.0017342022235830492 -> 2e-06
- link LFinger33_link: mass 0.0012119665608007826 -> 2e-06
- link LFinger41_link: mass 0.0017342022888397826 -> 2e-06
- link LFinger42_link: mass 0.0017342022167828866 -> 2e-06
- link LFinger43_link: mass 0.0012119663070476055 -> 2e-06
- link LForeArm: mass 0.13321114815783727 -> 0.16579
- link LShoulder: mass 0.1407150721615769 -> 0.3125
- link LThumb1_link: mass 0.0017342022979805805 -> 2e-06
- link LThumb2_link: mass 0.001211966381471568 -> 2e-06
- link Neck: mass 0.09146568603258816 -> 0.27391
- link Pelvis: mass 3.7955398538315377 -> 2.4592
- link RBicep: mass 0.3137032437994389 -> 0.50527
- link RElbow: mass 0.07380464672624755 -> 0.27495
- link RFinger11_link: mass 0.0017342022611750378 -> 2e-06
- link RFinger12_link: mass 0.001734202280194698 -> 2e-06
- link RFinger13_link: mass 0.001211966381471568 -> 2e-06
- link RFinger21_link: mass 0.0017342022480607796 -> 2e-06
- link RFinger22_link: mass 0.001734202428057582 -> 2e-06
- link RFinger23_link: mass 0.0012119663699255415 -> 2e-06
- link RFinger31_link: mass 0.001734202271258544 -> 2e-06
- link RFinger32_link: mass 0.0017342022235830492 -> 2e-06
- link RFinger33_link: mass 0.0012119665608007826 -> 2e-06
- link RFinger41_link: mass 0.0017342022888397826 -> 2e-06
- link RFinger42_link: mass 0.0017342022167828866 -> 2e-06
- link RFinger43_link: mass 0.0012119663070476055 -> 2e-06
- link RForeArm: mass 0.13321114815783727 -> 0.16579
- link RShoulder: mass 0.1407150721615769 -> 0.3125
- link RThumb1_link: mass 0.0017342022979805805 -> 2e-06
- link RThumb2_link: mass 0.001211966381471568 -> 2e-06
- link Tibia: mass 12.344158152172728 -> 15.485
- link WheelB_link: mass 0.7575690266305116 -> 0.05872
- link WheelFL_link: mass 0.7575690379154867 -> 0.05872
- link WheelFR_link: mass 0.75756900450011 -> 0.05872
- link l_gripper: mass 0.207591874180564 -> 2e-06
- link l_wrist: mass 0.207591874180564 -> 0.27555
- link r_gripper: mass 0.20759187418056393 -> 2e-06
- link r_wrist: mass 0.20759187418056393 -> 0.27555
- link torso: mass 4.89481724014063 -> 3.9953
Joints:
- joint HipPitch: limit lower=-1.03847 upper=1.03847 effort=19.787 velocity=2.93276 -> lower=-1.0385 upper=1.0385 effort=19.787 velocity=2.93276
- joint HipRoll: limit lower=-0.514872 upper=0.514872 effort=10.1884 velocity=2.27032 -> lower=-0.5149 upper=0.5149 effort=10.1884 velocity=2.27032
- joint KneePitch: limit lower=-0.514872 upper=0.514872 effort=27.702 velocity=2.93276 -> lower=-0.5149 upper=0.5149 effort=27.702 velocity=2.93276
- joint RElbowRoll: limit lower=0.00872665 upper=1.56207 effort=2.666 velocity=9.22756 -> lower=0.0087 upper=1.5620 effort=2.666 velocity=9.22756
- joint RWristYaw: limit lower=-1.82387 upper=1.82387 effort=0.2014 velocity=17.3835 -> lower=-1.8239 upper=1.8239 effort=0.2014 velocity=17.3835

Commit message: test

File: pepper_robot_description/urdf/pepper_robot.urdf (robot description, URDF)
Before this commit: robot pepper_robot, 50 links, 49 joints
Joints:
- joint LElbowRoll: limit lower=-1.56207 upper=-0.00872665 effort=2.666 velocity=9.22756 -> lower=-1.5620 upper=-0.0087 effort=2.666 velocity=9.22756
- joint LElbowYaw: limit lower=-2.08567 upper=2.08567 effort=5.428 velocity=7.33998 -> lower=-2.0857 upper=2.0857 effort=5.428 velocity=7.33998
- joint LShoulderPitch: limit lower=-2.08567 upper=2.08567 effort=5.428 velocity=7.33998 -> lower=-2.0857 upper=2.0857 effort=5.428 velocity=7.33998
- joint LShoulderRoll: limit lower=0.00872665 upper=1.56207 effort=2.666 velocity=9.22756 -> lower=0.0087 upper=1.56207 effort=2.666 velocity=9.22756
- joint LWristYaw: limit lower=-1.82387 upper=1.82387 effort=0.2014 velocity=17.3835 -> lower=-1.8239 upper=1.8239 effort=0.2014 velocity=17.3835

Commit message: test with new inertial properties

File: pepper_robot_description/urdf/pepper_robot.urdf (robot description, URDF)
Before this commit: robot pepper_robot, 50 links, 49 joints
Links:
- link WheelB_link: mass 0.05872 -> 0.804686790979882
- link WheelFL_link: mass 0.05872 -> 0.8046868029667374
- link WheelFR_link: mass 0.05872 -> 0.804686767473058

Commit message: test with new inertial properties

File: pepper_robot_description/urdf/pepper_robot.urdf (robot description, URDF)
Before this commit: robot pepper_robot, 50 links, 49 joints
Links:
- link Head: mass 1.5189 -> 3.7955398538315377
- link Hip: mass 1.0234 -> 1.007402858772892
- link LBicep: mass 0.50527 -> 0.3137032437994389
- link LElbow: mass 0.27495 -> 0.07380464672624755
- link LFinger11_link: mass 2e-06 -> 0.0017342022611750378
- link LFinger12_link: mass 2e-06 -> 0.001734202280194698
- link LFinger13_link: mass 2e-06 -> 0.001211966381471568
- link LFinger21_link: mass 2e-06 -> 0.0017342022480607796
- link LFinger22_link: mass 2e-06 -> 0.001734202428057582
- link LFinger23_link: mass 2e-06 -> 0.0012119663699255415
- link LFinger31_link: mass 2e-06 -> 0.001734202271258544
- link LFinger32_link: mass 2e-06 -> 0.0017342022235830492
- link LFinger33_link: mass 2e-06 -> 0.0012119665608007826
- link LFinger41_link: mass 2e-06 -> 0.0017342022888397826
- link LFinger42_link: mass 2e-06 -> 0.0017342022167828866
- link LFinger43_link: mass 2e-06 -> 0.0012119663070476055
- link LForeArm: mass 0.16579 -> 0.13321114815783727
- link LShoulder: mass 0.3125 -> 0.1407150721615769
- link LThumb1_link: mass 2e-06 -> 0.0017342022979805805
- link LThumb2_link: mass 2e-06 -> 0.001211966381471568
- link Neck: mass 0.27391 -> 0.09146568603258816
- link Pelvis: mass 2.4592 -> 3.7955398538315377
- link RBicep: mass 0.50527 -> 0.3137032437994389
- link RElbow: mass 0.27495 -> 0.07380464672624755
- link RFinger11_link: mass 2e-06 -> 0.0017342022611750378
- link RFinger12_link: mass 2e-06 -> 0.001734202280194698
- link RFinger13_link: mass 2e-06 -> 0.001211966381471568
- link RFinger21_link: mass 2e-06 -> 0.0017342022480607796
- link RFinger22_link: mass 2e-06 -> 0.001734202428057582
- link RFinger23_link: mass 2e-06 -> 0.0012119663699255415
- link RFinger31_link: mass 2e-06 -> 0.001734202271258544
- link RFinger32_link: mass 2e-06 -> 0.0017342022235830492
- link RFinger33_link: mass 2e-06 -> 0.0012119665608007826
- link RFinger41_link: mass 2e-06 -> 0.0017342022888397826
- link RFinger42_link: mass 2e-06 -> 0.0017342022167828866
- link RFinger43_link: mass 2e-06 -> 0.0012119663070476055
- link RForeArm: mass 0.16579 -> 0.13321114815783727
- link RShoulder: mass 0.3125 -> 0.1407150721615769
- link RThumb1_link: mass 2e-06 -> 0.0017342022979805805
- link RThumb2_link: mass 2e-06 -> 0.001211966381471568
- link Tibia: mass 15.485 -> 12.344158152172728
- link WheelB_link: mass 0.804686790979882 -> 0.7575690266305116
- link WheelFL_link: mass 0.8046868029667374 -> 0.7575690379154867
- link WheelFR_link: mass 0.804686767473058 -> 0.75756900450011
- link l_gripper: mass 2e-06 -> 0.207591874180564
- link l_wrist: mass 0.27555 -> 0.207591874180564
- link r_gripper: mass 2e-06 -> 0.20759187418056393
- link r_wrist: mass 0.27555 -> 0.20759187418056393
- link torso: mass 3.9953 -> 4.89481724014063
Joints:
- joint HipPitch: limit lower=-1.0385 upper=1.0385 effort=19.787 velocity=2.93276 -> lower=-1.03847 upper=1.03847 effort=19.787 velocity=2.93276
- joint HipRoll: limit lower=-0.5149 upper=0.5149 effort=10.1884 velocity=2.27032 -> lower=-0.514872 upper=0.514872 effort=10.1884 velocity=2.27032
- joint KneePitch: limit lower=-0.5149 upper=0.5149 effort=27.702 velocity=2.93276 -> lower=-0.514872 upper=0.514872 effort=27.702 velocity=2.93276
- joint LElbowRoll: limit lower=-1.5620 upper=-0.0087 effort=2.666 velocity=9.22756 -> lower=-1.56207 upper=-0.00872665 effort=2.666 velocity=9.22756
- joint LElbowYaw: limit lower=-2.0857 upper=2.0857 effort=5.428 velocity=7.33998 -> lower=-2.08567 upper=2.08567 effort=5.428 velocity=7.33998
- joint LShoulderPitch: limit lower=-2.0857 upper=2.0857 effort=5.428 velocity=7.33998 -> lower=-2.08567 upper=2.08567 effort=5.428 velocity=7.33998
- joint LShoulderRoll: limit lower=0.0087 upper=1.56207 effort=2.666 velocity=9.22756 -> lower=0.00872665 upper=1.56207 effort=2.666 velocity=9.22756
- joint LWristYaw: limit lower=-1.8239 upper=1.8239 effort=0.2014 velocity=17.3835 -> lower=-1.82387 upper=1.82387 effort=0.2014 velocity=17.3835
- joint RElbowRoll: limit lower=0.0087 upper=1.5620 effort=2.666 velocity=9.22756 -> lower=0.00872665 upper=1.56207 effort=2.666 velocity=9.22756
- joint RWristYaw: limit lower=-1.8239 upper=1.8239 effort=0.2014 velocity=17.3835 -> lower=-1.82387 upper=1.82387 effort=0.2014 velocity=17.3835

Commit message: fix urdf and sdf

File: pepper_robot_description/urdf/pepper_robot.urdf (robot description, URDF)
Before this commit: robot pepper_robot, 50 links, 49 joints
Links:
- link Head: mass 3.7955398538315377 -> 1.5189
- link Hip: mass 1.007402858772892 -> 1.0234
- link LBicep: mass 0.3137032437994389 -> 0.50527
- link LElbow: mass 0.07380464672624755 -> 0.27495
- link LFinger11_link: mass 0.0017342022611750378 -> 2e-06
- link LFinger12_link: mass 0.001734202280194698 -> 2e-06
- link LFinger13_link: mass 0.001211966381471568 -> 2e-06
- link LFinger21_link: mass 0.0017342022480607796 -> 2e-06
- link LFinger22_link: mass 0.001734202428057582 -> 2e-06
- link LFinger23_link: mass 0.0012119663699255415 -> 2e-06
- link LFinger31_link: mass 0.001734202271258544 -> 2e-06
- link LFinger32_link: mass 0.0017342022235830492 -> 2e-06
- link LFinger33_link: mass 0.0012119665608007826 -> 2e-06
- link LFinger41_link: mass 0.0017342022888397826 -> 2e-06
- link LFinger42_link: mass 0.0017342022167828866 -> 2e-06
- link LFinger43_link: mass 0.0012119663070476055 -> 2e-06
- link LForeArm: mass 0.13321114815783727 -> 0.16579
- link LShoulder: mass 0.1407150721615769 -> 0.3125
- link LThumb1_link: mass 0.0017342022979805805 -> 2e-06
- link LThumb2_link: mass 0.001211966381471568 -> 2e-06
- link Neck: mass 0.09146568603258816 -> 0.27391
- link Pelvis: mass 3.7955398538315377 -> 2.4592
- link RBicep: mass 0.3137032437994389 -> 0.50527
- link RElbow: mass 0.07380464672624755 -> 0.27495
- link RFinger11_link: mass 0.0017342022611750378 -> 2e-06
- link RFinger12_link: mass 0.001734202280194698 -> 2e-06
- link RFinger13_link: mass 0.001211966381471568 -> 2e-06
- link RFinger21_link: mass 0.0017342022480607796 -> 2e-06
- link RFinger22_link: mass 0.001734202428057582 -> 2e-06
- link RFinger23_link: mass 0.0012119663699255415 -> 2e-06
- link RFinger31_link: mass 0.001734202271258544 -> 2e-06
- link RFinger32_link: mass 0.0017342022235830492 -> 2e-06
- link RFinger33_link: mass 0.0012119665608007826 -> 2e-06
- link RFinger41_link: mass 0.0017342022888397826 -> 2e-06
- link RFinger42_link: mass 0.0017342022167828866 -> 2e-06
- link RFinger43_link: mass 0.0012119663070476055 -> 2e-06
- link RForeArm: mass 0.13321114815783727 -> 0.16579
- link RShoulder: mass 0.1407150721615769 -> 0.3125
- link RThumb1_link: mass 0.0017342022979805805 -> 2e-06
- link RThumb2_link: mass 0.001211966381471568 -> 2e-06
- link Tibia: mass 12.344158152172728 -> 15.485
- link WheelB_link: mass 0.7575690266305116 -> 1.29464
- link WheelFL_link: mass 0.7575690379154867 -> 1.29464
- link WheelFR_link: mass 0.75756900450011 -> 1.29464
- link l_gripper: mass 0.207591874180564 -> 2e-06
- link l_wrist: mass 0.207591874180564 -> 0.27555
- link r_gripper: mass 0.20759187418056393 -> 2e-06
- link r_wrist: mass 0.20759187418056393 -> 0.27555
- link torso: mass 4.89481724014063 -> 3.9953
Joints:
- joint HipPitch: limit lower=-1.03847 upper=1.03847 effort=19.787 velocity=2.93276 -> lower=-1.0385 upper=1.0385 effort=19.787 velocity=2.93276
- joint HipRoll: limit lower=-0.514872 upper=0.514872 effort=10.1884 velocity=2.27032 -> lower=-0.5149 upper=0.5149 effort=10.1884 velocity=2.27032
- joint KneePitch: limit lower=-0.514872 upper=0.514872 effort=27.702 velocity=2.93276 -> lower=-0.5149 upper=0.5149 effort=27.702 velocity=2.93276
- joint RElbowRoll: limit lower=0.00872665 upper=1.56207 effort=2.666 velocity=9.22756 -> lower=0.0087 upper=1.5620 effort=2.666 velocity=9.22756
- joint RWristYaw: limit lower=-1.82387 upper=1.82387 effort=0.2014 velocity=17.3835 -> lower=-1.8239 upper=1.8239 effort=0.2014 velocity=17.3835

Commit message: change inertial properties

File: pepper_robot_description/urdf/pepper_robot.urdf (robot description, URDF)
Before this commit: robot pepper_robot, 50 links, 49 joints
Links:
- link Head: mass 1.5189 -> 1.51893
- link Hip: mass 1.0234 -> 1.02338
- link Pelvis: mass 2.4592 -> 2.45917
- link Tibia: mass 15.485 -> 11.6015
- link WheelB_link: mass 1.29464 -> 1.58028
- link WheelFL_link: mass 1.29464 -> 1.58028
- link WheelFR_link: mass 1.29464 -> 1.58028
- link torso: mass 3.9953 -> 3.99533

Commit message: replace the meshes with meshes compatible with ros2

File: pepper_robot_description/urdf/pepper_robot.urdf (robot description, URDF)
Before this commit: robot pepper_robot, 50 links, 49 joints
Links:
- link Head: mass 1.51893 -> 1.5189
- link Hip: mass 1.02338 -> 1.0234
- link Pelvis: mass 2.45917 -> 2.4592
- link Tibia: mass 11.6015 -> 15.485
- link WheelB_link: mass 1.58028 -> 1.29464
- link WheelFL_link: mass 1.58028 -> 1.29464
- link WheelFR_link: mass 1.58028 -> 1.29464
- link torso: mass 3.99533 -> 3.9953

Commit message: change urdf and sdf

File: pepper_robot_description/urdf/pepper_robot.urdf (robot description, URDF)
Before this commit: robot pepper_robot, 50 links, 49 joints
Links:
- link Head: mass 1.5189 -> 3.7955398538315377
- link Hip: mass 1.0234 -> 1.007402858772892
- link LBicep: mass 0.50527 -> 0.3137032437994389
- link LElbow: mass 0.27495 -> 0.07380464672624755
- link LFinger11_link: mass 2e-06 -> 0.0017342022611750378
- link LFinger12_link: mass 2e-06 -> 0.001734202280194698
- link LFinger13_link: mass 2e-06 -> 0.001211966381471568
- link LFinger21_link: mass 2e-06 -> 0.0017342022480607796
- link LFinger22_link: mass 2e-06 -> 0.001734202428057582
- link LFinger23_link: mass 2e-06 -> 0.0012119663699255415
- link LFinger31_link: mass 2e-06 -> 0.001734202271258544
- link LFinger32_link: mass 2e-06 -> 0.0017342022235830492
- link LFinger33_link: mass 2e-06 -> 0.0012119665608007826
- link LFinger41_link: mass 2e-06 -> 0.0017342022888397826
- link LFinger42_link: mass 2e-06 -> 0.0017342022167828866
- link LFinger43_link: mass 2e-06 -> 0.0012119663070476055
- link LForeArm: mass 0.16579 -> 0.13321114815783727
- link LShoulder: mass 0.3125 -> 0.1407150721615769
- link LThumb1_link: mass 2e-06 -> 0.0017342022979805805
- link LThumb2_link: mass 2e-06 -> 0.001211966381471568
- link Neck: mass 0.27391 -> 0.09146568603258816
- link Pelvis: mass 2.4592 -> 3.7955398538315377
- link RBicep: mass 0.50527 -> 0.3137032437994389
- link RElbow: mass 0.27495 -> 0.07380464672624755
- link RFinger11_link: mass 2e-06 -> 0.0017342022611750378
- link RFinger12_link: mass 2e-06 -> 0.001734202280194698
- link RFinger13_link: mass 2e-06 -> 0.001211966381471568
- link RFinger21_link: mass 2e-06 -> 0.0017342022480607796
- link RFinger22_link: mass 2e-06 -> 0.001734202428057582
- link RFinger23_link: mass 2e-06 -> 0.0012119663699255415
- link RFinger31_link: mass 2e-06 -> 0.001734202271258544
- link RFinger32_link: mass 2e-06 -> 0.0017342022235830492
- link RFinger33_link: mass 2e-06 -> 0.0012119665608007826
- link RFinger41_link: mass 2e-06 -> 0.0017342022888397826
- link RFinger42_link: mass 2e-06 -> 0.0017342022167828866
- link RFinger43_link: mass 2e-06 -> 0.0012119663070476055
- link RForeArm: mass 0.16579 -> 0.13321114815783727
- link RShoulder: mass 0.3125 -> 0.1407150721615769
- link RThumb1_link: mass 2e-06 -> 0.0017342022979805805
- link RThumb2_link: mass 2e-06 -> 0.001211966381471568
- link Tibia: mass 15.485 -> 12.344158152172728
- link WheelB_link: mass 1.29464 -> 0.7575690266305116
- link WheelFL_link: mass 1.29464 -> 0.7575690379154867
- link WheelFR_link: mass 1.29464 -> 0.75756900450011
- link l_gripper: mass 2e-06 -> 0.207591874180564
- link l_wrist: mass 0.27555 -> 0.207591874180564
- link r_gripper: mass 2e-06 -> 0.20759187418056393
- link r_wrist: mass 0.27555 -> 0.20759187418056393
- link torso: mass 3.9953 -> 4.89481724014063
Joints:
- joint HipPitch: limit lower=-1.0385 upper=1.0385 effort=19.787 velocity=2.93276 -> lower=-1.03847 upper=1.03847 effort=19.787 velocity=2.93276
- joint HipRoll: limit lower=-0.5149 upper=0.5149 effort=10.1884 velocity=2.27032 -> lower=-0.514872 upper=0.514872 effort=10.1884 velocity=2.27032
- joint KneePitch: limit lower=-0.5149 upper=0.5149 effort=27.702 velocity=2.93276 -> lower=-0.514872 upper=0.514872 effort=27.702 velocity=2.93276
- joint RElbowRoll: limit lower=0.0087 upper=1.5620 effort=2.666 velocity=9.22756 -> lower=0.00872665 upper=1.56207 effort=2.666 velocity=9.22756
- joint RWristYaw: limit lower=-1.8239 upper=1.8239 effort=0.2014 velocity=17.3835 -> lower=-1.82387 upper=1.82387 effort=0.2014 velocity=17.3835
