Commit message: change inertial properties

File: pepper_robot_description/urdf/pepper_robot.urdf (robot description, URDF)
Before this commit: robot pepper_robot, 50 links, 49 joints
Links:
- link Head: mass 3.7955398538315377 -> 2.2879154181022487
- link Hip: mass 1.007402858772892 -> 0.9991965961004466
- link LBicep: mass 0.3137032437994389 -> 0.3111478299474749
- link LElbow: mass 0.07380464672624755 -> 0.0732034370788773
- link LForeArm: mass 0.13321114815783727 -> 0.13212601556846498
- link LShoulder: mass 0.1407150721615769 -> 0.13956881291278284
- link Neck: mass 0.09146568603258816 -> 0.09072061027807508
- link Pelvis: mass 3.7955398538315377 -> 3.7646215407127754
- link RBicep: mass 0.3137032437994389 -> 0.3111478299474749
- link RElbow: mass 0.07380464672624755 -> 0.0732034370788773
- link RForeArm: mass 0.13321114815783727 -> 0.13212601556846498
- link RShoulder: mass 0.1407150721615769 -> 0.13956881291278284
- link Tibia: mass 12.344158152172728 -> 12.243603142441735
- link l_gripper: mass 0.207591874180564 -> 0.2059008392253267
- link l_wrist: mass 0.207591874180564 -> 0.2059008392253267
- link r_wrist: mass 0.20759187418056393 -> 0.20590083922532662
- link torso: mass 4.89481724014063 -> 4.854944258188666
